Commit message: merge

File: unicorn_description/urdf/rplidar_a2.urdf.xacro (robot description, xacro)
@@ -1,5 +1,5 @@
 <?xml version="1.0"?>
 <robot xmlns:xacro="http://www.ros.org/wiki/xacro">
-	<xacro:macro name="rplidar_a2" params="frame:=laser topic:=scan
+	<xacro:macro name="rplidar_a2" params="frame:=scan topic:=/TX2_r2000Lidar/laserScan
 		robot_namespace:=/" >
 	   <link name="${frame}">
@@ -11,4 +11,7 @@
 	    <visual>
 		<origin xyz = "0.0 0.0 0.28" rpy= "0.0 0.0 0.0" />
+	        <geometry>
+		  <box size="0.07271 0.27794 0.073"/>
+	        </geometry>
    	    </visual>
 	    <collision>

File: unicorn_description/urdf/unicorn_target.urdf.xacro (robot description, xacro)
@@ -303,5 +303,5 @@
     </joint>
 -->
-   <rplidar_a2 frame="base_laser" topic="scan" robot_namespace="$(arg robot_namespace)"/>
+   <rplidar_a2 frame="base_laser" topic="/TX2_r2000Lidar/laserScan" robot_namespace="$(arg robot_namespace)"/>
    <joint name="laser_mount_joint" type="fixed">
       <origin xyz="$(arg laser_xyz)" rpy="$(arg laser_rpy)" />
