Commit message: Added lift to model in rviz

File: unicorn_description/urdf/lidar_gazebo.urdf.xacro (robot description, xacro)
@@ -31,9 +31,7 @@
     <link name="${frame}">
       <inertial>
-        <mass value="1.1" />
-        <origin xyz="0 0 0" />
-        <inertia ixx="${0.0833333 * 1.1 * (0.102*0.102 + 0.152*0.152)}" ixy="0.0" ixz="0.0"
-          iyy="${0.0833333 * 1.1 * (0.105*0.105 + 0.152*0.152)}" iyz="0.0"
-          izz="${0.0833333 * 1.1 * (0.105*0.105 + 0.102*0.102)}" />
+        <mass value="0" />
+        <origin xyz="0 0 0" rpy="0 0 0"/>
+        <inertia ixx="0" ixy="0" ixz="0" iyy="0" iyz="0" izz="0" />
       </inertial>
       <visual>

File: unicorn_description/urdf/stereo_camera_gazebo.urdf.xacro (robot description, xacro)
@@ -5,7 +5,7 @@
     <link name="${frame_rgb}">
       <inertial>
-        <mass value="1e-5" />
+        <mass value="0" />
         <origin xyz="0 0 0" rpy="0 0 0"/>
-        <inertia ixx="0.5" ixy="0" ixz="0" iyy="0.5" iyz="0" izz="0.5" />
+        <inertia ixx="0" ixy="0" ixz="0" iyy="0" iyz="0" izz="0" />
       </inertial>
      <visual>

File: unicorn_description/urdf/unicorn_sim.urdf.xacro (robot description, xacro)
@@ -38,4 +38,5 @@
   <xacro:arg name="real_rpy" default="0 0 ${M_PI}" />
   <xacro:arg name="realsense_meshfile" default="package://unicorn_description/meshes/real_sense.STL" />
+ <!-- Main Body-base -->
   <link
     name="chassis_link">
@@ -47,10 +48,10 @@
         value="15" />
       <inertia
-        ixx="0.5"
+        ixx="1"
         ixy="0"
-        ixz="0"
+        ixz="3"
         iyy="3"
-        iyz="0"
-        izz="0.5" />
+        iyz="3"
+        izz="1" />
     </inertial>
     <visual>
@@ -78,7 +79,7 @@
     </collision>
   </link>
-    <!-- Main Body-base
+<!-- Lift -->
   <link
-    name="base_link_gazebo">
+    name="lift_link">
     <inertial>
       <origin
@@ -86,6 +87,12 @@
         rpy="0 0 0" />
       <mass
-        value="0.01" />
-      <box_inertia  m="${5}" x="${base_x_size}" y="${base_y_size}" z="${base_z_size}"/>
+        value="4" />
+      <inertia
+        ixx="1"
+        ixy="0"
+        ixz="3"
+        iyy="3"
+        iyz="3"
+        izz="1" />
     </inertial>
     <visual>
@@ -94,10 +101,11 @@
         rpy="0 0 0" />
       <geometry>
-        <box size="0.1 0.1 0.1"/>
+        <mesh
+          filename="package://unicorn_description/meshes/lift_link.STL" />
       </geometry>
       <material
         name="">
         <color
-          rgba="0.79216 0.81961 0.93333 1" />
+          rgba="0.752941176470588 0.752941176470588 0.752941176470588 1" />
       </material>
     </visual>
@@ -107,25 +115,26 @@
         rpy="0 0 0" />
       <geometry>
-          <box size="0.01 0.01 0.01"/>
+        <mesh
+          filename="package://unicorn_description/meshes/lift_link.STL" />
       </geometry>
-       <surface>
-         <friction>
-           <ode><mu>0</mu><mu2>0</mu2></ode>
-         </friction>
-      </surface>
     </collision>
   </link>
-  <gazebo reference="base_link_gazebo">
-    <material>Gazebo/Green</material>
-    <turnGravityOff>false</turnGravityOff>
-  </gazebo>
-  <joint name="base_link_gazebo_joint" type="fixed">
-    <parent link="chassis_link"/>
-    <child link="base_link_gazebo" />
-  <origin xyz="0 0.0 0" rpy="0 0 ${M_PI}" />
-  </joint> -->
+  <joint
+    name="lift_joint"
+    type="fixed">
+    <origin
+      xyz="0 0 0"
+      rpy="0 0 0" />
+    <parent
+      link="chassis_link" />
+    <child
+      link="lift_link" />
+    <axis
+      xyz="0 0 0" />
+    <joint_properties damping="0.0" friction="0.0" />
+  </joint>
   <!-- driving wheels -->
-  <wheel fb="back" lr="left" parent="chassis_link" translateY="0.24" translateX="0" translateZ="0.122" wheel_radius="0.1225" wheel_height="0.032" flip="1"/>
-  <wheel fb="back" lr="right" parent="chassis_link" translateY="-0.24" translateX="0 " translateZ="0.122" wheel_radius="0.1225" wheel_height="0.032" flip="1"/>
+  <wheel fb="back" lr="left" parent="chassis_link" translateY="0.25" translateX="0" translateZ="0.122" wheel_radius="0.122" wheel_height="0.032" flip="1"/>
+  <wheel fb="back" lr="right" parent="chassis_link" translateY="-0.25" translateX="0 " translateZ="0.122" wheel_radius="0.122" wheel_height="0.032" flip="1"/>
   <!-- others wheels -->
   <swivel_wheel fb="front" lr="left" parent="chassis_link" translateY="0.16" translateX="-0.355" translateZ="0.1526" wheel_radius="0.05" wheel_height="0.05" flip="0"/>

File: unicorn_description/urdf/unicorn_target.urdf.xacro (robot description, xacro)
@@ -38,4 +38,5 @@
   <xacro:arg name="real_rpy" default="0 0 ${M_PI}" />
   <xacro:arg name="realsense_meshfile" default="package://unicorn_description/meshes/real_sense.STL" />
+ <!-- Main Body-base -->
   <link
     name="chassis_link">
@@ -47,10 +48,10 @@
         value="15" />
       <inertia
-        ixx="0.5"
+        ixx="1"
         ixy="0"
-        ixz="0"
+        ixz="3"
         iyy="3"
-        iyz="0"
-        izz="0.5" />
+        iyz="3"
+        izz="1" />
     </inertial>
     <visual>
@@ -78,7 +79,7 @@
     </collision>
   </link>
-    <!-- Main Body-base
+<!-- Lift -->
   <link
-    name="base_link_gazebo">
+    name="lift_link">
     <inertial>
       <origin
@@ -86,6 +87,12 @@
         rpy="0 0 0" />
       <mass
-        value="0.01" />
-      <box_inertia  m="${5}" x="${base_x_size}" y="${base_y_size}" z="${base_z_size}"/>
+        value="4" />
+      <inertia
+        ixx="1"
+        ixy="0"
+        ixz="3"
+        iyy="3"
+        iyz="3"
+        izz="1" />
     </inertial>
     <visual>
@@ -94,10 +101,11 @@
         rpy="0 0 0" />
       <geometry>
-        <box size="0.1 0.1 0.1"/>
+        <mesh
+          filename="package://unicorn_description/meshes/lift_link.STL" />
       </geometry>
       <material
         name="">
         <color
-          rgba="0.79216 0.81961 0.93333 1" />
+          rgba="0.752941176470588 0.752941176470588 0.752941176470588 1" />
       </material>
     </visual>
@@ -107,25 +115,26 @@
         rpy="0 0 0" />
       <geometry>
-          <box size="0.01 0.01 0.01"/>
+        <mesh
+          filename="package://unicorn_description/meshes/lift_link.STL" />
       </geometry>
-       <surface>
-         <friction>
-           <ode><mu>0</mu><mu2>0</mu2></ode>
-         </friction>
-      </surface>
     </collision>
   </link>
-  <gazebo reference="base_link_gazebo">
-    <material>Gazebo/Green</material>
-    <turnGravityOff>false</turnGravityOff>
-  </gazebo>
-  <joint name="base_link_gazebo_joint" type="fixed">
-    <parent link="chassis_link"/>
-    <child link="base_link_gazebo" />
-  <origin xyz="0 0.0 0" rpy="0 0 ${M_PI}" />
-  </joint> -->
+  <joint
+    name="lift_joint"
+    type="fixed">
+    <origin
+      xyz="0 0 0"
+      rpy="0 0 0" />
+    <parent
+      link="chassis_link" />
+    <child
+      link="lift_link" />
+    <axis
+      xyz="0 0 0" />
+    <joint_properties damping="0.0" friction="0.0" />
+  </joint>
   <!-- driving wheels -->
-  <wheel fb="back" lr="left" parent="chassis_link" translateY="0.24" translateX="0" translateZ="0.122" wheel_radius="0.1225" wheel_height="0.032" flip="1"/>
-  <wheel fb="back" lr="right" parent="chassis_link" translateY="-0.24" translateX="0 " translateZ="0.122" wheel_radius="0.1225" wheel_height="0.032" flip="1"/>
+  <wheel fb="back" lr="left" parent="chassis_link" translateY="0.25" translateX="0" translateZ="0.122" wheel_radius="0.122" wheel_height="0.032" flip="1"/>
+  <wheel fb="back" lr="right" parent="chassis_link" translateY="-0.25" translateX="0 " translateZ="0.122" wheel_radius="0.122" wheel_height="0.032" flip="1"/>
   <!-- others wheels -->
   <swivel_wheel fb="front" lr="left" parent="chassis_link" translateY="0.16" translateX="-0.355" translateZ="0.1526" wheel_radius="0.05" wheel_height="0.05" flip="0"/>
@@ -267,5 +276,5 @@
     <rpyOffsets>0 0 0</rpyOffsets> <!-- deprecated -->
 <!--
-      <gaussianNoise>0.0</gaussianNoise>
+      <gaussianNoise>0.1</gaussianNoise>
       <accelDrift>0.5 0.5 0.5</accelDrift>
       <accelGaussianNoise>0.35 0.35 0.3</accelGaussianNoise>
@@ -273,13 +282,30 @@
       <rateGaussianNoise>0.05 0.05 0.015</rateGaussianNoise>
       <headingDrift>0.1</headingDrift>
-      <headingGaussianNoise>1.00</headingGaussianNoise>
--->
-    <gaussianNoise>0.0</gaussianNoise>  <!-- deprecated -->
-      <accelDrift>0.0 0.0 0.0</accelDrift>
-      <accelGaussianNoise>0.0 0.0 0.0</accelGaussianNoise>
-      <rateDrift>0.0 0.0 0.0</rateDrift>
-      <rateGaussianNoise>0.0 0.0 0.0</rateGaussianNoise>
-      <headingDrift>0.0</headingDrift>
-      <headingGaussianNoise>0.00</headingGaussianNoise>
+      <headingGaussianNoise>1.00</headingGaussianNoise>-->
+    </plugin>
+    <plugin name="gazebo_ros_control" filename="libgazebo_ros_control.so" />
+    <plugin name="imu_plugin" filename="libhector_gazebo_ros_imu.so">
+      <alwaysOn>true</alwaysOn>
+      <bodyName>chassis_link</bodyName>
+      <topicName>zed/imu</topicName>
+      <serviceName>imu_service</serviceName>
+      <updateRate>10.0</updateRate>
+      <rpyOffsets>0 0 0</rpyOffsets> <!-- deprecated -->
+  <!--
+        <gaussianNoise>0.1</gaussianNoise>
+        <accelDrift>0.5 0.5 0.5</accelDrift>
+        <accelGaussianNoise>0.35 0.35 0.3</accelGaussianNoise>
+        <rateDrift>0.1 0.1 0.1</rateDrift>
+        <rateGaussianNoise>0.05 0.05 0.015</rateGaussianNoise>
+        <headingDrift>0.1</headingDrift>
+        <headingGaussianNoise>1.00</headingGaussianNoise>-->
+  <!-- deprecated -->
+      <gaussianNoise>0.0</gaussianNoise>
+        <accelDrift>0.0 0.0 0.0</accelDrift>
+        <accelGaussianNoise>0.0 0.0 0.0</accelGaussianNoise>
+        <rateDrift>0.0 0.0 0.0</rateDrift>
+        <rateGaussianNoise>0.0 0.0 0.0</rateGaussianNoise>
+        <headingDrift>0.0</headingDrift>
+        <headingGaussianNoise>0.00</headingGaussianNoise>
     </plugin>
     <plugin name="am_gazebo_wheelencoder" filename="libam_gazebo_wheelencoder.so">
