Commit message: Updated urdf to reduce unwanted movment and changed frame in target for realsense

File: unicorn_description/urdf/lidar_gazebo.urdf.xacro (robot description, xacro)
@@ -30,9 +30,4 @@
     <xacro:arg name="sim" default="${simulation}" />
     <link name="${frame}">
-      <inertial>
-        <mass value="0" />
-        <origin xyz="0 0 0" rpy="0 0 0"/>
-        <inertia ixx="0" ixy="0" ixz="0" iyy="0" iyz="0" izz="0" />
-      </inertial>
       <visual>
         <origin xyz="0 0 0" rpy="0 0 0" />
@@ -42,13 +37,4 @@
         </geometry>
       </visual>
-      <collision>
-        <origin
-            xyz="0 0 0"
-            rpy="0 0 0" />
-        <geometry>
-            <mesh
-            filename="${filename}" />
-        </geometry>
-      </collision>
     </link>
     <xacro:if value="$(arg sim)">

File: unicorn_description/urdf/stereo_camera_gazebo.urdf.xacro (robot description, xacro)
@@ -4,9 +4,4 @@
   <xacro:arg name="sim" default="${simulation}" />
     <link name="${frame_rgb}">
-      <inertial>
-        <mass value="0" />
-        <origin xyz="0 0 0" rpy="0 0 0"/>
-        <inertia ixx="0" ixy="0" ixz="0" iyy="0" iyz="0" izz="0" />
-      </inertial>
      <visual>
         <origin xyz="0 0 0" rpy="0 0 0"/>
@@ -15,13 +10,6 @@
         </geometry>
       </visual>
-      <collision>
-        <origin xyz="0 0 0" rpy="0 0 0"/>
-        <geometry>
-          <mesh
-            filename="${filename}" />
-        </geometry>
-      </collision>
     </link>
-<!-- -->
+<!-- Gazebo simulation -->
     <link name="${frame_depth}"></link>
     <xacro:if value="$(arg sim)">

File: unicorn_description/urdf/swivel_wheel.urdf.xacro (robot description, xacro)
@@ -85,6 +85,6 @@
           <friction>
             <ode>
-              <mu>0.05</mu>
-              <mu2>0.05</mu2>
+              <mu>0.4</mu>
+              <mu2>0.4</mu2>
             </ode>
           </friction>

File: unicorn_description/urdf/unicorn_sim.urdf.xacro (robot description, xacro)
@@ -52,4 +52,5 @@
   <link
     name="chassis_link">
+    <!--
     <inertial>
       <origin
@@ -65,5 +66,5 @@
         iyz="3"
         izz="1" />
-    </inertial>
+    </inertial>-->
     <visual>
       <origin
@@ -80,4 +81,5 @@
       </material>
     </visual>
+    <!--
     <collision>
       <origin
@@ -93,5 +95,5 @@
       </surface>
       </geometry>
-    </collision>
+    </collision>-->
   </link>
 <!-- Lift -->
@@ -111,5 +113,5 @@
         iyz="3"
         izz="1" />
-    </inertial>
+    </inertial>-
     <visual>
       <origin
@@ -150,50 +152,4 @@
     <joint_properties damping="1" friction="0.5" />
   </joint>
-<!--
-  <link
-    name="wheel_link">
-    <inertial>
-      <origin
-        xyz="0 0 0"
-        rpy="0 0 0" />
-      <mass
-        value="0.01" />
-      <box_inertia  m="${5*0.01}" x="${base_x_size}" y="${base_y_size}" z="${base_z_size}"/>
-    </inertial>
-    <visual>
-      <origin
-        xyz="0 0 0"
-        rpy="0 0 0" />
-      <geometry>
-        <box size="0.01 0.01 0.01"/>
-      </geometry>
-      <material
-        name="">
-        <color
-          rgba="0.79216 0.81961 0.93333 1" />
-      </material>
-    </visual>
-    <collision>
-      <origin
-        xyz="0 0 0"
-        rpy="0 0 0" />
-      <geometry>
-          <box size="0.01 0.01 0.01"/>
-      </geometry>
-    </collision>
-  </link>
-  <gazebo reference="base_link_gazebo">
-    <material>Gazebo/Green</material>
-    <turnGravityOff>false</turnGravityOff>
-  </gazebo>
-  <joint name="base_chassis_joint" type="fixed">
-    <parent link="chassis_link"/>
-    <child link="wheel_link" />
-  <origin xyz="0 0.0 0" rpy="0 0 ${M_PI}" />
-  </joint>-->
-  <!-- driving wheels
-  <wheel fb="back" lr="left" parent="chassis_link" rotationZ="3.14159" translateY="0.23" translateX="0" translateZ="0.1225" wheel_radius="0.1225" wheel_height="0.032" flip="1"/>
-  <wheel fb="back" lr="right" parent="chassis_link" rotationZ="0" translateY="-0.23" translateX="0 " translateZ="0.1225" wheel_radius="0.1225" wheel_height="0.032" flip="1"/>
-  -->
   <wheel fb="back" lr="left" parent="lift_link"  translateY="0.24" translateX="0" translateZ="0.1225" wheel_radius="0.1225" wheel_height="0.032" flip="1"/>
   <wheel fb="back" lr="right" parent="lift_link" translateY="-0.24" translateX="0 " translateZ="0.1225" wheel_radius="0.1225" wheel_height="0.032" flip="1"/>
@@ -207,5 +163,4 @@
     <parent link="chassis_link" />
     <child link="base_laser" />
-    <joint_properties damping="1" friction="0.5" />
   </joint>
    <!-- Back Lidar -->
@@ -215,5 +170,4 @@
     <parent link="chassis_link" />
     <child link="rear_laser" />
-    <joint_properties damping="1" friction="0.5" />
   </joint>
   <!-- Zed Camera -->
@@ -223,5 +177,4 @@
       <parent link="chassis_link"/>
       <child link="zed_camera"/>
-      <joint_properties damping="1" friction="0.5" />
     </joint>
     <joint name="zed_camera_depth_joint" type="fixed">
@@ -229,28 +182,18 @@
       <parent link="zed_camera"/>
       <child link="zed_depth"/>
-      <joint_properties damping="1" friction="0.5" />
     </joint>
   <!-- realsense Camera -->
+  <link
+    name="realsense_link">
+  </link>
+  <joint name="realsense_joint" type="fixed">
+    <origin xyz="$(arg real_base)" rpy="$(arg real_rpy)"/>
+    <parent link="chassis_link"/>
+    <child link="realsense_link"/>
+  </joint>
+  <!-- Links only needed in simulation, created by realsense software otherwise-->
+<xacro:if value="$(arg sim)">
   <stereo_camera frame_rgb="realsense_color_frame" frame_depth="realsense_depth_frame" cameraName="realsense" simulation="$(arg sim)" filename="$(arg realsense_meshfile)"  topic="pointcloud" robot_namespace="$(arg robot_namespace)"/>
   <link
-    name="realsense_link">
-    <inertial>
-      <origin
-        xyz="0 0 0"
-        rpy="0 0 0" />
-      <mass
-        value="0.01" />
-      <box_inertia  m="${5*0.01}" x="${base_x_size}" y="${base_y_size}" z="${base_z_size}"/>
-    </inertial>
-    <collision>
-      <origin
-        xyz="0 0 0"
-        rpy="0 0 0" />
-      <geometry>
-          <box size="0.01 0.01 0.01"/>
-      </geometry>
-    </collision>
-  </link>
-  <link
     name="realsense_depth_optical_frame">
   </link>
@@ -258,29 +201,25 @@
     name="realsense_color_optical_frame">
   </link>
-    <joint name="realsense_joint" type="fixed">
-      <origin xyz="$(arg real_base)" rpy="$(arg real_rpy)"/>
-      <parent link="chassis_link"/>
-      <child link="realsense_link"/>
-    </joint>
-    <joint name="realsense_gb_joint" type="fixed">
-      <origin xyz="$(arg real_rgb_xyz)" rpy="0 0 0"/>
-      <parent link="realsense_link"/>
-      <child link="realsense_color_frame"/>
-    </joint>
-    <joint name="realsense_depth_joint" type="fixed">
-      <origin xyz="$(arg real_depth_xyz)" rpy="0 0 0"/>
-      <parent link="realsense_link"/>
-      <child link="realsense_depth_frame"/>
-    </joint>
-    <joint name="realsense_optical_color_joint" type="fixed">
-      <origin xyz="0 0 0" rpy="$(arg real_optical_rpy)"/>
-      <parent link="realsense_color_frame"/>
-      <child link="realsense_color_optical_frame"/>
-    </joint>
-    <joint name="realsense_optical_depth_joint" type="fixed">
-      <origin xyz="0 0 0" rpy="$(arg real_depth_rpy)"/>
-      <parent link="realsense_depth_frame"/>
-      <child link="realsense_depth_optical_frame"/>
-    </joint>
+  <joint name="realsense_gb_joint" type="fixed">
+    <origin xyz="$(arg real_rgb_xyz)" rpy="0 0 0"/>
+    <parent link="realsense_link"/>
+    <child link="realsense_color_frame"/>
+  </joint>
+  <joint name="realsense_depth_joint" type="fixed">
+    <origin xyz="$(arg real_depth_xyz)" rpy="0 0 0"/>
+    <parent link="realsense_link"/>
+    <child link="realsense_depth_frame"/>
+  </joint>
+  <joint name="realsense_optical_color_joint" type="fixed">
+    <origin xyz="0 0 0" rpy="$(arg real_optical_rpy)"/>
+    <parent link="realsense_color_frame"/>
+    <child link="realsense_color_optical_frame"/>
+  </joint>
+  <joint name="realsense_optical_depth_joint" type="fixed">
+    <origin xyz="0 0 0" rpy="$(arg real_depth_rpy)"/>
+    <parent link="realsense_depth_frame"/>
+    <child link="realsense_depth_optical_frame"/>
+  </joint>
+</xacro:if>
 <xacro:if value="$(arg sim)">
   <!-- GPS -->

File: unicorn_description/urdf/unicorn_target.urdf.xacro (robot description, xacro)
@@ -224,24 +224,15 @@
     </joint>
   <!-- realsense Camera -->
-    <stereo_camera frame_rgb="realsense_color_frame" frame_depth="realsense_depth_frame" cameraName="realsense" simulation="$(arg sim)" filename="$(arg realsense_meshfile)"  topic="pointcloud" robot_namespace="$(arg robot_namespace)"/>
   <link
     name="realsense_link">
-    <inertial>
-      <origin
-        xyz="0 0 0"
-        rpy="0 0 0" />
-      <mass
-        value="0.01" />
-      <box_inertia  m="${5*0.01}" x="${base_x_size}" y="${base_y_size}" z="${base_z_size}"/>
-    </inertial>
-    <collision>
-      <origin
-        xyz="0 0 0"
-        rpy="0 0 0" />
-      <geometry>
-          <box size="0.01 0.01 0.01"/>
-      </geometry>
-    </collision>
-  </link>
+  </link>
+  <joint name="realsense_joint" type="fixed">
+    <origin xyz="$(arg real_base)" rpy="$(arg real_rpy)"/>
+    <parent link="base_link"/>
+    <child link="realsense_link"/>
+  </joint>
+  <!-- Links only needed in simulation, created by realsense software otherwise-->
+<xacro:if value="$(arg sim)">
+  <stereo_camera frame_rgb="realsense_color_frame" frame_depth="realsense_depth_frame" cameraName="realsense" simulation="$(arg sim)" filename="$(arg realsense_meshfile)"  topic="pointcloud" robot_namespace="$(arg robot_namespace)"/>
   <link
     name="realsense_depth_optical_frame">
@@ -250,29 +241,25 @@
     name="realsense_color_optical_frame">
   </link>
-    <joint name="realsense_joint" type="fixed">
-      <origin xyz="$(arg real_base)" rpy="$(arg real_rpy)"/>
-      <parent link="chassis_link"/>
-      <child link="realsense_link"/>
-    </joint>
-    <joint name="realsense_gb_joint" type="fixed">
-      <origin xyz="$(arg real_rgb_xyz)" rpy="0 0 0"/>
-      <parent link="realsense_link"/>
-      <child link="realsense_color_frame"/>
-    </joint>
-    <joint name="realsense_depth_joint" type="fixed">
-      <origin xyz="$(arg real_depth_xyz)" rpy="0 0 0"/>
-      <parent link="realsense_link"/>
-      <child link="realsense_depth_frame"/>
-    </joint>
-    <joint name="realsense_optical_color_joint" type="fixed">
-      <origin xyz="0 0 0" rpy="$(arg real_optical_rpy)"/>
-      <parent link="realsense_color_frame"/>
-      <child link="realsense_color_optical_frame"/>
-    </joint>
-    <joint name="realsense_optical_depth_joint" type="fixed">
-      <origin xyz="0 0 0" rpy="$(arg real_depth_rpy)"/>
-      <parent link="realsense_depth_frame"/>
-      <child link="realsense_depth_optical_frame"/>
-    </joint>
+  <joint name="realsense_gb_joint" type="fixed">
+    <origin xyz="$(arg real_rgb_xyz)" rpy="0 0 0"/>
+    <parent link="realsense_link"/>
+    <child link="realsense_color_frame"/>
+  </joint>
+  <joint name="realsense_depth_joint" type="fixed">
+    <origin xyz="$(arg real_depth_xyz)" rpy="0 0 0"/>
+    <parent link="realsense_link"/>
+    <child link="realsense_depth_frame"/>
+  </joint>
+  <joint name="realsense_optical_color_joint" type="fixed">
+    <origin xyz="0 0 0" rpy="$(arg real_optical_rpy)"/>
+    <parent link="realsense_color_frame"/>
+    <child link="realsense_color_optical_frame"/>
+  </joint>
+  <joint name="realsense_optical_depth_joint" type="fixed">
+    <origin xyz="0 0 0" rpy="$(arg real_depth_rpy)"/>
+    <parent link="realsense_depth_frame"/>
+    <child link="realsense_depth_optical_frame"/>
+  </joint>
+</xacro:if>
 <xacro:if value="$(arg sim)">
   <!-- GPS -->

File: unicorn_description/urdf/unicorn_target_backwards.urdf.xacro (robot description, xacro)
@@ -2,5 +2,5 @@
 <robot name="unicorn" xmlns:xacro="http://www.ros.org/wiki/xacro">
   <xacro:arg name="robot_namespace" default="/" />
-  <xacro:arg name="sim" default="true" />
+  <xacro:arg name="sim" default="false" />
     <!-- Swivel wheel -->
   <xacro:include filename="$(find unicorn_description)/urdf/swivel_wheel.urdf.xacro" />
@@ -190,24 +190,15 @@
     </joint>
   <!-- realsense Camera -->
-    <stereo_camera frame_rgb="realsense_color_frame" frame_depth="realsense_depth_frame" cameraName="realsense" simulation="$(arg sim)" filename="$(arg realsense_meshfile)"  topic="pointcloud" robot_namespace="$(arg robot_namespace)"/>
   <link
     name="realsense_link">
-    <inertial>
-      <origin
-        xyz="0 0 0"
-        rpy="0 0 0" />
-      <mass
-        value="0.01" />
-      <box_inertia  m="${5*0.01}" x="${base_x_size}" y="${base_y_size}" z="${base_z_size}"/>
-    </inertial>
-    <collision>
-      <origin
-        xyz="0 0 0"
-        rpy="0 0 0" />
-      <geometry>
-          <box size="0.01 0.01 0.01"/>
-      </geometry>
-    </collision>
-  </link>
+  </link>
+  <joint name="realsense_joint" type="fixed">
+    <origin xyz="$(arg real_base)" rpy="$(arg real_rpy)"/>
+    <parent link="chassis_link"/>
+    <child link="realsense_link"/>
+  </joint>
+  <!-- Links only needed in simulation, created by realsense software otherwise-->
+<xacro:if value="$(arg sim)">
+  <stereo_camera frame_rgb="realsense_color_frame" frame_depth="realsense_depth_frame" cameraName="realsense" simulation="$(arg sim)" filename="$(arg realsense_meshfile)"  topic="pointcloud" robot_namespace="$(arg robot_namespace)"/>
   <link
     name="realsense_depth_optical_frame">
@@ -216,29 +207,25 @@
     name="realsense_color_optical_frame">
   </link>
-    <joint name="realsense_joint" type="fixed">
-      <origin xyz="$(arg real_base)" rpy="$(arg real_rpy)"/>
-      <parent link="chassis_link"/>
-      <child link="realsense_link"/>
-    </joint>
-    <joint name="realsense_gb_joint" type="fixed">
-      <origin xyz="$(arg real_rgb_xyz)" rpy="0 0 0"/>
-      <parent link="realsense_link"/>
-      <child link="realsense_color_frame"/>
-    </joint>
-    <joint name="realsense_depth_joint" type="fixed">
-      <origin xyz="$(arg real_depth_xyz)" rpy="0 0 0"/>
-      <parent link="realsense_link"/>
-      <child link="realsense_depth_frame"/>
-    </joint>
-    <joint name="realsense_optical_color_joint" type="fixed">
-      <origin xyz="0 0 0" rpy="$(arg real_optical_rpy)"/>
-      <parent link="realsense_color_frame"/>
-      <child link="realsense_color_optical_frame"/>
-    </joint>
-    <joint name="realsense_optical_depth_joint" type="fixed">
-      <origin xyz="0 0 0" rpy="$(arg real_depth_rpy)"/>
-      <parent link="realsense_depth_frame"/>
-      <child link="realsense_depth_optical_frame"/>
-    </joint>
+  <joint name="realsense_gb_joint" type="fixed">
+    <origin xyz="$(arg real_rgb_xyz)" rpy="0 0 0"/>
+    <parent link="realsense_link"/>
+    <child link="realsense_color_frame"/>
+  </joint>
+  <joint name="realsense_depth_joint" type="fixed">
+    <origin xyz="$(arg real_depth_xyz)" rpy="0 0 0"/>
+    <parent link="realsense_link"/>
+    <child link="realsense_depth_frame"/>
+  </joint>
+  <joint name="realsense_optical_color_joint" type="fixed">
+    <origin xyz="0 0 0" rpy="$(arg real_optical_rpy)"/>
+    <parent link="realsense_color_frame"/>
+    <child link="realsense_color_optical_frame"/>
+  </joint>
+  <joint name="realsense_optical_depth_joint" type="fixed">
+    <origin xyz="0 0 0" rpy="$(arg real_depth_rpy)"/>
+    <parent link="realsense_depth_frame"/>
+    <child link="realsense_depth_optical_frame"/>
+  </joint>
+</xacro:if>
 <xacro:if value="$(arg sim)">
   <!-- GPS -->

File: unicorn_description/urdf/wheel.urdf.xacro (robot description, xacro)
@@ -27,4 +27,12 @@
         <material name="Black" />
       </visual>
+      <surface>
+        <friction>
+          <ode>
+            <mu>0.4</mu>
+            <mu2>0.4</mu2>
+          </ode>
+        </friction>
+      </surface>
       <collision>
         <origin xyz="0 0 0" rpy="${flip*M_PI/2} 0 0" />
