Commit message: update robot urdf

File: unicorn_description/urdf/stereo_camera_gazebo.urdf.xacro (robot description, xacro)
@@ -1,22 +1,6 @@
 <?xml version="1.0"?>
 <robot xmlns:xacro="http://ros.org/wiki/xacro">
-  <xacro:macro name="stereo_camera" params="frame topic:=pointcloud robot_namespace:=/" >
-    <link name="${frame}">
-      <collision>
-        <origin xyz="0 0 0" rpy="0 0 0"/>
-        <geometry>
-          <box size="${0.05} ${0.05} ${0.05}"/>
-        </geometry>
-      </collision>
-      <visual>
-        <origin xyz="0 0 0" rpy="0 0 0"/>
-        <geometry>
-        <!-- Mesh file or a mesh box -->
-        <!-- Origin of this mesh is the focal point of the LIDAR. -->
-        <!-- <mesh filename="package://unicorn_description/stereo_camera_model/zed_model.dae" /> -->
-          <box size="${0.005} ${0.025} ${0.19}"/>
-        </geometry>
-        <material name="red"/>
-      </visual>
+  <xacro:macro name="stereo_camera" params="frame_rgb frame_depth topic:=pointcloud filename cameraName:=camera robot_namespace:=/" >
+    <link name="${frame_rgb}">
       <inertial>
         <mass value="1e-5" />
@@ -24,8 +8,22 @@
         <inertia ixx="1e-6" ixy="0" ixz="0" iyy="1e-6" iyz="0" izz="1e-6" />
       </inertial>
+     <visual>
+        <origin xyz="0 0 0" rpy="0 0 0"/>
+        <geometry>
+            <mesh filename="${filename}" />
+        </geometry>
+      </visual>
+      <collision>
+        <origin xyz="0 0 0" rpy="0 0 0"/>
+        <geometry>
+          <mesh
+            filename="${filename}" />
+        </geometry>
+      </collision>
     </link>
-    <link name="camera_left_depth_link"></link>
+<!-- -->
+    <link name="${frame_depth}"></link>
     <!-- camera -->
-    <gazebo reference="${frame}">
+    <gazebo reference="${frame_rgb}">
         <sensor type="depth" name="openni_camera_camera">
         <always_on>1</always_on>
@@ -46,14 +44,12 @@
           <baseline>0.2</baseline>
           <alwaysOn>true</alwaysOn>
-          <!-- Keep this zero, update_rate in the parent <sensor> tag
-            will control the frame rate. -->
           <updateRate>0.0</updateRate>
-          <cameraName>camera</cameraName>
-          <imageTopicName>/camera/depth/image_raw</imageTopicName>
-          <cameraInfoTopicName>/camera/depth/camera_info</cameraInfoTopicName>
-          <depthImageTopicName>/camera/depth/image_raw</depthImageTopicName>
-          <depthImageInfoTopicName>/camera/depth/camera_info</depthImageInfoTopicName>
-          <pointCloudTopicName>/camera/depth/points</pointCloudTopicName>
-          <frameName>camera_left_depth_link</frameName>
+          <cameraName>${cameraName}</cameraName>
+          <imageTopicName>/${cameraName}/depth/image_raw</imageTopicName>
+          <cameraInfoTopicName>/${cameraName}/depth/camera_info</cameraInfoTopicName>
+          <depthImageTopicName>/${cameraName}/depth/image_raw</depthImageTopicName>
+          <depthImageInfoTopicName>/${cameraName}/depth/camera_info</depthImageInfoTopicName>
+          <pointCloudTopicName>/${cameraName}/depth/points</pointCloudTopicName>
+          <frameName>${frame_depth}</frameName>
           <robotNamespace>${robot_namespace}</robotNamespace>
           <pointCloudCutoff>0.05</pointCloudCutoff>

File: unicorn_description/urdf/unicorn_sim.urdf.xacro (robot description, xacro)
@@ -1,55 +1,98 @@
-<?xml version="1.0"?>
+<?xml version="1.0" encoding="utf-8"?>
+<!-- This URDF was automatically created by SolidWorks to URDF Exporter! Originally created by Stephen Brawner (brawner@gmail.com)
+     Commit Version: 1.6.0-1-g15f4949  Build Version: 1.6.7594.29634
+     For more information, please see http://wiki.ros.org/sw_urdf_exporter -->
 <robot name="unicorn" xmlns:xacro="http://www.ros.org/wiki/xacro">
-  <!-- PROPERTY LIST -->
   <xacro:arg name="robot_namespace" default="/" />
-  <!--All units in m-kg-s-radians unit system -->
+    <!-- Swivel wheel -->
+  <xacro:include filename="$(find am_description)/urdf/swivel_wheel.urdf.xacro" />
+    <!-- Wheel -->
+  <xacro:include filename="$(find am_description)/urdf/wheel.urdf.xacro" />
+    <!-- camera pack-->
+  <xacro:include filename="$(find unicorn_description)/urdf/stereo_camera_gazebo.urdf.xacro" />
+   <!-- lidar pack-->
+  <xacro:include filename="$(find unicorn_description)/urdf/lidar_gazebo.urdf.xacro" />
   <xacro:property name="M_PI" value="3.1415926535897931" />
-  <!-- Main Body-base -->
-  <xacro:property name="base_x_size" value="0.72" />
+  <xacro:property name="M_PI2" value="1.57079632679" />
+  <!-- base -->
+    <xacro:property name="base_x_size" value="0.72" />
   <xacro:property name="base_y_size" value="0.55" />
   <xacro:property name="base_z_size" value="0.6" />
-  <xacro:property name="base_mass" value="15" /> <!-- 21.446 in kg-->
-  <!--Inertial macros for the box and cylinder. Units are kg*m^2-->
-  <xacro:macro name="box_inertia" params="m x y z">
-    <inertia  ixx="${m*(y*y+z*z)/12}" ixy = "0" ixz = "0"
-              iyy="${m*(x*x+z*z)/12}" iyz = "0"
-              izz="${m*(x*x+z*z)/12}" />
-  </xacro:macro>
-  <!-- LMS111 -->
-  <xacro:arg name="laser_xyz" default="0.0 0.0 0.260" />
-  <xacro:arg name="laser_rpy" default="0.0 0.0 ${M_PI}" />
-  <xacro:include filename="$(find lms1xx)/urdf/sick_lms1xx.urdf.xacro" />
-  <!-- Ultrasonic sensor -->
-  <xacro:arg name="ultrasonic_xyz" default="-0.3 0 0.2" />
-  <xacro:arg name="ultrasonic_rpy" default="0 0 ${M_PI}" />
-  <xacro:include filename="$(find unicorn_description)/urdf/ultrasonic_sensor.urdf.xacro" />
-  <!-- Camera -->
-  <xacro:arg name="camera_enabled" default="false" />
-  <xacro:arg name="camera_xyz" default="1.0 1.0 1.0" />
-  <xacro:arg name="camera_rpy" default="0.0 0.0 0.0" />
-  <xacro:include filename="$(find unicorn_description)/urdf/stereo_camera.urdf.xacro" />
-  <!-- Wheel -->
-  <xacro:include filename="$(find am_description)/urdf/wheel.urdf.xacro" />
-  <!-- Swivel wheel -->
-  <xacro:include filename="$(find am_description)/urdf/swivel_wheel.urdf.xacro" />
-  <!-- Materials -->
-  <xacro:include filename="$(find am_description)/urdf/materials.urdf.xacro" />
+  <xacro:property name="base_mass" value="21.446" /> <!-- 21.446 in kg-->
+  <!-- Front Lidar -->
+  <xacro:arg name="laser_xyz" default="-0.0214 -0.0049 0.465" />
+  <xacro:arg name="laser_rpy" default="0 0 0" />
+  <xacro:arg name="frontlidar_meshfile" default="package://unicorn_description/meshes/base_laser.STL" />
+<!-- Rear Lidar  -->
+  <xacro:arg name="rear_laser_xyz" default="-0.42145 0.00645 0.28652" />
+  <xacro:arg name="rear_laser_rpy" default="0 0 ${M_PI}" />
+  <xacro:arg name="rearlidar_meshfile" default="package://unicorn_description/meshes/rear_lidar.STL" />
+  <xacro:arg name="camera_enabled" default="true" />
+  <!-- Zed Camera -->
+  <xacro:arg name="zed_xyz" default="0.03112 -0.00552 0.36395" />
+  <xacro:arg name="zed_rpy" default="0 0 0" />
+  <xacro:arg name="zed_meshfile" default="package://unicorn_description/meshes/zed_link.STL" />
+  <!-- Real Sense -->
+  <xacro:arg name="real_rgb_xyz" default="-0.4065 -0.03882 0.33658" />
+  <xacro:arg name="real_depth_xyz" default="-0.4065 -0.00518 0.33658" />
+  <xacro:arg name="real_rpy" default="0 0 ${M_PI}" />
+  <xacro:arg name="realsense_meshfile" default="package://unicorn_description/meshes/real_sense.STL" />
   <link
     name="chassis_link">
     <inertial>
       <origin
-        xyz="0.17 0 -0.10"
+        xyz="0 0 0"
         rpy="0 0 0" />
       <mass
-        value="${base_mass}" />
-      <box_inertia  m="${5*base_mass}" x="${base_x_size}" y="${base_y_size}" z="${base_z_size}"/>
+        value="15" />
+      <inertia
+        ixx="0.0975408765842248"
+        ixy="0.00235153300726134"
+        ixz="1"
+        iyy="0.162888218399927"
+        iyz="1"
+        izz="0.253342051396573" />
     </inertial>
     <visual>
       <origin
-        xyz="-0.17 0 0"
+        xyz="0 0 0"
         rpy="0 0 0" />
       <geometry>
         <mesh
-          filename="package://unicorn_description/meshes/base_link.STL" />
+          filename="package://unicorn_description/meshes/chassis_link.STL" />
+      </geometry>
+      <material
+        name="">
+        <color
+          rgba="0.792156862745098 0.819607843137255 0.933333333333333 1" />
+      </material>
+    </visual>
+    <collision>
+      <origin
+        xyz="0 0 0"
+        rpy="0 0 0" />
+      <geometry>
+        <mesh
+          filename="package://unicorn_description/meshes/chassis_link.STL" />
+      </geometry>
+    </collision>
+  </link>
+    <!-- Main Body-base
+  <link
+    name="base_link_gazebo">
+    <inertial>
+      <origin
+        xyz="0 0 0"
+        rpy="0 0 0" />
+      <mass
+        value="0.01" />
+      <box_inertia  m="${5}" x="${base_x_size}" y="${base_y_size}" z="${base_z_size}"/>
+    </inertial>
+    <visual>
+      <origin
+        xyz="0 0 0"
+        rpy="0 0 0" />
+      <geometry>
+        <box size="0.01 0.01 0.01"/>
       </geometry>
       <material
@@ -61,55 +104,14 @@
     <collision>
       <origin
-        xyz="-0.17 0 0.08"
-        rpy="0 0 0" />
-      <geometry>
-        <!-- <mesh
-          filename="package://unicorn_description/meshes/base_link.STL" /> -->
-          <box size="0.65 0.5 0.2"/>
-      </geometry>
-      <!-- <surface>
+        xyz="0 0 0"
+        rpy="0 0 0" />
+      <geometry>
+          <box size="0.01 0.01 0.01"/>
+      </geometry>
+       <surface>
          <friction>
            <ode><mu>0</mu><mu2>0</mu2></ode>
          </friction>
-      </surface> -->
-    </collision>
-  </link>
-  <link
-    name="base_link_gazebo">
-    <inertial>
-      <origin
-        xyz="0.17 0 0"
-        rpy="0 0 0" />
-      <mass
-        value="0.01" />
-      <box_inertia  m="${5*0.01}" x="${base_x_size}" y="${base_y_size}" z="${base_z_size}"/>
-    </inertial>
-    <visual>
-      <origin
-        xyz="0 0 0"
-        rpy="0 0 0" />
-      <geometry>
-        <box size="0.01 0.01 0.01"/>
-      </geometry>
-      <material
-        name="">
-        <color
-          rgba="0.79216 0.81961 0.93333 1" />
-      </material>
-    </visual>
-    <collision>
-      <origin
-        xyz="0 0 0"
-        rpy="0 0 0" />
-      <geometry>
-        <!-- <mesh
-          filename="package://unicorn_description/meshes/base_link.STL" /> -->
-          <box size="0.01 0.01 0.01"/>
-      </geometry>
-      <!-- <surface>
-         <friction>
-           <ode><mu>0</mu><mu2>0</mu2></ode>
-         </friction>
-      </surface> -->
+      </surface>
     </collision>
   </link>
@@ -122,79 +124,51 @@
     <child link="base_link_gazebo" />
   <origin xyz="0 0.0 0" rpy="0 0 ${M_PI}" />
-  </joint>
-  <wheel fb="back" lr="right" parent="base_link_gazebo" translateY="-0.24" translateX="0.0" translateZ="-0.006" wheel_radius="0.1225" wheel_height="0.032" flip="1"/>
-  <wheel fb="back" lr="left" parent="base_link_gazebo" translateY="0.24" translateX="0.0" translateZ="-0.006" wheel_radius="0.1225" wheel_height="0.032" flip="1"/>
-  <swivel_wheel fb="front" lr="right" parent="base_link_gazebo" translateY="-0.16" translateX="0.355" translateZ="0.03" wheel_radius="0.05" wheel_height="0.05" flip="0"/>
-  <swivel_wheel fb="front" lr="left" parent="base_link_gazebo" translateY="0.16" translateX="0.355" translateZ="0.03" wheel_radius="0.05" wheel_height="0.05" flip="0"/>
-  <!-- LOOP SENSORs -->
-  <!-- <sensorpos name="loop_front_center" parent="base_link_gazebo" translateX="0.38" translateY="0.0" translateZ="-0.04"/>
-  <sensorpos name="loop_front_right" parent="base_link_gazebo" translateX="0.38" translateY="-0.07" translateZ="-0.04"/>
-  <sensorpos name="loop_rear_left" parent="base_link_gazebo" translateX="-0.07" translateY="0.14" translateZ="-0.04"/>
-  <sensorpos name="loop_rear_right" parent="base_link_gazebo" translateX="-0.07" translateY="-0.14" translateZ="-0.04"/> -->
-  <!-- CONFINEMENT SENSORs -->
-  <!-- <sensorpos name="col_front_chassis" parent="base_link_gazebo" translateX="0.55" translateY="0.0" translateZ="0.00"/>
-  <sensorpos name="col_front_left" parent="base_link_gazebo" translateX="0.43" translateY="0.24" translateZ="0.00"/>
-  <sensorpos name="col_front_right" parent="base_link_gazebo" translateX="0.43" translateY="-0.24" translateZ="0.00"/>
-  <sensorpos name="col_rear_left" parent="base_link_gazebo" translateX="-0.10" translateY="0.24" translateZ="0.0"/>
-  <sensorpos name="col_rear_right" parent="base_link_gazebo" translateX="-0.10" translateY="-0.24" translateZ="0.0"/> -->
-  <!-- CUTTING DISC -->
-  <!-- <link name="cutting_disc_center">
-    <visual>
-        <origin xyz="0 0 0" rpy="0 0 0" />
-        <geometry>
-            <cylinder length="0.01" radius="0.11" />
-        </geometry>
-        <material name="Purple" />
-    </visual>
-  </link>
-  <gazebo reference="cutting_disc_center">
-    <turnGravityOff>false</turnGravityOff>
-  </gazebo>
-  <joint name="cutting_disc_center_joint" type="fixed">
-    <parent link="base_link_gazebo"/>
-    <child link="cutting_disc_center" />
-  <origin xyz="0.25 0.0 -0.07" rpy="0 0 0" />
   </joint> -->
-  <!-- Antenna -->
-  <!-- <link name="antenna_center">
-    <visual>
-        <origin xyz="0 0 0" rpy="0 0 0" />
-        <geometry>
-            <cylinder length="0.01" radius="0.05" />
-        </geometry>
-        <material name="Purple" />
-    </visual>
-  </link>
-  <gazebo reference="antenna_center">
-    <turnGravityOff>false</turnGravityOff>
-  </gazebo>
-  <joint name="antenna_center_joint" type="fixed">
-    <parent link="base_link_gazebo"/>
-    <child link="antenna_center" />
-  <origin xyz="0.27 0.0 0.0" rpy="0 0 0" />
-  </joint> -->
-  <!--<sick_lms1xx_mount prefix="base"/>-->
-  <sick_lms1xx frame="base_laser" topic="scan" robot_namespace="$(arg robot_namespace)"/>
+  <!-- driving wheels -->
+  <wheel fb="back" lr="left" parent="chassis_link" translateY="0.24" translateX="0" translateZ="0.122" wheel_radius="0.1225" wheel_height="0.032" flip="1"/>
+  <wheel fb="back" lr="right" parent="chassis_link" translateY="-0.24" translateX="0 " translateZ="0.122" wheel_radius="0.1225" wheel_height="0.032" flip="1"/>
+  <!-- others wheels -->
+  <swivel_wheel fb="front" lr="left" parent="chassis_link" translateY="0.16" translateX="-0.355" translateZ="0.1526" wheel_radius="0.05" wheel_height="0.05" flip="0"/>
+  <swivel_wheel fb="front" lr="right" parent="chassis_link" translateY="-0.16" translateX="-0.355" translateZ="0.1526" wheel_radius="0.05" wheel_height="0.05" flip="0"/>
+ <!-- Front Lidar -->
+  <lidar_gazebo frame="base_laser" topic="scan" sample_size="800" min_angle="-2.35619" max_angle="2.35619" robot_namespace="$(arg robot_namespace)" filename="$(arg frontlidar_meshfile)" />
   <joint name="laser_mount_joint" type="fixed">
     <origin xyz="$(arg laser_xyz)" rpy="$(arg laser_rpy)" />
-    <parent link="base_link_gazebo" />
+    <parent link="chassis_link" />
     <child link="base_laser" />
   </joint>
-  <!-- Camera -->
+   <!-- Back Lidar -->
+  <lidar_gazebo frame="rear_laser" topic="rearLidar/scan" sample_size="11" min_angle="-0.767944871" max_angle="0.767944871" robot_namespace="$(arg robot_namespace)" filename="$(arg rearlidar_meshfile)"/>
+  <joint name="rear_laser_mount_joint" type="fixed">
+    <origin xyz="$(arg rear_laser_xyz)" rpy="$(arg rear_laser_rpy)" />
+    <parent link="chassis_link" />
+    <child link="rear_laser" />
+  </joint>
+  <!-- Zed Camera -->
   <xacro:if value="$(arg camera_enabled)">
-    <stereo_camera frame="camera_left_link" topic="pointcloud" robot_namespace="$(arg robot_namespace)"/>
-    <!-- generate an optical frame http://www.ros.org/reps/rep-0103.html#suffix-frames
-        so that ros and opencv can operate on the camera frame correctly -->
-    <joint name="camera_optical_joint" type="fixed">
-      <!-- these values have to be these values otherwise the gazebo camera image
-          won't be aligned properl  y with the frame it is supposedly originating from -->
-      <origin xyz="$(arg camera_xyz)" rpy="0 0 ${-pi}"/>
-      <parent link="base_link_gazebo"/>
-      <child link="camera_left_link"/>
-    </joint>
-    <joint name="camera_depth_joint" type="fixed">
+    <stereo_camera frame_rgb="zed_camera" frame_depth="zed_depth_joint" cameraName="zed" filename="$(arg zed_meshfile)"  topic="pointcloud" robot_namespace="$(arg robot_namespace)"/>
+    <joint name="zed_camera_rgb_joint" type="fixed">
+      <origin xyz="$(arg zed_xyz)" rpy="$(arg zed_rpy)"/>
+      <parent link="chassis_link"/>
+      <child link="zed_camera"/>
+    </joint>
+    <joint name="zed_camera_depth_joint" type="fixed">
       <origin xyz="0 0 0" rpy="${-pi/2} 0 ${-pi/2}"/>
-      <parent link="camera_left_link"/>
-      <child link="camera_left_depth_link"/>
+      <parent link="zed_camera"/>
+      <child link="zed_depth_joint"/>
+    </joint>
+  </xacro:if>
+  <!-- realsense Camera -->
+  <xacro:if value="$(arg camera_enabled)">
+    <stereo_camera frame_rgb="realsense_camera" frame_depth="realsense_depth_joint" cameraName="realsense" filename="$(arg realsense_meshfile)"  topic="pointcloud" robot_namespace="$(arg robot_namespace)"/>
+    <joint name="realsense_gb_joint" type="fixed">
+      <origin xyz="$(arg real_rgb_xyz)" rpy="$(arg real_rpy)"/>
+      <parent link="chassis_link"/>
+      <child link="realsense_camera"/>
+    </joint>
+    <joint name="realsense_depth_joint" type="fixed">
+      <origin xyz="$(arg real_depth_xyz)" rpy="${-pi/2} 0 ${-pi/2}"/>
+      <parent link="realsense_camera"/>
+      <child link="realsense_depth_joint"/>
     </joint>
   </xacro:if>
@@ -213,65 +187,5 @@
     </plugin>
   </gazebo>
-  <!-- Ultrasonic sensors -->
-  <ultrasonic_sensor frame="base_ultrasonic_fr" topic="fr" robot_namespace="$(arg robot_namespace)"/>
-  <joint name="ultrasonic_mount_joint_fr" type="fixed">
-    <origin xyz="-0.2 0.2 0.0" rpy="0 0 ${M_PI + M_PI/4}"/>
-    <parent link="base_link_gazebo"/>
-    <child link="base_ultrasonic_fr" />
-  </joint>
-  <ultrasonic_sensor frame="base_ultrasonic_fm" topic="fm" robot_namespace="$(arg robot_namespace)"/>
-  <joint name="ultrasonic_mount_joint_fm" type="fixed">
-    <origin xyz="-0.2 0.0 0.0" rpy="0 0 ${M_PI}"/>
-    <parent link="base_link_gazebo"/>
-    <child link="base_ultrasonic_fm" />
-  </joint>
-  <ultrasonic_sensor frame="base_ultrasonic_fl" topic="fl" robot_namespace="$(arg robot_namespace)"/>
-  <joint name="ultrasonic_mount_joint_fl" type="fixed">
-    <origin xyz="-0.2 -0.2 0.0" rpy="0 0 ${M_PI - M_PI/4}"/>
-    <parent link="base_link_gazebo"/>
-    <child link="base_ultrasonic_fl" />
-  </joint>
-  <ultrasonic_sensor frame="base_ultrasonic_r" topic="r" robot_namespace="$(arg robot_namespace)"/>
-  <joint name="ultrasonic_mount_joint_r" type="fixed">
-    <origin xyz="0.4 0.25 0.0" rpy="0 -${M_PI/64} ${3*M_PI/4}"/>
-    <parent link="base_link_gazebo"/>
-    <child link="base_ultrasonic_r" />
-  </joint>
-  <ultrasonic_sensor frame="base_ultrasonic_l" topic="l" robot_namespace="$(arg robot_namespace)"/>
-  <joint name="ultrasonic_mount_joint_l" type="fixed">
-    <origin xyz="0.4 -0.25 0.0" rpy="0 -${M_PI/64} -${3*M_PI/4}"/>
-    <parent link="base_link_gazebo"/>
-    <child link="base_ultrasonic_l" />
-  </joint>
-  <ultrasonic_sensor frame="base_ultrasonic_rm" topic="rm" robot_namespace="$(arg robot_namespace)"/>
-  <joint name="ultrasonic_mount_joint_rm" type="fixed">
-    <origin xyz="0.15 0.25 0.0" rpy="0 -${M_PI/64} ${M_PI/4}"/>
-    <parent link="base_link_gazebo"/>
-    <child link="base_ultrasonic_rm" />
-  </joint>
-  <ultrasonic_sensor frame="base_ultrasonic_lm" topic="lm" robot_namespace="$(arg robot_namespace)"/>
-  <joint name="ultrasonic_mount_joint_lm" type="fixed">
-    <origin xyz="0.15 -0.25 0.0" rpy="0 -${M_PI/64} -${M_PI/4}"/>
-    <parent link="base_link_gazebo"/>
-    <child link="base_ultrasonic_lm"/>
-  </joint>
-  <ultrasonic_sensor frame="base_ultrasonic_br" topic="br" robot_namespace="$(arg robot_namespace)"/>
-  <joint name="ultrasonic_mount_joint_br" type="fixed">
-    <origin xyz="0.5 0.2 0.0" rpy="0 -${M_PI/64} -${M_PI/4}"/>
-    <parent link="base_link_gazebo"/>
-    <child link="base_ultrasonic_br" />
-  </joint>
-  <ultrasonic_sensor frame="base_ultrasonic_bm" topic="bm" robot_namespace="$(arg robot_namespace)"/>
-  <joint name="ultrasonic_mount_joint_bm" type="fixed">
-    <origin xyz="0.5 0.0 0.0" rpy="0 -${M_PI/64} 0"/>
-    <parent link="base_link_gazebo"/>
-    <child link="base_ultrasonic_bm" />
-  </joint>
-  <ultrasonic_sensor frame="base_ultrasonic_bl" topic="bl" robot_namespace="$(arg robot_namespace)"/>
-  <joint name="ultrasonic_mount_joint_bl" type="fixed">
-    <origin xyz="0.5 -0.2 0.0" rpy="0 -${M_PI/64} ${M_PI/4}"/>
-    <parent link="base_link_gazebo"/>
-    <child link="base_ultrasonic_bl" />
-  </joint>
+  <!-- Problable need this stuff -->
   <!-- GAZEBO STUFF -->
   <gazebo>
@@ -286,5 +200,5 @@
       <commandTopic>cmd_vel</commandTopic>
       <odometryTopic>odom</odometryTopic>
-      <odometryFrame>odom_gazebo_dont_use</odometryFrame>
+      <odometryFrame>odom_gazebo</odometryFrame>
       <robotBaseFrame>chassis_link</robotBaseFrame>
       <publishWheelTF>false</publishWheelTF>
@@ -319,3 +233,20 @@
   </plugin>
   </gazebo>
+ <!--
+    <gazebo reference="chassis_link">
+    <sensor name="automower_sensor" type="contact">
+      <always_on>true</always_on>
+      <update_rate>50</update_rate>
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
File: unicorn_description/urdf/unicorn_target.urdf.xacro (robot description, xacro)
@@ -35,5 +35,5 @@
   <xacro:include filename="$(find am_description)/urdf/wheel.urdf.xacro" />
   <!-- Swivel wheel -->
-  <xacro:include filename="$(find am_description)/urdf/swivel_wheel.urdf.xacro" />
+  <!-- <xacro:include filename="$(find am_description)/urdf/swivel_wheel.urdf.xacro" /> -->
   <!-- Materials -->
   <xacro:include filename="$(find am_description)/urdf/materials.urdf.xacro" />
