Commit message: Updated unicorn model and added lift in simulation, a controller for lift is still needed

File: unicorn_description/urdf/stereo_camera_gazebo.urdf.xacro (robot description, xacro)
@@ -1,17 +1,6 @@
 <?xml version="1.0"?>
 <robot xmlns:xacro="http://ros.org/wiki/xacro">
-  <xacro:macro name="stereo_camera" params="frame_rgb frame_depth topic:=pointcloud simulation:=true filename cameraName:=camera robot_namespace:=/" >
-  <xacro:arg name="sim" default="${simulation}" />
-    <link name="${frame_rgb}">
-     <visual>
-        <origin xyz="0 0 0" rpy="0 0 0"/>
-        <geometry>
-            <mesh filename="${filename}" />
-        </geometry>
-      </visual>
-    </link>
+  <xacro:macro name="stereo_camera" params="frame_rgb frame_depth topic:=pointcloud cameraName:=camera robot_namespace:=/" >
 <!-- Gazebo simulation -->
-    <link name="${frame_depth}"></link>
-    <xacro:if value="$(arg sim)">
       <!-- camera -->
       <gazebo reference="${frame_rgb}">
@@ -57,5 +46,4 @@
         </sensor>
       </gazebo>
-    </xacro:if>
   </xacro:macro>
 </robot>

File: unicorn_description/urdf/unicorn_sim.urdf.xacro (robot description, xacro)
@@ -42,5 +42,5 @@
   <xacro:arg name="zed_meshfile" default="package://unicorn_description/meshes/zed_link.STL" />
   <!-- Real Sense -->
-  <xacro:arg name="real_base" default="-0.4065 ${-0.03882+0.015} 0.33658" />
+  <xacro:arg name="real_base" default="${-0.4065-0.025} ${-0.03882+0.015} 0.33658" />
   <xacro:arg name="real_rgb_xyz" default="0 0.015 0" />
   <xacro:arg name="real_depth_xyz" default="0 0 0" />
@@ -49,4 +49,5 @@
   <xacro:arg name="real_depth_rpy" default="${-M_PI2} 0 ${-M_PI2}" />
   <xacro:arg name="realsense_meshfile" default="package://unicorn_description/meshes/real_sense.STL" />
+  <!-- Lift -->
  <!-- Main Body-base -->
   <link
@@ -105,5 +106,5 @@
         rpy="0 0 0" />
       <mass
-        value="4" />
+        value="10" />
       <inertia
         ixx="1"
@@ -128,4 +129,12 @@
       </material>
     </visual>
+      <surface>
+        <friction>
+          <ode>
+            <mu>0.5</mu>
+            <mu2>0.5</mu2>
+          </ode>
+        </friction>
+      </surface>
     <collision>
       <origin
@@ -152,4 +161,159 @@
     <joint_properties damping="1" friction="0.5" />
   </joint>
+  <link
+    name="lift_horizontal_link">
+    <visual>
+      <origin
+        xyz="0 0 0"
+        rpy="0 0 0" />
+      <geometry>
+        <mesh
+          filename="package://unicorn_description/meshes/lift_horizontal_link.STL" />
+      </geometry>
+      <material
+        name="">
+        <color
+          rgba="0.898039215686275 0.917647058823529 0.929411764705882 1" />
+      </material>
+    </visual>
+      <surface>
+        <friction>
+          <ode>
+            <mu>0.5</mu>
+            <mu2>0.5</mu2>
+          </ode>
+        </friction>
+      </surface>
+    <collision>
+      <origin
+        xyz="0 0 0"
+        rpy="0 0 0" />
+      <geometry>
+        <mesh
+          filename="package://unicorn_description/meshes/lift_horizontal_link.STL" />
+      </geometry>
+    </collision>
+    <inertial>
+      <origin
+        xyz="0 0 0"
+        rpy="0 0 0" />
+      <mass
+        value="1.50791731426345" />
+      <inertia
+        ixx="0.00998369504134607"
+        ixy="1.05918049885466E-06"
+        ixz="-3.20101525315815E-06"
+        iyy="0.0148024039374132"
+        iyz="1.02762580499191E-05"
+        izz="0.0197484509547163" />
+    </inertial>
+  </link>
+  <joint name="lift_horizontal_joint" type="prismatic">
+    <parent  link="lift_link" />
+    <child  link="lift_horizontal_link" />
+    <origin xyz="0.05 0 0.137" rpy="${M_PI2} 0 ${-M_PI2}" />
+    <axis xyz="0 0.0024714 -1" rpy="0 0 0"  />
+    <limit lower="0.17" upper="0" effort="100" velocity="100" />
+    <joint_properties damping="1000" friction="0.5" />
+  </joint>
+  <gazebo reference="lift_horizontal_joint">
+      <mu1 value="10000.0" />
+      <mu2 value="10000.0" />
+      <kp value="100000.0" />
+      <kd value="10000.0" />
+      <dampingFactor value="0.5" />
+      <fdir1 value="1 0 0" />
+      <material>Gazebo/Black</material>
+      <turnGravityOff>false</turnGravityOff>
+  </gazebo>
+  <transmission name="lift_horizontal_joint_trans">
+      <type>transmission_interface/SimpleTransmission</type>
+      <joint name="lift_horizontal_joint">
+        <hardwareInterface>hardware_interface/EffortJointInterface</hardwareInterface>
+      </joint>
+      <actuator name="lift_horizontal_joint_motor">
+        <hardwareInterface>hardware_interface/EffortJointInterface</hardwareInterface>
+        <mechanicalReduction>5</mechanicalReduction>
+      </actuator>
+  </transmission>
+  <link
+    name="lift_vertical_link">
+    <inertial>
+      <origin
+        xyz="-0.0046764 0.62992 -0.22573"
+        rpy="0 0 0" />
+      <mass
+        value="0.61742" />
+      <inertia
+        ixx="0.00029455"
+        ixy="9.8754E-10"
+        ixz="2.0681E-19"
+        iyy="0.00411"
+        iyz="3.0422E-05"
+        izz="0.0043679" />
+    </inertial>
+    <visual>
+      <origin
+        xyz="0 0 0"
+        rpy="0 0 0" />
+      <geometry>
+        <mesh
+          filename="package://unicorn_description/meshes/lift_vertical_link.STL" />
+      </geometry>
+      <material
+        name="">
+        <color
+          rgba="1 0.69412 0.27843 1" />
+      </material>
+    </visual>
+    <collision>
+      <origin
+        xyz="0 0 0"
+        rpy="0 0 0" />
+      <geometry>
+        <mesh
+          filename="package://unicorn_description/meshes/lift_vertical_link.STL" />
+      </geometry>
+    </collision>
+  </link>
+  <joint
+    name="lift_vertical_joint"
+    type="prismatic">
+    <origin
+      xyz="0 -0.16 0"
+      rpy="0 0 0" />
+    <parent
+      link="lift_horizontal_link" />
+    <child
+      link="lift_vertical_link" />
+    <axis
+      xyz="0 1 0" />
+    <limit
+      lower="0"
+      upper="0.16"
+      effort="100"
+      velocity="0.4" />
+      <joint_properties damping="10" friction="0.5" />
+  </joint>
+  <gazebo reference="lift_vertical_joint">
+      <mu1 value="10000.0" />
+      <mu2 value="10000.0" />
+      <kp value="100000.0" />
+      <kd value="10000.0" />
+      <dampingFactor value="0.5" />
+      <fdir1 value="1 0 0" />
+      <material>Gazebo/Black</material>
+      <turnGravityOff>false</turnGravityOff>
+  </gazebo>
+  <transmission name="lift_vertical_joint_trans">
+      <type>transmission_interface/SimpleTransmission</type>
+      <joint name="lift_vertical_joint">
+        <hardwareInterface>hardware_interface/EffortJointInterface</hardwareInterface>
+      </joint>
+      <actuator name="lift_vertical_joint_motor">
+        <hardwareInterface>hardware_interface/EffortJointInterface</hardwareInterface>
+        <mechanicalReduction>5</mechanicalReduction>
+      </actuator>
+  </transmission>
   <wheel fb="back" lr="left" parent="lift_link"  translateY="0.24" translateX="0" translateZ="0.1225" wheel_radius="0.1225" wheel_height="0.032" flip="1"/>
   <wheel fb="back" lr="right" parent="lift_link" translateY="-0.24" translateX="0 " translateZ="0.1225" wheel_radius="0.1225" wheel_height="0.032" flip="1"/>
@@ -172,5 +336,14 @@
   </joint>
   <!-- Zed Camera -->
-    <stereo_camera frame_rgb="zed_camera" frame_depth="zed_depth" cameraName="zed" simulation="$(arg sim)" filename="$(arg zed_meshfile)"  topic="pointcloud" robot_namespace="$(arg robot_namespace)"/>
+    <stereo_camera frame_rgb="zed_camera" frame_depth="zed_depth" cameraName="zed"  topic="pointcloud" robot_namespace="$(arg robot_namespace)"/>
+  <link name="zed_camera">
+    <visual>
+      <origin xyz="0 0 0" rpy="0 0 0"/>
+      <geometry>
+          <mesh filename="$(arg zed_meshfile)"/>
+      </geometry>
+    </visual>
+  </link>
+  <link name="zed_depth"></link>
     <joint name="zed_camera_rgb_joint" type="fixed">
       <origin xyz="$(arg zed_xyz)" rpy="$(arg zed_rpy)"/>
@@ -187,4 +360,10 @@
   <link
     name="realsense_link">
+      <visual>
+      <origin xyz="0 0 0" rpy="0 0 0"/>
+      <geometry>
+          <mesh filename="$(arg realsense_meshfile)" />
+      </geometry>
+    </visual>
   </link>
   <joint name="realsense_joint" type="fixed">
@@ -194,21 +373,7 @@
   </joint>
 <xacro:if value="$(arg sim)">
-  <link
-    name="realsense_model_dummy_link">
-    <visual>
-        <origin xyz="0 0 0" rpy="0 0 0"/>
-        <geometry>
-            <mesh filename="$(arg realsense_meshfile)" />
-        </geometry>
-      </visual>
-  </link>
-  <joint name="realsense_model_joint" type="fixed">
-    <origin xyz="$(arg real_rgb_xyz)" rpy="0 0 0"/>
-    <parent link="realsense_link"/>
-    <child link="realsense_model_dummy_link"/>
-  </joint>
-</xacro:if>
-<xacro:if value="$(arg sim)">
-  <stereo_camera frame_rgb="realsense_color_frame" frame_depth="realsense_depth_frame" cameraName="realsense" simulation="$(arg sim)" filename="$(arg realsense_meshfile)"  topic="pointcloud" robot_namespace="$(arg robot_namespace)"/>
+  <stereo_camera frame_rgb="realsense_color_frame" frame_depth="realsense_depth_frame" cameraName="realsense" topic="pointcloud" robot_namespace="$(arg robot_namespace)"/>
+  <link name="realsense_color_frame"> </link>
+  <link name="realsense_depth_frame"></link>
   <link
     name="realsense_depth_optical_frame">

File: unicorn_description/urdf/unicorn_target.urdf.xacro (robot description, xacro)
@@ -212,5 +212,14 @@
   </joint>
   <!-- Zed Camera -->
-    <stereo_camera frame_rgb="zed_camera" frame_depth="zed_depth_joint" cameraName="zed" simulation="$(arg sim)" filename="$(arg zed_meshfile)"  topic="pointcloud" robot_namespace="$(arg robot_namespace)"/>
+    <stereo_camera frame_rgb="zed_camera" frame_depth="zed_depth" cameraName="zed"  topic="pointcloud" robot_namespace="$(arg robot_namespace)"/>
+  <link name="zed_camera">
+    <visual>
+      <origin xyz="0 0 0" rpy="0 0 0"/>
+      <geometry>
+          <mesh filename="$(arg zed_meshfile)"/>
+      </geometry>
+    </visual>
+  </link>
+  <link name="zed_depth"></link>
     <joint name="zed_camera_rgb_joint" type="fixed">
       <origin xyz="$(arg zed_xyz)" rpy="$(arg zed_rpy)"/>
@@ -221,9 +230,16 @@
       <origin xyz="0 0 0" rpy="${-pi/2} 0 ${-pi/2}"/>
       <parent link="zed_camera"/>
-      <child link="zed_depth_joint"/>
+      <child link="zed_depth"/>
     </joint>
   <!-- realsense Camera -->
+<!-- Links only needed in simulation, created by realsense software otherwise-->
   <link
     name="realsense_link">
+      <visual>
+      <origin xyz="0 0 0" rpy="0 0 0"/>
+      <geometry>
+          <mesh filename="$(arg realsense_meshfile)" />
+      </geometry>
+    </visual>
   </link>
   <joint name="realsense_joint" type="fixed">
@@ -233,22 +249,7 @@
   </joint>
 <xacro:if value="$(arg sim)">
-  <link
-    name="realsense_model_dummy_link">
-    <visual>
-        <origin xyz="0 0 0" rpy="0 0 0"/>
-        <geometry>
-            <mesh filename="$(arg realsense_meshfile)" />
-        </geometry>
-      </visual>
-  </link>
-  <joint name="realsense_model_joint" type="fixed">
-    <origin xyz="$(arg real_rgb_xyz)" rpy="0 0 0"/>
-    <parent link="realsense_link"/>
-    <child link="realsense_model_dummy_link"/>
-  </joint>
-</xacro:if>
-  <!-- Links only needed in simulation, created by realsense software otherwise-->
-<xacro:if value="$(arg sim)">
-  <stereo_camera frame_rgb="realsense_color_frame" frame_depth="realsense_depth_frame" cameraName="realsense" simulation="$(arg sim)" filename="$(arg realsense_meshfile)"  topic="pointcloud" robot_namespace="$(arg robot_namespace)"/>
+  <stereo_camera frame_rgb="realsense_color_frame" frame_depth="realsense_depth_frame" cameraName="realsense" topic="pointcloud" robot_namespace="$(arg robot_namespace)"/>
+  <link name="realsense_color_frame"> </link>
+  <link name="realsense_depth_frame"></link>
   <link
     name="realsense_depth_optical_frame">

File: unicorn_description/urdf/unicorn_target_backwards.urdf.xacro (robot description, xacro)
@@ -176,10 +176,18 @@
   </joint>
   <!-- Zed Camera -->
-    <stereo_camera frame_rgb="zed_camera" frame_depth="zed_depth" cameraName="zed" simulation="$(arg sim)" filename="$(arg zed_meshfile)"  topic="pointcloud" robot_namespace="$(arg robot_namespace)"/>
+    <stereo_camera frame_rgb="zed_camera" frame_depth="zed_depth" cameraName="zed"  topic="pointcloud" robot_namespace="$(arg robot_namespace)"/>
+  <link name="zed_camera">
+    <visual>
+      <origin xyz="0 0 0" rpy="0 0 0"/>
+      <geometry>
+          <mesh filename="$(arg zed_meshfile)"/>
+      </geometry>
+    </visual>
+  </link>
+  <link name="zed_depth"></link>
     <joint name="zed_camera_rgb_joint" type="fixed">
       <origin xyz="$(arg zed_xyz)" rpy="$(arg zed_rpy)"/>
       <parent link="chassis_link"/>
       <child link="zed_camera"/>
-      <joint_properties damping="1" friction="0.5" />
     </joint>
     <joint name="zed_camera_depth_joint" type="fixed">
@@ -187,9 +195,15 @@
       <parent link="zed_camera"/>
       <child link="zed_depth"/>
-      <joint_properties damping="1" friction="0.5" />
     </joint>
   <!-- realsense Camera -->
+<!-- Links only needed in simulation, created by realsense software otherwise-->
   <link
     name="realsense_link">
+      <visual>
+      <origin xyz="0 0 0" rpy="0 0 0"/>
+      <geometry>
+          <mesh filename="$(arg realsense_meshfile)" />
+      </geometry>
+    </visual>
   </link>
   <joint name="realsense_joint" type="fixed">
@@ -199,22 +213,7 @@
   </joint>
 <xacro:if value="$(arg sim)">
-  <link
-    name="realsense_model_dummy_link">
-    <visual>
-        <origin xyz="0 0 0" rpy="0 0 0"/>
-        <geometry>
-            <mesh filename="$(arg realsense_meshfile)" />
-        </geometry>
-      </visual>
-  </link>
-  <joint name="realsense_model_joint" type="fixed">
-    <origin xyz="$(arg real_rgb_xyz)" rpy="0 0 0"/>
-    <parent link="realsense_link"/>
-    <child link="realsense_model_dummy_link"/>
-  </joint>
-</xacro:if>
-  <!-- Links only needed in simulation, created by realsense software otherwise-->
-<xacro:if value="$(arg sim)">
-  <stereo_camera frame_rgb="realsense_color_frame" frame_depth="realsense_depth_frame" cameraName="realsense" simulation="$(arg sim)" filename="$(arg realsense_meshfile)"  topic="pointcloud" robot_namespace="$(arg robot_namespace)"/>
+  <stereo_camera frame_rgb="realsense_color_frame" frame_depth="realsense_depth_frame" cameraName="realsense" topic="pointcloud" robot_namespace="$(arg robot_namespace)"/>
+  <link name="realsense_color_frame"> </link>
+  <link name="realsense_depth_frame"></link>
   <link
     name="realsense_depth_optical_frame">
