Commit message: update inertia

File: unicorn_description/urdf/unicorn_sim.urdf.xacro (robot description, xacro)
@@ -78,5 +78,5 @@
     </collision>
   </link>
-    <!-- Main Body-base
+    <!-- Main Body-base -->
   <link
     name="base_link_gazebo">
@@ -94,5 +94,5 @@
         rpy="0 0 0" />
       <geometry>
-        <box size="0.01 0.01 0.01"/>
+        <box size="0.1 0.1 0.1"/>
       </geometry>
       <material
@@ -124,8 +124,8 @@
     <child link="base_link_gazebo" />
   <origin xyz="0 0.0 0" rpy="0 0 ${M_PI}" />
-  </joint> -->
+  </joint>
   <!-- driving wheels -->
-  <wheel fb="back" lr="left" parent="chassis_link" translateY="0.24" translateX="0" translateZ="0.122" wheel_radius="0.1225" wheel_height="0.032" flip="1"/>
-  <wheel fb="back" lr="right" parent="chassis_link" translateY="-0.24" translateX="0 " translateZ="0.122" wheel_radius="0.1225" wheel_height="0.032" flip="1"/>
+  <wheel fb="back" lr="left" parent="base_link_gazebo" translateY="0.24" translateX="0" translateZ="0.122" wheel_radius="0.1225" wheel_height="0.032" flip="1"/>
+  <wheel fb="back" lr="right" parent="base_link_gazebo" translateY="-0.24" translateX="0 " translateZ="0.122" wheel_radius="0.1225" wheel_height="0.032" flip="1"/>
   <!-- others wheels -->
   <swivel_wheel fb="front" lr="left" parent="chassis_link" translateY="0.16" translateX="-0.355" translateZ="0.1526" wheel_radius="0.05" wheel_height="0.05" flip="0"/>
@@ -173,5 +173,5 @@
     </joint>
   </xacro:if>
-  <!-- GPS -->
+  <!-- GPS
   <gazebo>
     <plugin name="novatel_gps_sim" filename="libhector_gazebo_ros_gps.so">
@@ -181,10 +181,10 @@
       <topicName>gps</topicName>
       <velocityTopicName>gps_velocity</velocityTopicName>
-      <drift>5.0 5.0 5.0</drift>
-      <gaussianNoise>0.1 0.1 0.1</gaussianNoise>
+      <drift>0 0 0</drift>
+      <gaussianNoise>0 0 0</gaussianNoise>
       <velocityDrift>0 0 0</velocityDrift>
-      <velocityGaussianNoise>0.1 0.1 0.1</velocityGaussianNoise>
+      <velocityGaussianNoise>0 0 0</velocityGaussianNoise>
     </plugin>
-  </gazebo>
+  </gazebo>-->
   <!-- Problable need this stuff -->
   <!-- GAZEBO STUFF -->
@@ -233,20 +233,3 @@
   </plugin>
   </gazebo>
- <!--
-    <gazebo reference="chassis_link">
-    <sensor name="automower_sensor" type="contact">
-      <always_on>true</always_on>
-      <update_rate>50</update_rate>
-      <contact>
-        <collision>base_link_collision</collision>
-      </contact>
-      <plugin name="automower_sensors_plugin" filename="libam_gazebo_sensors.so">
-        <always_on>true</always_on>
-        <update_rate>20</update_rate>
-        <bumperTopicName>sensor_status</bumperTopicName>
-        <loopTopicName>loop</loopTopicName>
-        <loopOutsideSensors>15</loopOutsideSensors>
-      </plugin>
-    </sensor>
-  </gazebo>-->
 </robot>

Commit message: update urdf

File: unicorn_description/urdf/unicorn_sim.urdf.xacro (robot description, xacro)
@@ -25,5 +25,5 @@
   <xacro:arg name="frontlidar_meshfile" default="package://unicorn_description/meshes/base_laser.STL" />
 <!-- Rear Lidar  -->
-  <xacro:arg name="rear_laser_xyz" default="-0.42145 0.00645 0.28652" />
+  <xacro:arg name="rear_laser_xyz" default="-0.42145 -0.00645 0.28652" />
   <xacro:arg name="rear_laser_rpy" default="0 0 ${M_PI}" />
   <xacro:arg name="rearlidar_meshfile" default="package://unicorn_description/meshes/rear_lidar.STL" />
@@ -47,10 +47,10 @@
         value="15" />
       <inertia
-        ixx="0.0975408765842248"
-        ixy="0.00235153300726134"
-        ixz="1"
-        iyy="0.162888218399927"
-        iyz="1"
-        izz="0.253342051396573" />
+        ixx="0.5"
+        ixy="0"
+        ixz="0"
+        iyy="0.5"
+        iyz="0"
+        izz="0.5" />
     </inertial>
     <visual>
@@ -78,5 +78,5 @@
     </collision>
   </link>
-    <!-- Main Body-base -->
+    <!-- Main Body-base
   <link
     name="base_link_gazebo">
@@ -124,8 +124,8 @@
     <child link="base_link_gazebo" />
   <origin xyz="0 0.0 0" rpy="0 0 ${M_PI}" />
-  </joint>
+  </joint> -->
   <!-- driving wheels -->
-  <wheel fb="back" lr="left" parent="base_link_gazebo" translateY="0.24" translateX="0" translateZ="0.122" wheel_radius="0.1225" wheel_height="0.032" flip="1"/>
-  <wheel fb="back" lr="right" parent="base_link_gazebo" translateY="-0.24" translateX="0 " translateZ="0.122" wheel_radius="0.1225" wheel_height="0.032" flip="1"/>
+  <wheel fb="back" lr="left" parent="chassis_link" translateY="0.24" translateX="0" translateZ="0.122" wheel_radius="0.1225" wheel_height="0.032" flip="1"/>
+  <wheel fb="back" lr="right" parent="chassis_link" translateY="-0.24" translateX="0 " translateZ="0.122" wheel_radius="0.1225" wheel_height="0.032" flip="1"/>
   <!-- others wheels -->
   <swivel_wheel fb="front" lr="left" parent="chassis_link" translateY="0.16" translateX="-0.355" translateZ="0.1526" wheel_radius="0.05" wheel_height="0.05" flip="0"/>
@@ -173,18 +173,18 @@
     </joint>
   </xacro:if>
-  <!-- GPS
+  <!-- GPS -->
   <gazebo>
     <plugin name="novatel_gps_sim" filename="libhector_gazebo_ros_gps.so">
-      <alwaysOn>1</alwaysOn>
+      <alwaysOn>true</alwaysOn>
       <updateRate>10.0</updateRate>
       <bodyName>chassis_link</bodyName>
       <topicName>gps</topicName>
       <velocityTopicName>gps_velocity</velocityTopicName>
-      <drift>0 0 0</drift>
-      <gaussianNoise>0 0 0</gaussianNoise>
+      <drift>5.0 5.0 5.0</drift>
+      <gaussianNoise>0.1 0.1 0.1</gaussianNoise>
       <velocityDrift>0 0 0</velocityDrift>
-      <velocityGaussianNoise>0 0 0</velocityGaussianNoise>
+      <velocityGaussianNoise>0.1 0.1 0.1</velocityGaussianNoise>
     </plugin>
-  </gazebo>-->
+  </gazebo>
   <!-- Problable need this stuff -->
   <!-- GAZEBO STUFF -->
@@ -199,20 +199,11 @@
       <wheelTorque>100</wheelTorque>
       <commandTopic>cmd_vel</commandTopic>
-      <odometryTopic>odom</odometryTopic>
+      <odometryTopic>wheel/odom</odometryTopic>
       <odometryFrame>odom_gazebo</odometryFrame>
       <robotBaseFrame>chassis_link</robotBaseFrame>
       <publishWheelTF>false</publishWheelTF>
       <publishWheelJointState>false</publishWheelJointState>
-    </plugin>
-    <plugin name="gazebo_ros_control" filename="libgazebo_ros_control.so" />
-    <plugin name="imu_plugin" filename="libhector_gazebo_ros_imu.so">
-    <alwaysOn>true</alwaysOn>
-    <bodyName>chassis_link</bodyName>
-    <topicName>imu</topicName>
-    <serviceName>imu_service</serviceName>
-    <updateRate>100.0</updateRate>
-    <rpyOffsets>0 0 0</rpyOffsets> <!-- deprecated -->
 <!--
-      <gaussianNoise>0.0</gaussianNoise>
+      <gaussianNoise>0.1</gaussianNoise>
       <accelDrift>0.5 0.5 0.5</accelDrift>
       <accelGaussianNoise>0.35 0.35 0.3</accelGaussianNoise>
@@ -220,16 +211,50 @@
       <rateGaussianNoise>0.05 0.05 0.015</rateGaussianNoise>
       <headingDrift>0.1</headingDrift>
-      <headingGaussianNoise>1.00</headingGaussianNoise>
--->
-    <gaussianNoise>0.0</gaussianNoise>  <!-- deprecated -->
-      <accelDrift>0.0 0.0 0.0</accelDrift>
-      <accelGaussianNoise>0.0 0.0 0.0</accelGaussianNoise>
-      <rateDrift>0.0 0.0 0.0</rateDrift>
-      <rateGaussianNoise>0.0 0.0 0.0</rateGaussianNoise>
-      <headingDrift>0.0</headingDrift>
-      <headingGaussianNoise>0.00</headingGaussianNoise>
+      <headingGaussianNoise>1.00</headingGaussianNoise>-->
+    </plugin>
+    <plugin name="gazebo_ros_control" filename="libgazebo_ros_control.so" />
+    <plugin name="imu_plugin" filename="libhector_gazebo_ros_imu.so">
+      <alwaysOn>true</alwaysOn>
+      <bodyName>chassis_link</bodyName>
+      <topicName>zed/imu</topicName>
+      <serviceName>imu_service</serviceName>
+      <updateRate>10.0</updateRate>
+      <rpyOffsets>0 0 0</rpyOffsets> <!-- deprecated -->
+  <!--
+        <gaussianNoise>0.1</gaussianNoise>
+        <accelDrift>0.5 0.5 0.5</accelDrift>
+        <accelGaussianNoise>0.35 0.35 0.3</accelGaussianNoise>
+        <rateDrift>0.1 0.1 0.1</rateDrift>
+        <rateGaussianNoise>0.05 0.05 0.015</rateGaussianNoise>
+        <headingDrift>0.1</headingDrift>
+        <headingGaussianNoise>1.00</headingGaussianNoise>-->
+  <!-- deprecated -->
+      <gaussianNoise>0.0</gaussianNoise>
+        <accelDrift>0.0 0.0 0.0</accelDrift>
+        <accelGaussianNoise>0.0 0.0 0.0</accelGaussianNoise>
+        <rateDrift>0.0 0.0 0.0</rateDrift>
+        <rateGaussianNoise>0.0 0.0 0.0</rateGaussianNoise>
+        <headingDrift>0.0</headingDrift>
+        <headingGaussianNoise>0.00</headingGaussianNoise>
     </plugin>
     <plugin name="am_gazebo_wheelencoder" filename="libam_gazebo_wheelencoder.so">
   </plugin>
   </gazebo>
+ <!--
+    <gazebo reference="chassis_link">
+    <sensor name="automower_sensor" type="contact">
+      <always_on>true</always_on>
+      <update_rate>50</update_rate>
+      <contact>
+        <collision>base_link_collision</collision>
+      </contact>
+      <plugin name="automower_sensors_plugin" filename="libam_gazebo_sensors.so">
+        <always_on>true</always_on>
+        <update_rate>20</update_rate>
+        <bumperTopicName>sensor_status</bumperTopicName>
+        <loopTopicName>loop</loopTopicName>
+        <loopOutsideSensors>15</loopOutsideSensors>
+      </plugin>
+    </sensor>
+  </gazebo>-->
 </robot>

Commit message: Added static frame between map and odom link

File: unicorn_description/urdf/unicorn_sim.urdf.xacro (robot description, xacro)
@@ -9,5 +9,5 @@
   <xacro:include filename="$(find am_description)/urdf/swivel_wheel.urdf.xacro" />
     <!-- Wheel -->
-  <xacro:include filename="$(find am_description)/urdf/wheel.urdf.xacro" />
+  <xacro:include filename="$(find unicorn_description)/urdf/wheel.urdf.xacro" />
     <!-- camera pack-->
   <xacro:include filename="$(find unicorn_description)/urdf/stereo_camera_gazebo.urdf.xacro" />
@@ -16,9 +16,20 @@
   <xacro:property name="M_PI" value="3.1415926535897931" />
   <xacro:property name="M_PI2" value="1.57079632679" />
-  <!-- base -->
+  <!-- base --><!--
     <xacro:property name="base_x_size" value="0.72" />
   <xacro:property name="base_y_size" value="0.55" />
   <xacro:property name="base_z_size" value="0.6" />
-  <xacro:property name="base_mass" value="21.446" /> <!-- 21.446 in kg-->
+  <xacro:property name="base_mass" value="21.446" /> 21.446 in kg-->
+    <!-- Main Body-base -->
+  <xacro:property name="base_x_size" value="0.72" />
+  <xacro:property name="base_y_size" value="0.55" />
+  <xacro:property name="base_z_size" value="0.23" />
+  <xacro:property name="base_mass" value="15" /> <!-- in kg-->
+    <!--Inertial macros for the box and cylinder. Units are kg*m^2-->
+  <xacro:macro name="box_inertia" params="m x y z">
+    <inertia ixx="${m*(y*y+z*z)/12}" ixy="0" ixz="0"
+             iyy="${m*(x*x+z*z)/12}" iyz="0"
+             izz="${m*(x*x+z*z)/12}" />
+  </xacro:macro>
   <!-- Front Lidar -->
   <xacro:arg name="laser_xyz" default="-0.0214 -0.0049 0.465" />
@@ -135,9 +146,9 @@
   </joint>
   <!-- driving wheels -->
-  <wheel fb="back" lr="left" parent="chassis_link" translateY="0.25" translateX="0" translateZ="0.122" wheel_radius="0.122" wheel_height="0.032" flip="1"/>
-  <wheel fb="back" lr="right" parent="chassis_link" translateY="-0.25" translateX="0 " translateZ="0.122" wheel_radius="0.122" wheel_height="0.032" flip="1"/>
+  <wheel fb="back" lr="left" parent="chassis_link" translateY="0.23" translateX="0" translateZ="0.1225" wheel_radius="0.1225" wheel_height="0.032" flip="1"/>
+  <wheel fb="back" lr="right" parent="chassis_link" translateY="-0.23" translateX="0 " translateZ="0.1225" wheel_radius="0.1225" wheel_height="0.032" flip="1"/>
   <!-- others wheels -->
-  <swivel_wheel fb="front" lr="left" parent="chassis_link" translateY="0.16" translateX="-0.355" translateZ="0.1526" wheel_radius="0.05" wheel_height="0.05" flip="0"/>
-  <swivel_wheel fb="front" lr="right" parent="chassis_link" translateY="-0.16" translateX="-0.355" translateZ="0.1526" wheel_radius="0.05" wheel_height="0.05" flip="0"/>
+  <swivel_wheel fb="front" lr="left" parent="chassis_link" translateY="0.16" translateX="-0.355" translateZ="0.1531" wheel_radius="0.05" wheel_height="0.05" flip="0"/>
+  <swivel_wheel fb="front" lr="right" parent="chassis_link" translateY="-0.16" translateX="-0.355" translateZ="0.1531" wheel_radius="0.05" wheel_height="0.05" flip="0"/>
  <!-- Front Lidar -->
   <lidar_gazebo frame="base_laser" topic="frontLidar/scan" simulation="$(arg sim)" sample_size="800" min_angle="-2.35619" max_angle="2.35619" robot_namespace="$(arg robot_namespace)" filename="$(arg frontlidar_meshfile)" />

File: unicorn_description/urdf/unicorn_target.urdf.xacro (robot description, xacro)
@@ -167,5 +167,5 @@
     </joint>
   <!-- realsense Camera -->
-    <stereo_camera frame_rgb="realsense_camera" frame_depth="realsense_depth_joint" cameraName="realsense" simulation="$(arg sim)" filename="$(arg realsense_meshfile)"  topic="pointcloud" robot_namespace="$(arg robot_namespace)"/>
+    <stereo_camera frame_rgb="realsense_camera" frame_depth="realsense_depth" cameraName="realsense" simulation="$(arg sim)" filename="$(arg realsense_meshfile)"  topic="pointcloud" robot_namespace="$(arg robot_namespace)"/>
     <joint name="realsense_gb_joint" type="fixed">
       <origin xyz="$(arg real_rgb_xyz)" rpy="$(arg real_rpy)"/>
@@ -174,7 +174,7 @@
     </joint>
     <joint name="realsense_depth_joint" type="fixed">
-      <origin xyz="$(arg real_depth_xyz)" rpy="${-pi/2} 0 ${-pi/2}"/>
+      <origin xyz="0 0 0" rpy="${-pi/2} 0 ${-pi/2}"/>
       <parent link="realsense_camera"/>
-      <child link="realsense_depth_joint"/>
+      <child link="realsense_depth"/>
     </joint>
 <xacro:if value="$(arg sim)">

File: unicorn_description/urdf/wheel.urdf.xacro (robot description, xacro)
@@ -20,33 +20,52 @@
                params="fb lr parent translateX translateY translateZ wheel_radius wheel_height flip"> <!--fb : front, back ; lr: left, right -->
     <link name="${fb}_${lr}_wheel">
-      <visual>
-        <origin xyz="0 0 0" rpy="${flip*M_PI/2} 0 0" />
-        <geometry>
-          <cylinder length="${wheel_height}" radius="${wheel_radius}" />
-        </geometry>
-        <material name="Black" />
-      </visual>
-      <collision>
-        <origin xyz="0 0 0" rpy="${flip*M_PI/2} 0 0" />
-        <geometry>
-          <cylinder length="${wheel_height}" radius="${wheel_radius}" />
-        </geometry>
-      </collision>
-      <inertial>
-        <mass value="${wheel_mass}" />
-        <!-- <origin xyz="0 0 0" rpy="${flip*M_PI/2} 0 0"/> -->
-        <origin xyz="0 0 0" />
-        <cylinder_inertia m="${wheel_mass}" r="${wheel_radius}" h="${wheel_height}" />
-      </inertial>
+    <visual>
+      <origin
+        xyz="0 0 0"
+        rpy="0 0 0" />
+      <geometry>
+        <mesh
+          filename="package://unicorn_description/meshes/wheel_driver.STL" />
+      </geometry>
+      <material
+        name="">
+        <color
+          rgba="0.752941176470588 0.752941176470588 0.752941176470588 1" />
+      </material>
+    </visual>
+    <collision>
+      <origin
+        xyz="0 0 0"
+        rpy="0 0 0" />
+      <geometry>
+        <mesh
+          filename="package://unicorn_description/meshes/wheel_driver.STL" />
+      </geometry>
+    </collision>
+    <inertial>
+      <origin
+        xyz="-6.0591E-12 -0.012242 1.8648E-11"
+        rpy="0 0 0" />
+      <mass
+        value="1.0564" />
+      <inertia
+        ixx="0.0040937"
+        ixy="3.2935E-14"
+        ixz="-4.4864E-13"
+        iyy="0.008088"
+        iyz="-6.8807E-12"
+        izz="0.0040937" />
+    </inertial>
     </link>
+<!--
     <gazebo reference="${fb}_${lr}_wheel">
       <mu1 value="100.0" />
       <mu2 value="100.0" />
-      <kp value="10000000.0" />
+      <kp value="1000.0" />
       <kd value="1.0" />
       <fdir1 value="1 0 0" />
       <material>Gazebo/Black</material>
       <turnGravityOff>false</turnGravityOff>
-    </gazebo>
+    </gazebo>-->
     <joint name="${fb}_${lr}_wheel_joint" type="continuous">
       <parent link="${parent}" />
