Commit message: updated frame issue

File: unicorn_description/urdf/unicorn_sim.urdf.xacro (robot description, xacro)
@@ -1,6 +1,3 @@
 <?xml version="1.0" encoding="utf-8"?>
-<!-- This URDF was automatically created by SolidWorks to URDF Exporter! Originally created by Stephen Brawner (brawner@gmail.com)
-     Commit Version: 1.6.0-1-g15f4949  Build Version: 1.6.7594.29634
-     For more information, please see http://wiki.ros.org/sw_urdf_exporter -->
 <robot name="unicorn" xmlns:xacro="http://www.ros.org/wiki/xacro">
   <xacro:arg name="robot_namespace" default="/" />
@@ -9,5 +6,5 @@
   <xacro:include filename="$(find am_description)/urdf/swivel_wheel.urdf.xacro" />
     <!-- Wheel -->
-  <xacro:include filename="$(find unicorn_description)/urdf/wheel.urdf.xacro" />
+  <xacro:include filename="$(find am_description)/urdf/wheel.urdf.xacro" />
     <!-- camera pack-->
   <xacro:include filename="$(find unicorn_description)/urdf/stereo_camera_gazebo.urdf.xacro" />
@@ -57,5 +54,5 @@
         rpy="0 0 0" />
       <mass
-        value="15" />
+        value="10" />
       <inertia
         ixx="1"
@@ -87,4 +84,9 @@
         <mesh
           filename="package://unicorn_description/meshes/chassis_link.STL" />
+        <surface>
+         <friction>
+           <ode><mu>0.4</mu><mu2>0.4</mu2></ode>
+         </friction>
+      </surface>
       </geometry>
     </collision>
@@ -145,6 +147,47 @@
     <joint_properties damping="0.0" friction="0.0" />
   </joint>
-  <!-- driving wheels -->
-  <wheel fb="back" lr="left" parent="chassis_link" translateY="0.23" translateX="0" translateZ="0.1225" wheel_radius="0.1225" wheel_height="0.032" flip="1"/>
+<!--
+    <link
+    name="wheel_link">
+    <inertial>
+      <origin
+        xyz="0 0 0"
+        rpy="0 0 0" />
+      <mass
+        value="0.01" />
+      <box_inertia  m="${5*0.01}" x="${base_x_size}" y="${base_y_size}" z="${base_z_size}"/>
+    </inertial>
+    <visual>
+      <origin
+        xyz="0 0 0"
+        rpy="0 0 0" />
+      <geometry>
+        <box size="0.01 0.01 0.01"/>
+      </geometry>
+      <material
+        name="">
+        <color
+          rgba="0.79216 0.81961 0.93333 1" />
+      </material>
+    </visual>
+    <collision>
+      <origin
+        xyz="0 0 0"
+        rpy="0 0 0" />
+      <geometry>
+          <box size="0.01 0.01 0.01"/>
+      </geometry>
+    </collision>
+  </link>
+  <joint name="base_chassis_joint" type="fixed">
+    <parent link="chassis_link"/>
+    <child link="wheel_link" />wheel_link
+  <origin xyz="0 0.0 0" rpy="0 0 ${M_PI}" />
+  </joint>-->
+  <!-- driving wheels
+  <wheel fb="back" lr="left" parent="chassis_link" rotationZ="3.14159" translateY="0.23" translateX="0" translateZ="0.1225" wheel_radius="0.1225" wheel_height="0.032" flip="1"/>
+  <wheel fb="back" lr="right" parent="chassis_link" rotationZ="0" translateY="-0.23" translateX="0 " translateZ="0.1225" wheel_radius="0.1225" wheel_height="0.032" flip="1"/>
+  -->
+  <wheel fb="back" lr="left" parent="chassis_link"  translateY="0.23" translateX="0" translateZ="0.1225" wheel_radius="0.1225" wheel_height="0.032" flip="1"/>
   <wheel fb="back" lr="right" parent="chassis_link" translateY="-0.23" translateX="0 " translateZ="0.1225" wheel_radius="0.1225" wheel_height="0.032" flip="1"/>
   <!-- others wheels -->
@@ -218,6 +261,6 @@
       <wheelTorque>100</wheelTorque>
       <commandTopic>cmd_vel</commandTopic>
-      <odometryTopic>wheelencoder/odom</odometryTopic>
-      <odometryFrame>odom_chassis</odometryFrame>
+      <odometryTopic>wheel_encoder/odom</odometryTopic>
+      <odometryFrame>odom_chassis_dont_use</odometryFrame>
       <robotBaseFrame>chassis_link</robotBaseFrame>
       <publishWheelTF>false</publishWheelTF>
@@ -234,9 +277,9 @@
     <plugin name="imu_plugin" filename="libhector_gazebo_ros_imu.so">
       <alwaysOn>true</alwaysOn>
-      <bodyName>chassis_link</bodyName>
+      <bodyName>zed_camera</bodyName>
       <topicName>zed/imu</topicName>
       <serviceName>imu_service</serviceName>
       <updateRate>100.0</updateRate>
-      <rpyOffsets>0 ${M_PI} 0</rpyOffsets>
+      <rpyOffsets>0 0 0</rpyOffsets>
   <!---->
         <gaussianNoise>0.1</gaussianNoise>
@@ -260,68 +303,4 @@
   </gazebo>
 </xacro:if>
-<xacro:unless value="$(arg sim)">
-  <!-- GAZEBO STUFF for unicorn -->
-  <gazebo>
-    <plugin name="automower_gazebo_controller" filename="libam_gazebo_controller_2wd.so">
-      <alwaysOn>true</alwaysOn>
-      <updateRate>100.0</updateRate>
-      <leftJoint>back_right_wheel_joint</leftJoint>
-      <rightJoint>back_left_wheel_joint</rightJoint>
-      <wheelSeparation>0.4645</wheelSeparation>
-      <wheelDiameter>0.245</wheelDiameter>
-      <wheelTorque>100</wheelTorque>
-      <commandTopic>cmd_vel</commandTopic>
-      <odometryTopic>wheelencoder/odom</odometryTopic>
-      <odometryFrame>odom_gazebo</odometryFrame>
-      <robotBaseFrame>chassis_link_gazebo</robotBaseFrame>
-      <publishWheelTF>false</publishWheelTF>
-      <publishWheelJointState>false</publishWheelJointState>
-    </plugin>
-    <plugin name="gazebo_ros_control" filename="libgazebo_ros_control.so" />
-    <plugin name="imu_plugin" filename="libhector_gazebo_ros_imu.so">
-    <alwaysOn>false</alwaysOn>
-    <bodyName>chassis_link_gazebo</bodyName>
-    <topicName>imu</topicName>
-    <serviceName>imu_service</serviceName>
-    <updateRate>100.0</updateRate>
-    <rpyOffsets>0 0 0</rpyOffsets> <!-- deprecated -->
-<!--
-      <gaussianNoise>0.1</gaussianNoise>
-      <accelDrift>0.5 0.5 0.5</accelDrift>
-      <accelGaussianNoise>0.35 0.35 0.3</accelGaussianNoise>
-      <rateDrift>0.1 0.1 0.1</rateDrift>
-      <rateGaussianNoise>0.05 0.05 0.015</rateGaussianNoise>
-      <headingDrift>0.1</headingDrift>
-      <headingGaussianNoise>1.00</headingGaussianNoise>-->
-    </plugin>
-    <plugin name="gazebo_ros_control" filename="libgazebo_ros_control.so" />
-    <plugin name="imu_plugin" filename="libhector_gazebo_ros_imu.so">
-      <alwaysOn>true</alwaysOn>
-      <bodyName>chassis_link</bodyName>
-      <topicName>zed/imu</topicName>
-      <serviceName>imu_service</serviceName>
-      <updateRate>10.0</updateRate>
-      <rpyOffsets>0 0 0</rpyOffsets> <!-- deprecated -->
-  <!--
-        <gaussianNoise>0.1</gaussianNoise>
-        <accelDrift>0.5 0.5 0.5</accelDrift>
-        <accelGaussianNoise>0.35 0.35 0.3</accelGaussianNoise>
-        <rateDrift>0.1 0.1 0.1</rateDrift>
-        <rateGaussianNoise>0.05 0.05 0.015</rateGaussianNoise>
-        <headingDrift>0.1</headingDrift>
-        <headingGaussianNoise>1.00</headingGaussianNoise>-->
-  <!-- deprecated -->
-      <gaussianNoise>0.0</gaussianNoise>
-        <accelDrift>0.0 0.0 0.0</accelDrift>
-        <accelGaussianNoise>0.0 0.0 0.0</accelGaussianNoise>
-        <rateDrift>0.0 0.0 0.0</rateDrift>
-        <rateGaussianNoise>0.0 0.0 0.0</rateGaussianNoise>
-        <headingDrift>0.0</headingDrift>
-        <headingGaussianNoise>0.00</headingGaussianNoise>
-    </plugin>
-    <plugin name="am_gazebo_wheelencoder" filename="libam_gazebo_wheelencoder.so">
-  </plugin>
-  </gazebo>
-</xacro:unless>
  <!--
     <gazebo reference="chassis_link">

File: unicorn_description/urdf/wheel.urdf.xacro (robot description, xacro)
@@ -20,52 +20,33 @@
                params="fb lr parent translateX translateY translateZ wheel_radius wheel_height flip"> <!--fb : front, back ; lr: left, right -->
     <link name="${fb}_${lr}_wheel">
-    <visual>
-      <origin
-        xyz="0 0 0"
-        rpy="0 0 0" />
-      <geometry>
-        <mesh
-          filename="package://unicorn_description/meshes/wheel_driver.STL" />
-      </geometry>
-      <material
-        name="">
-        <color
-          rgba="0.752941176470588 0.752941176470588 0.752941176470588 1" />
-      </material>
-    </visual>
-    <collision>
-      <origin
-        xyz="0 0 0"
-        rpy="0 0 0" />
-      <geometry>
-        <mesh
-          filename="package://unicorn_description/meshes/wheel_driver.STL" />
-      </geometry>
-    </collision>
-    <inertial>
-      <origin
-        xyz="-6.0591E-12 -0.012242 1.8648E-11"
-        rpy="0 0 0" />
-      <mass
-        value="1.0564" />
-      <inertia
-        ixx="0.0040937"
-        ixy="3.2935E-14"
-        ixz="-4.4864E-13"
-        iyy="0.008088"
-        iyz="-6.8807E-12"
-        izz="0.0040937" />
-    </inertial>
+      <visual>
+        <origin xyz="0 0 0" rpy="${flip*M_PI/2} 0 0" />
+        <geometry>
+          <cylinder length="${wheel_height}" radius="${wheel_radius}" />
+        </geometry>
+        <material name="Black" />
+      </visual>
+      <collision>
+        <origin xyz="0 0 0" rpy="${flip*M_PI/2} 0 0" />
+        <geometry>
+          <cylinder length="${wheel_height}" radius="${wheel_radius}" />
+        </geometry>
+      </collision>
+      <inertial>
+        <mass value="${wheel_mass}" />
+        <!-- <origin xyz="0 0 0" rpy="${flip*M_PI/2} 0 0"/> -->
+        <origin xyz="0 0 0" />
+        <cylinder_inertia m="${wheel_mass}" r="${wheel_radius}" h="${wheel_height}" />
+      </inertial>
     </link>
-<!--
     <gazebo reference="${fb}_${lr}_wheel">
       <mu1 value="100.0" />
       <mu2 value="100.0" />
-      <kp value="1000.0" />
+      <kp value="10000000.0" />
       <kd value="1.0" />
       <fdir1 value="1 0 0" />
       <material>Gazebo/Black</material>
       <turnGravityOff>false</turnGravityOff>
-    </gazebo>-->
+    </gazebo>
     <joint name="${fb}_${lr}_wheel_joint" type="continuous">
       <parent link="${parent}" />
