Commit message: Add reverse movment for target file

File: unicorn_description/urdf/unicorn_sim.urdf.xacro (robot description, xacro)
@@ -112,5 +112,5 @@
       <origin
         xyz="0 0 0"
-        rpy="0 0 0" />
+        rpy="0 0 ${M_PI}" />
       <geometry>
         <mesh
@@ -126,5 +126,5 @@
       <origin
         xyz="0 0 0"
-        rpy="0 0 0" />
+        rpy="0 0 ${M_PI}" />
       <geometry>
         <mesh
@@ -138,5 +138,5 @@
     <origin
       xyz="0 0 0"
-      rpy="0 0 0" />
+      rpy="0 0 ${M_PI}" />
     <parent
       link="chassis_link" />
@@ -148,5 +148,5 @@
   </joint>
 <!--
-    <link
+  <link
     name="wheel_link">
     <inertial>
@@ -180,7 +180,11 @@
     </collision>
   </link>
+  <gazebo reference="base_link_gazebo">
+    <material>Gazebo/Green</material>
+    <turnGravityOff>false</turnGravityOff>
+  </gazebo>
   <joint name="base_chassis_joint" type="fixed">
     <parent link="chassis_link"/>
-    <child link="wheel_link" />wheel_link
+    <child link="wheel_link" />
   <origin xyz="0 0.0 0" rpy="0 0 ${M_PI}" />
   </joint>-->
@@ -189,6 +193,6 @@
   <wheel fb="back" lr="right" parent="chassis_link" rotationZ="0" translateY="-0.23" translateX="0 " translateZ="0.1225" wheel_radius="0.1225" wheel_height="0.032" flip="1"/>
   -->
-  <wheel fb="back" lr="left" parent="chassis_link"  translateY="0.23" translateX="0" translateZ="0.1225" wheel_radius="0.1225" wheel_height="0.032" flip="1"/>
-  <wheel fb="back" lr="right" parent="chassis_link" translateY="-0.23" translateX="0 " translateZ="0.1225" wheel_radius="0.1225" wheel_height="0.032" flip="1"/>
+  <wheel fb="back" lr="left" parent="lift_link"  translateY="0.24" translateX="0" translateZ="0.1225" wheel_radius="0.1225" wheel_height="0.032" flip="1"/>
+  <wheel fb="back" lr="right" parent="lift_link" translateY="-0.24" translateX="0 " translateZ="0.1225" wheel_radius="0.1225" wheel_height="0.032" flip="1"/>
   <!-- others wheels -->
   <swivel_wheel fb="front" lr="left" parent="chassis_link" translateY="0.16" translateX="-0.355" translateZ="0.1531" wheel_radius="0.05" wheel_height="0.05" flip="0"/>
@@ -303,20 +307,3 @@
   </gazebo>
 </xacro:if>
- <!--
-    <gazebo reference="chassis_link">
-    <sensor name="automower_sensor" type="contact">
-      <always_on>true</always_on>
-      <update_rate>50</update_rate>
-      <contact>
-        <collision>base_link_collision</collision>
-      </contact>
-      <plugin name="automower_sensors_plugin" filename="libam_gazebo_sensors.so">
-        <always_on>true</always_on>
-        <update_rate>20</update_rate>
-        <bumperTopicName>sensor_status</bumperTopicName>
-        <loopTopicName>loop</loopTopicName>
-        <loopOutsideSensors>15</loopOutsideSensors>
-      </plugin>
-    </sensor>
-  </gazebo>-->
 </robot>

File: unicorn_description/urdf/unicorn_target.urdf.xacro (robot description, xacro)
@@ -1,6 +1,3 @@
 <?xml version="1.0" encoding="utf-8"?>
-<!-- This URDF was automatically created by SolidWorks to URDF Exporter! Originally created by Stephen Brawner (brawner@gmail.com)
-     Commit Version: 1.6.0-1-g15f4949  Build Version: 1.6.7594.29634
-     For more information, please see http://wiki.ros.org/sw_urdf_exporter -->
 <robot name="unicorn" xmlns:xacro="http://www.ros.org/wiki/xacro">
   <xacro:arg name="robot_namespace" default="/" />
@@ -16,9 +13,20 @@
   <xacro:property name="M_PI" value="3.1415926535897931" />
   <xacro:property name="M_PI2" value="1.57079632679" />
-  <!-- base -->
+  <!-- base --><!--
     <xacro:property name="base_x_size" value="0.72" />
   <xacro:property name="base_y_size" value="0.55" />
   <xacro:property name="base_z_size" value="0.6" />
-  <xacro:property name="base_mass" value="21.446" /> <!-- 21.446 in kg-->
+  <xacro:property name="base_mass" value="21.446" /> 21.446 in kg-->
+    <!-- Main Body-base -->
+  <xacro:property name="base_x_size" value="0.72" />
+  <xacro:property name="base_y_size" value="0.55" />
+  <xacro:property name="base_z_size" value="0.23" />
+  <xacro:property name="base_mass" value="15" /> <!-- in kg-->
+    <!--Inertial macros for the box and cylinder. Units are kg*m^2-->
+  <xacro:macro name="box_inertia" params="m x y z">
+    <inertia ixx="${m*(y*y+z*z)/12}" ixy="0" ixz="0"
+             iyy="${m*(x*x+z*z)/12}" iyz="0"
+             izz="${m*(x*x+z*z)/12}" />
+  </xacro:macro>
   <!-- Front Lidar -->
   <xacro:arg name="laser_xyz" default="-0.0214 -0.0049 0.465" />
@@ -46,5 +54,5 @@
         rpy="0 0 0" />
       <mass
-        value="15" />
+        value="10" />
       <inertia
         ixx="1"
@@ -76,4 +84,9 @@
         <mesh
           filename="package://unicorn_description/meshes/chassis_link.STL" />
+        <surface>
+         <friction>
+           <ode><mu>0.4</mu><mu2>0.4</mu2></ode>
+         </friction>
+      </surface>
       </geometry>
     </collision>
@@ -99,5 +112,5 @@
       <origin
         xyz="0 0 0"
-        rpy="0 0 0" />
+        rpy="0 0 ${M_PI}" />
       <geometry>
         <mesh
@@ -113,5 +126,5 @@
       <origin
         xyz="0 0 0"
-        rpy="0 0 0" />
+        rpy="0 0 ${M_PI}" />
       <geometry>
         <mesh
@@ -125,5 +138,5 @@
     <origin
       xyz="0 0 0"
-      rpy="0 0 0" />
+      rpy="0 0 ${M_PI}" />
     <parent
       link="chassis_link" />
@@ -134,10 +147,55 @@
     <joint_properties damping="0.0" friction="0.0" />
   </joint>
-  <!-- driving wheels -->
-  <wheel fb="back" lr="left" parent="chassis_link" translateY="0.25" translateX="0" translateZ="0.122" wheel_radius="0.122" wheel_height="0.032" flip="1"/>
-  <wheel fb="back" lr="right" parent="chassis_link" translateY="-0.25" translateX="0 " translateZ="0.122" wheel_radius="0.122" wheel_height="0.032" flip="1"/>
+<!--
+  <link
+    name="wheel_link">
+    <inertial>
+      <origin
+        xyz="0 0 0"
+        rpy="0 0 0" />
+      <mass
+        value="0.01" />
+      <box_inertia  m="${5*0.01}" x="${base_x_size}" y="${base_y_size}" z="${base_z_size}"/>
+    </inertial>
+    <visual>
+      <origin
+        xyz="0 0 0"
+        rpy="0 0 0" />
+      <geometry>
+        <box size="0.01 0.01 0.01"/>
+      </geometry>
+      <material
+        name="">
+        <color
+          rgba="0.79216 0.81961 0.93333 1" />
+      </material>
+    </visual>
+    <collision>
+      <origin
+        xyz="0 0 0"
+        rpy="0 0 0" />
+      <geometry>
+          <box size="0.01 0.01 0.01"/>
+      </geometry>
+    </collision>
+  </link>
+  <gazebo reference="base_link_gazebo">
+    <material>Gazebo/Green</material>
+    <turnGravityOff>false</turnGravityOff>
+  </gazebo>
+  <joint name="base_chassis_joint" type="fixed">
+    <parent link="chassis_link"/>
+    <child link="wheel_link" />
+  <origin xyz="0 0.0 0" rpy="0 0 ${M_PI}" />
+  </joint>-->
+  <!-- driving wheels
+  <wheel fb="back" lr="left" parent="chassis_link" rotationZ="3.14159" translateY="0.23" translateX="0" translateZ="0.1225" wheel_radius="0.1225" wheel_height="0.032" flip="1"/>
+  <wheel fb="back" lr="right" parent="chassis_link" rotationZ="0" translateY="-0.23" translateX="0 " translateZ="0.1225" wheel_radius="0.1225" wheel_height="0.032" flip="1"/>
+  -->
+  <wheel fb="back" lr="left" parent="lift_link"  translateY="0.24" translateX="0" translateZ="0.1225" wheel_radius="0.1225" wheel_height="0.032" flip="1"/>
+  <wheel fb="back" lr="right" parent="lift_link" translateY="-0.24" translateX="0 " translateZ="0.1225" wheel_radius="0.1225" wheel_height="0.032" flip="1"/>
   <!-- others wheels -->
-  <swivel_wheel fb="front" lr="left" parent="chassis_link" translateY="0.16" translateX="-0.355" translateZ="0.1526" wheel_radius="0.05" wheel_height="0.05" flip="0"/>
-  <swivel_wheel fb="front" lr="right" parent="chassis_link" translateY="-0.16" translateX="-0.355" translateZ="0.1526" wheel_radius="0.05" wheel_height="0.05" flip="0"/>
+  <swivel_wheel fb="front" lr="left" parent="chassis_link" translateY="0.16" translateX="-0.355" translateZ="0.1531" wheel_radius="0.05" wheel_height="0.05" flip="0"/>
+  <swivel_wheel fb="front" lr="right" parent="chassis_link" translateY="-0.16" translateX="-0.355" translateZ="0.1531" wheel_radius="0.05" wheel_height="0.05" flip="0"/>
  <!-- Front Lidar -->
   <lidar_gazebo frame="base_laser" topic="frontLidar/scan" simulation="$(arg sim)" sample_size="800" min_angle="-2.35619" max_angle="2.35619" robot_namespace="$(arg robot_namespace)" filename="$(arg frontlidar_meshfile)" />
@@ -167,5 +225,5 @@
     </joint>
   <!-- realsense Camera -->
-    <stereo_camera frame_rgb="realsense_camera" frame_depth="realsense_depth" cameraName="realsense" simulation="$(arg sim)" filename="$(arg realsense_meshfile)"  topic="pointcloud" robot_namespace="$(arg robot_namespace)"/>
+    <stereo_camera frame_rgb="realsense_camera" frame_depth="realsense_depth_joint" cameraName="realsense" simulation="$(arg sim)" filename="$(arg realsense_meshfile)"  topic="pointcloud" robot_namespace="$(arg robot_namespace)"/>
     <joint name="realsense_gb_joint" type="fixed">
       <origin xyz="$(arg real_rgb_xyz)" rpy="$(arg real_rpy)"/>
@@ -174,7 +232,7 @@
     </joint>
     <joint name="realsense_depth_joint" type="fixed">
-      <origin xyz="0 0 0" rpy="${-pi/2} 0 ${-pi/2}"/>
+      <origin xyz="$(arg real_depth_xyz)" rpy="${-pi/2} 0 ${-pi/2}"/>
       <parent link="realsense_camera"/>
-      <child link="realsense_depth"/>
+      <child link="realsense_depth_joint"/>
     </joint>
 <xacro:if value="$(arg sim)">
@@ -207,6 +265,6 @@
       <wheelTorque>100</wheelTorque>
       <commandTopic>cmd_vel</commandTopic>
-      <odometryTopic>wheelencoder/odom</odometryTopic>
-      <odometryFrame>odom_chassis</odometryFrame>
+      <odometryTopic>wheel_encoder/odom</odometryTopic>
+      <odometryFrame>odom_chassis_dont_use</odometryFrame>
       <robotBaseFrame>chassis_link</robotBaseFrame>
       <publishWheelTF>false</publishWheelTF>
@@ -223,9 +281,9 @@
     <plugin name="imu_plugin" filename="libhector_gazebo_ros_imu.so">
       <alwaysOn>true</alwaysOn>
-      <bodyName>chassis_link</bodyName>
+      <bodyName>zed_camera</bodyName>
       <topicName>zed/imu</topicName>
       <serviceName>imu_service</serviceName>
       <updateRate>100.0</updateRate>
-      <rpyOffsets>0 ${M_PI} 0</rpyOffsets>
+      <rpyOffsets>0 0 0</rpyOffsets>
   <!---->
         <gaussianNoise>0.1</gaussianNoise>
@@ -249,84 +307,3 @@
   </gazebo>
 </xacro:if>
-<xacro:unless value="$(arg sim)">
-  <!-- GAZEBO STUFF for unicorn -->
-  <gazebo>
-    <plugin name="automower_gazebo_controller" filename="libam_gazebo_controller_2wd.so">
-      <alwaysOn>true</alwaysOn>
-      <updateRate>100.0</updateRate>
-      <leftJoint>back_right_wheel_joint</leftJoint>
-      <rightJoint>back_left_wheel_joint</rightJoint>
-      <wheelSeparation>0.4645</wheelSeparation>
-      <wheelDiameter>0.245</wheelDiameter>
-      <wheelTorque>100</wheelTorque>
-      <commandTopic>cmd_vel</commandTopic>
-      <odometryTopic>wheelencoder/odom</odometryTopic>
-      <odometryFrame>odom_gazebo</odometryFrame>
-      <robotBaseFrame>chassis_link_gazebo</robotBaseFrame>
-      <publishWheelTF>false</publishWheelTF>
-      <publishWheelJointState>false</publishWheelJointState>
-    </plugin>
-    <plugin name="gazebo_ros_control" filename="libgazebo_ros_control.so" />
-    <plugin name="imu_plugin" filename="libhector_gazebo_ros_imu.so">
-    <alwaysOn>false</alwaysOn>
-    <bodyName>chassis_link_gazebo</bodyName>
-    <topicName>imu</topicName>
-    <serviceName>imu_service</serviceName>
-    <updateRate>100.0</updateRate>
-    <rpyOffsets>0 0 0</rpyOffsets> <!-- deprecated -->
-<!--
-      <gaussianNoise>0.1</gaussianNoise>
-      <accelDrift>0.5 0.5 0.5</accelDrift>
-      <accelGaussianNoise>0.35 0.35 0.3</accelGaussianNoise>
-      <rateDrift>0.1 0.1 0.1</rateDrift>
-      <rateGaussianNoise>0.05 0.05 0.015</rateGaussianNoise>
-      <headingDrift>0.1</headingDrift>
-      <headingGaussianNoise>1.00</headingGaussianNoise>-->
-    </plugin>
-    <plugin name="gazebo_ros_control" filename="libgazebo_ros_control.so" />
-    <plugin name="imu_plugin" filename="libhector_gazebo_ros_imu.so">
-      <alwaysOn>true</alwaysOn>
-      <bodyName>chassis_link</bodyName>
-      <topicName>zed/imu</topicName>
-      <serviceName>imu_service</serviceName>
-      <updateRate>10.0</updateRate>
-      <rpyOffsets>0 0 0</rpyOffsets> <!-- deprecated -->
-  <!--
-        <gaussianNoise>0.1</gaussianNoise>
-        <accelDrift>0.5 0.5 0.5</accelDrift>
-        <accelGaussianNoise>0.35 0.35 0.3</accelGaussianNoise>
-        <rateDrift>0.1 0.1 0.1</rateDrift>
-        <rateGaussianNoise>0.05 0.05 0.015</rateGaussianNoise>
-        <headingDrift>0.1</headingDrift>
-        <headingGaussianNoise>1.00</headingGaussianNoise>-->
-  <!-- deprecated -->
-      <gaussianNoise>0.0</gaussianNoise>
-        <accelDrift>0.0 0.0 0.0</accelDrift>
-        <accelGaussianNoise>0.0 0.0 0.0</accelGaussianNoise>
-        <rateDrift>0.0 0.0 0.0</rateDrift>
-        <rateGaussianNoise>0.0 0.0 0.0</rateGaussianNoise>
-        <headingDrift>0.0</headingDrift>
-        <headingGaussianNoise>0.00</headingGaussianNoise>
-    </plugin>
-    <plugin name="am_gazebo_wheelencoder" filename="libam_gazebo_wheelencoder.so">
-  </plugin>
-  </gazebo>
-</xacro:unless>
- <!--
-    <gazebo reference="chassis_link">
-    <sensor name="automower_sensor" type="contact">
-      <always_on>true</always_on>
-      <update_rate>50</update_rate>
-      <contact>
-        <collision>base_link_collision</collision>
-      </contact>
-      <plugin name="automower_sensors_plugin" filename="libam_gazebo_sensors.so">
-        <always_on>true</always_on>
-        <update_rate>20</update_rate>
-        <bumperTopicName>sensor_status</bumperTopicName>
-        <loopTopicName>loop</loopTopicName>
-        <loopOutsideSensors>15</loopOutsideSensors>
-      </plugin>
-    </sensor>
-  </gazebo>-->
 </robot>
