Commit message: Updated realsense links in urdf

File: unicorn_description/urdf/unicorn_sim.urdf.xacro (robot description, xacro)
@@ -42,7 +42,10 @@
   <xacro:arg name="zed_meshfile" default="package://unicorn_description/meshes/zed_link.STL" />
   <!-- Real Sense -->
-  <xacro:arg name="real_rgb_xyz" default="-0.4065 -0.03882 0.33658" />
-  <xacro:arg name="real_depth_xyz" default="-0.4065 -0.00518 0.33658" />
+  <xacro:arg name="real_base" default="-0.4065 ${-0.03882+0.015} 0.33658" />
+  <xacro:arg name="real_rgb_xyz" default="0 0.015 0" />
+  <xacro:arg name="real_depth_xyz" default="0 0 0" />
   <xacro:arg name="real_rpy" default="0 0 ${M_PI}" />
+  <xacro:arg name="real_optical_rpy" default="${-M_PI2} 0 ${-M_PI2}" />
+  <xacro:arg name="real_depth_rpy" default="${-M_PI2} 0 ${-M_PI2}" />
   <xacro:arg name="realsense_meshfile" default="package://unicorn_description/meshes/real_sense.STL" />
  <!-- Main Body-base -->
@@ -215,5 +218,5 @@
   </joint>
   <!-- Zed Camera -->
-    <stereo_camera frame_rgb="zed_camera" frame_depth="zed_depth_joint" cameraName="zed" simulation="$(arg sim)" filename="$(arg zed_meshfile)"  topic="pointcloud" robot_namespace="$(arg robot_namespace)"/>
+    <stereo_camera frame_rgb="zed_camera" frame_depth="zed_depth" cameraName="zed" simulation="$(arg sim)" filename="$(arg zed_meshfile)"  topic="pointcloud" robot_namespace="$(arg robot_namespace)"/>
     <joint name="zed_camera_rgb_joint" type="fixed">
       <origin xyz="$(arg zed_xyz)" rpy="$(arg zed_rpy)"/>
@@ -225,20 +228,58 @@
       <origin xyz="0 0 0" rpy="${-pi/2} 0 ${-pi/2}"/>
       <parent link="zed_camera"/>
-      <child link="zed_depth_joint"/>
+      <child link="zed_depth"/>
       <joint_properties damping="1" friction="0.5" />
     </joint>
   <!-- realsense Camera -->
-    <stereo_camera frame_rgb="realsense_camera" frame_depth="realsense_depth_joint" cameraName="realsense" simulation="$(arg sim)" filename="$(arg realsense_meshfile)"  topic="pointcloud" robot_namespace="$(arg robot_namespace)"/>
+  <stereo_camera frame_rgb="realsense_color_frame" frame_depth="realsense_depth_frame" cameraName="realsense" simulation="$(arg sim)" filename="$(arg realsense_meshfile)"  topic="pointcloud" robot_namespace="$(arg robot_namespace)"/>
+  <link
+    name="realsense_link">
+    <inertial>
+      <origin
+        xyz="0 0 0"
+        rpy="0 0 0" />
+      <mass
+        value="0.01" />
+      <box_inertia  m="${5*0.01}" x="${base_x_size}" y="${base_y_size}" z="${base_z_size}"/>
+    </inertial>
+    <collision>
+      <origin
+        xyz="0 0 0"
+        rpy="0 0 0" />
+      <geometry>
+          <box size="0.01 0.01 0.01"/>
+      </geometry>
+    </collision>
+  </link>
+  <link
+    name="realsense_depth_optical_frame">
+  </link>
+  <link
+    name="realsense_color_optical_frame">
+  </link>
+    <joint name="realsense_joint" type="fixed">
+      <origin xyz="$(arg real_base)" rpy="$(arg real_rpy)"/>
+      <parent link="chassis_link"/>
+      <child link="realsense_link"/>
+    </joint>
     <joint name="realsense_gb_joint" type="fixed">
-      <origin xyz="$(arg real_rgb_xyz)" rpy="$(arg real_rpy)"/>
-      <parent link="chassis_link"/>
-      <child link="realsense_camera"/>
-      <joint_properties damping="1" friction="0.5" />
+      <origin xyz="$(arg real_rgb_xyz)" rpy="0 0 0"/>
+      <parent link="realsense_link"/>
+      <child link="realsense_color_frame"/>
     </joint>
     <joint name="realsense_depth_joint" type="fixed">
-      <origin xyz="$(arg real_depth_xyz)" rpy="${-pi/2} 0 ${-pi/2}"/>
-      <parent link="realsense_camera"/>
-      <child link="realsense_depth_joint"/>
-      <joint_properties damping="1" friction="0.5" />
+      <origin xyz="$(arg real_depth_xyz)" rpy="0 0 0"/>
+      <parent link="realsense_link"/>
+      <child link="realsense_depth_frame"/>
+    </joint>
+    <joint name="realsense_optical_color_joint" type="fixed">
+      <origin xyz="0 0 0" rpy="$(arg real_optical_rpy)"/>
+      <parent link="realsense_color_frame"/>
+      <child link="realsense_color_optical_frame"/>
+    </joint>
+    <joint name="realsense_optical_depth_joint" type="fixed">
+      <origin xyz="0 0 0" rpy="$(arg real_depth_rpy)"/>
+      <parent link="realsense_depth_frame"/>
+      <child link="realsense_depth_optical_frame"/>
     </joint>
 <xacro:if value="$(arg sim)">

File: unicorn_description/urdf/unicorn_target.urdf.xacro (robot description, xacro)
@@ -42,7 +42,10 @@
   <xacro:arg name="zed_meshfile" default="package://unicorn_description/meshes/zed_link.STL" />
   <!-- Real Sense -->
-  <xacro:arg name="real_rgb_xyz" default="-0.4065 -0.03882 0.33658" />
-  <xacro:arg name="real_depth_xyz" default="-0.4065 -0.00518 0.33658" />
+  <xacro:arg name="real_base" default="-0.4065 ${-0.03882+0.015} 0.33658" />
+  <xacro:arg name="real_rgb_xyz" default="0 0.015 0" />
+  <xacro:arg name="real_depth_xyz" default="0 0 0" />
   <xacro:arg name="real_rpy" default="0 0 ${M_PI}" />
+  <xacro:arg name="real_optical_rpy" default="${-M_PI2} 0 ${-M_PI2}" />
+  <xacro:arg name="real_depth_rpy" default="${-M_PI2} 0 ${-M_PI2}" />
   <xacro:arg name="realsense_meshfile" default="package://unicorn_description/meshes/real_sense.STL" />
  <!-- Main Body-base -->
@@ -185,46 +188,4 @@
   <origin xyz="0 0.0 0" rpy="0 0 ${M_PI}" />
   </joint>
-<!--
-  <link
-    name="wheel_link">
-    <inertial>
-      <origin
-        xyz="0 0 0"
-        rpy="0 0 0" />
-      <mass
-        value="0.01" />
-      <box_inertia  m="${5*0.01}" x="${base_x_size}" y="${base_y_size}" z="${base_z_size}"/>
-    </inertial>
-    <visual>
-      <origin
-        xyz="0 0 0"
-        rpy="0 0 0" />
-      <geometry>
-        <box size="0.01 0.01 0.01"/>
-      </geometry>
-      <material
-        name="">
-        <color
-          rgba="0.79216 0.81961 0.93333 1" />
-      </material>
-    </visual>
-    <collision>
-      <origin
-        xyz="0 0 0"
-        rpy="0 0 0" />
-      <geometry>
-          <box size="0.01 0.01 0.01"/>
-      </geometry>
-    </collision>
-  </link>
-  <gazebo reference="base_link_gazebo">
-    <material>Gazebo/Green</material>
-    <turnGravityOff>false</turnGravityOff>
-  </gazebo>
-  <joint name="base_chassis_joint" type="fixed">
-    <parent link="base_link"/>
-    <child link="wheel_link" />
-  <origin xyz="0 0.0 0" rpy="0 0 ${M_PI}" />
-  </joint>-->
   <!-- driving wheels
   <wheel fb="back" lr="left" parent="base_link" rotationZ="3.14159" translateY="0.23" translateX="0" translateZ="0.1225" wheel_radius="0.1225" wheel_height="0.032" flip="1"/>
@@ -263,14 +224,54 @@
     </joint>
   <!-- realsense Camera -->
-    <stereo_camera frame_rgb="realsense_camera" frame_depth="realsense_depth_joint" cameraName="realsense" simulation="$(arg sim)" filename="$(arg realsense_meshfile)"  topic="pointcloud" robot_namespace="$(arg robot_namespace)"/>
+    <stereo_camera frame_rgb="realsense_color_frame" frame_depth="realsense_depth_frame" cameraName="realsense" simulation="$(arg sim)" filename="$(arg realsense_meshfile)"  topic="pointcloud" robot_namespace="$(arg robot_namespace)"/>
+  <link
+    name="realsense_link">
+    <inertial>
+      <origin
+        xyz="0 0 0"
+        rpy="0 0 0" />
+      <mass
+        value="0.01" />
+      <box_inertia  m="${5*0.01}" x="${base_x_size}" y="${base_y_size}" z="${base_z_size}"/>
+    </inertial>
+    <collision>
+      <origin
+        xyz="0 0 0"
+        rpy="0 0 0" />
+      <geometry>
+          <box size="0.01 0.01 0.01"/>
+      </geometry>
+    </collision>
+  </link>
+  <link
+    name="realsense_depth_optical_frame">
+  </link>
+  <link
+    name="realsense_color_optical_frame">
+  </link>
+    <joint name="realsense_joint" type="fixed">
+      <origin xyz="$(arg real_base)" rpy="$(arg real_rpy)"/>
+      <parent link="chassis_link"/>
+      <child link="realsense_link"/>
+    </joint>
     <joint name="realsense_gb_joint" type="fixed">
-      <origin xyz="$(arg real_rgb_xyz)" rpy="$(arg real_rpy)"/>
-      <parent link="base_link"/>
-      <child link="realsense_camera"/>
+      <origin xyz="$(arg real_rgb_xyz)" rpy="0 0 0"/>
+      <parent link="realsense_link"/>
+      <child link="realsense_color_frame"/>
     </joint>
     <joint name="realsense_depth_joint" type="fixed">
-      <origin xyz="$(arg real_depth_xyz)" rpy="${-pi/2} 0 ${-pi/2}"/>
-      <parent link="realsense_camera"/>
-      <child link="realsense_depth_joint"/>
+      <origin xyz="$(arg real_depth_xyz)" rpy="0 0 0"/>
+      <parent link="realsense_link"/>
+      <child link="realsense_depth_frame"/>
+    </joint>
+    <joint name="realsense_optical_color_joint" type="fixed">
+      <origin xyz="0 0 0" rpy="$(arg real_optical_rpy)"/>
+      <parent link="realsense_color_frame"/>
+      <child link="realsense_color_optical_frame"/>
+    </joint>
+    <joint name="realsense_optical_depth_joint" type="fixed">
+      <origin xyz="0 0 0" rpy="$(arg real_depth_rpy)"/>
+      <parent link="realsense_depth_frame"/>
+      <child link="realsense_depth_optical_frame"/>
     </joint>
 <xacro:if value="$(arg sim)">

File: unicorn_description/urdf/unicorn_target_backwards.urdf.xacro (robot description, xacro)
@@ -2,9 +2,9 @@
 <robot name="unicorn" xmlns:xacro="http://www.ros.org/wiki/xacro">
   <xacro:arg name="robot_namespace" default="/" />
-  <xacro:arg name="sim" default="false" />
+  <xacro:arg name="sim" default="true" />
     <!-- Swivel wheel -->
   <xacro:include filename="$(find unicorn_description)/urdf/swivel_wheel.urdf.xacro" />
     <!-- Wheel -->
-  <xacro:include filename="$(find am_description)/urdf/wheel.urdf.xacro" />
+  <xacro:include filename="$(find unicorn_description)/urdf/wheel.urdf.xacro" />
     <!-- camera pack-->
   <xacro:include filename="$(find unicorn_description)/urdf/stereo_camera_gazebo.urdf.xacro" />
@@ -42,7 +42,10 @@
   <xacro:arg name="zed_meshfile" default="package://unicorn_description/meshes/zed_link.STL" />
   <!-- Real Sense -->
-  <xacro:arg name="real_rgb_xyz" default="-0.4065 -0.03882 0.33658" />
-  <xacro:arg name="real_depth_xyz" default="-0.4065 -0.00518 0.33658" />
+  <xacro:arg name="real_base" default="-0.4065 ${-0.03882+0.015} 0.33658" />
+  <xacro:arg name="real_rgb_xyz" default="0 0.015 0" />
+  <xacro:arg name="real_depth_xyz" default="0 0 0" />
   <xacro:arg name="real_rpy" default="0 0 ${M_PI}" />
+  <xacro:arg name="real_optical_rpy" default="${-M_PI2} 0 ${-M_PI2}" />
+  <xacro:arg name="real_depth_rpy" default="${-M_PI2} 0 ${-M_PI2}" />
   <xacro:arg name="realsense_meshfile" default="package://unicorn_description/meshes/real_sense.STL" />
  <!-- Main Body-base -->
@@ -54,5 +57,5 @@
         rpy="0 0 0" />
       <mass
-        value="10" />
+        value="15" />
       <inertia
         ixx="1"
@@ -145,21 +148,22 @@
     <axis
       xyz="0 0 0" />
-    <joint_properties damping="0.0" friction="0.0" />
+    <joint_properties damping="1" friction="0.5" />
   </joint>
   <!-- driving wheels
-  <wheel fb="back" lr="left" parent="base_link" rotationZ="3.14159" translateY="0.23" translateX="0" translateZ="0.1225" wheel_radius="0.1225" wheel_height="0.032" flip="1"/>
-  <wheel fb="back" lr="right" parent="base_link" rotationZ="0" translateY="-0.23" translateX="0 " translateZ="0.1225" wheel_radius="0.1225" wheel_height="0.032" flip="1"/>
+  <wheel fb="back" lr="left" parent="chassis_link" rotationZ="3.14159" translateY="0.23" translateX="0" translateZ="0.1225" wheel_radius="0.1225" wheel_height="0.032" flip="1"/>
+  <wheel fb="back" lr="right" parent="chassis_link" rotationZ="0" translateY="-0.23" translateX="0 " translateZ="0.1225" wheel_radius="0.1225" wheel_height="0.032" flip="1"/>
   -->
   <wheel fb="back" lr="left" parent="lift_link"  translateY="0.24" translateX="0" translateZ="0.1225" wheel_radius="0.1225" wheel_height="0.032" flip="1"/>
   <wheel fb="back" lr="right" parent="lift_link" translateY="-0.24" translateX="0 " translateZ="0.1225" wheel_radius="0.1225" wheel_height="0.032" flip="1"/>
   <!-- others wheels -->
-  <swivel_wheel fb="front" lr="left" parent="base_link" translateY="0.16" translateX="-0.355" translateZ="0.1531" wheel_radius="0.05" wheel_height="0.05" flip="0"/>
-  <swivel_wheel fb="front" lr="right" parent="base_link" translateY="-0.16" translateX="-0.355" translateZ="0.1531" wheel_radius="0.05" wheel_height="0.05" flip="0"/>
+  <swivel_wheel fb="front" lr="left" parent="chassis_link" translateY="0.16" translateX="-0.355" translateZ="0.1531" wheel_radius="0.05" wheel_height="0.05" flip="0"/>
+  <swivel_wheel fb="front" lr="right" parent="chassis_link" translateY="-0.16" translateX="-0.355" translateZ="0.1531" wheel_radius="0.05" wheel_height="0.05" flip="0"/>
  <!-- Front Lidar -->
   <lidar_gazebo frame="base_laser" topic="frontLidar/scan" simulation="$(arg sim)" sample_size="800" min_angle="-2.35619" max_angle="2.35619" robot_namespace="$(arg robot_namespace)" filename="$(arg frontlidar_meshfile)" />
   <joint name="laser_mount_joint" type="fixed">
     <origin xyz="$(arg laser_xyz)" rpy="$(arg laser_rpy)" />
-    <parent link="base_link" />
+    <parent link="chassis_link" />
     <child link="base_laser" />
+    <joint_properties damping="1" friction="0.5" />
   </joint>
    <!-- Back Lidar -->
@@ -167,30 +171,73 @@
   <joint name="rear_laser_mount_joint" type="fixed">
     <origin xyz="$(arg rear_laser_xyz)" rpy="$(arg rear_laser_rpy)" />
-    <parent link="base_link" />
+    <parent link="chassis_link" />
     <child link="rear_laser" />
+    <joint_properties damping="1" friction="0.5" />
   </joint>
   <!-- Zed Camera -->
-    <stereo_camera frame_rgb="zed_camera" frame_depth="zed_depth_joint" cameraName="zed" simulation="$(arg sim)" filename="$(arg zed_meshfile)"  topic="pointcloud" robot_namespace="$(arg robot_namespace)"/>
+    <stereo_camera frame_rgb="zed_camera" frame_depth="zed_depth" cameraName="zed" simulation="$(arg sim)" filename="$(arg zed_meshfile)"  topic="pointcloud" robot_namespace="$(arg robot_namespace)"/>
     <joint name="zed_camera_rgb_joint" type="fixed">
       <origin xyz="$(arg zed_xyz)" rpy="$(arg zed_rpy)"/>
-      <parent link="base_link"/>
+      <parent link="chassis_link"/>
       <child link="zed_camera"/>
+      <joint_properties damping="1" friction="0.5" />
     </joint>
     <joint name="zed_camera_depth_joint" type="fixed">
       <origin xyz="0 0 0" rpy="${-pi/2} 0 ${-pi/2}"/>
       <parent link="zed_camera"/>
-      <child link="zed_depth_joint"/>
+      <child link="zed_depth"/>
+      <joint_properties damping="1" friction="0.5" />
     </joint>
   <!-- realsense Camera -->
-    <stereo_camera frame_rgb="realsense_camera" frame_depth="realsense_depth_joint" cameraName="realsense" simulation="$(arg sim)" filename="$(arg realsense_meshfile)"  topic="pointcloud" robot_namespace="$(arg robot_namespace)"/>
+    <stereo_camera frame_rgb="realsense_color_frame" frame_depth="realsense_depth_frame" cameraName="realsense" simulation="$(arg sim)" filename="$(arg realsense_meshfile)"  topic="pointcloud" robot_namespace="$(arg robot_namespace)"/>
+  <link
+    name="realsense_link">
+    <inertial>
+      <origin
+        xyz="0 0 0"
+        rpy="0 0 0" />
+      <mass
+        value="0.01" />
+      <box_inertia  m="${5*0.01}" x="${base_x_size}" y="${base_y_size}" z="${base_z_size}"/>
+    </inertial>
+    <collision>
+      <origin
+        xyz="0 0 0"
+        rpy="0 0 0" />
+      <geometry>
+          <box size="0.01 0.01 0.01"/>
+      </geometry>
+    </collision>
+  </link>
+  <link
+    name="realsense_depth_optical_frame">
+  </link>
+  <link
+    name="realsense_color_optical_frame">
+  </link>
+    <joint name="realsense_joint" type="fixed">
+      <origin xyz="$(arg real_base)" rpy="$(arg real_rpy)"/>
+      <parent link="chassis_link"/>
+      <child link="realsense_link"/>
+    </joint>
     <joint name="realsense_gb_joint" type="fixed">
-      <origin xyz="$(arg real_rgb_xyz)" rpy="$(arg real_rpy)"/>
-      <parent link="base_link"/>
-      <child link="realsense_camera"/>
+      <origin xyz="$(arg real_rgb_xyz)" rpy="0 0 0"/>
+      <parent link="realsense_link"/>
+      <child link="realsense_color_frame"/>
     </joint>
     <joint name="realsense_depth_joint" type="fixed">
-      <origin xyz="$(arg real_depth_xyz)" rpy="${-pi/2} 0 ${-pi/2}"/>
-      <parent link="realsense_camera"/>
-      <child link="realsense_depth_joint"/>
+      <origin xyz="$(arg real_depth_xyz)" rpy="0 0 0"/>
+      <parent link="realsense_link"/>
+      <child link="realsense_depth_frame"/>
+    </joint>
+    <joint name="realsense_optical_color_joint" type="fixed">
+      <origin xyz="0 0 0" rpy="$(arg real_optical_rpy)"/>
+      <parent link="realsense_color_frame"/>
+      <child link="realsense_color_optical_frame"/>
+    </joint>
+    <joint name="realsense_optical_depth_joint" type="fixed">
+      <origin xyz="0 0 0" rpy="$(arg real_depth_rpy)"/>
+      <parent link="realsense_depth_frame"/>
+      <child link="realsense_depth_optical_frame"/>
     </joint>
 <xacro:if value="$(arg sim)">
@@ -201,5 +248,5 @@
       <updateRate>5</updateRate>
       <frameId>odom_chassis</frameId>
-      <bodyName>base_link</bodyName>
+      <bodyName>chassis_link</bodyName>
       <topicName>gps</topicName>
       <velocityTopicName>gps_velocity</velocityTopicName>
@@ -216,5 +263,5 @@
     <plugin name="automower_gazebo_controller" filename="libam_gazebo_controller_2wd.so">
       <alwaysOn>true</alwaysOn>
-      <updateRate>100.0</updateRate>
+      <updateRate>50.0</updateRate>
       <leftJoint>back_right_wheel_joint</leftJoint>
       <rightJoint>back_left_wheel_joint</rightJoint>
@@ -224,7 +271,8 @@
       <commandTopic>cmd_vel</commandTopic>
       <odometryTopic>wheel_encoder/odom</odometryTopic>
-      <odometryFrame>odom_chassis_dont_use</odometryFrame>
-      <robotBaseFrame>base_link</robotBaseFrame>
+      <odometryFrame>odom_chassis</odometryFrame>
+      <robotBaseFrame>chassis_link</robotBaseFrame>
       <publishWheelTF>false</publishWheelTF>
+      <publishOdomTF>false</publishOdomTF>
       <publishWheelJointState>false</publishWheelJointState>
       <gaussianNoise>0.1</gaussianNoise>

Commit message: Added dummy link for realsense model for real robot description

File: unicorn_description/urdf/unicorn_sim.urdf.xacro (robot description, xacro)
@@ -184,4 +184,5 @@
     </joint>
   <!-- realsense Camera -->
+<!-- Links only needed in simulation, created by realsense software otherwise-->
   <link
     name="realsense_link">
@@ -192,5 +193,20 @@
     <child link="realsense_link"/>
   </joint>
-  <!-- Links only needed in simulation, created by realsense software otherwise-->
+<xacro:if value="$(arg sim)">
+  <link
+    name="realsense_model_dummy_link">
+    <visual>
+        <origin xyz="0 0 0" rpy="0 0 0"/>
+        <geometry>
+            <mesh filename="$(arg realsense_meshfile)" />
+        </geometry>
+      </visual>
+  </link>
+  <joint name="realsense_model_joint" type="fixed">
+    <origin xyz="$(arg real_rgb_xyz)" rpy="0 0 0"/>
+    <parent link="realsense_link"/>
+    <child link="realsense_model_dummy_link"/>
+  </joint>
+</xacro:if>
 <xacro:if value="$(arg sim)">
   <stereo_camera frame_rgb="realsense_color_frame" frame_depth="realsense_depth_frame" cameraName="realsense" simulation="$(arg sim)" filename="$(arg realsense_meshfile)"  topic="pointcloud" robot_namespace="$(arg robot_namespace)"/>

File: unicorn_description/urdf/unicorn_target.urdf.xacro (robot description, xacro)
@@ -232,4 +232,20 @@
     <child link="realsense_link"/>
   </joint>
+<xacro:if value="$(arg sim)">
+  <link
+    name="realsense_model_dummy_link">
+    <visual>
+        <origin xyz="0 0 0" rpy="0 0 0"/>
+        <geometry>
+            <mesh filename="$(arg realsense_meshfile)" />
+        </geometry>
+      </visual>
+  </link>
+  <joint name="realsense_model_joint" type="fixed">
+    <origin xyz="$(arg real_rgb_xyz)" rpy="0 0 0"/>
+    <parent link="realsense_link"/>
+    <child link="realsense_model_dummy_link"/>
+  </joint>
+</xacro:if>
   <!-- Links only needed in simulation, created by realsense software otherwise-->
 <xacro:if value="$(arg sim)">

File: unicorn_description/urdf/unicorn_target_backwards.urdf.xacro (robot description, xacro)
@@ -198,4 +198,20 @@
     <child link="realsense_link"/>
   </joint>
+<xacro:if value="$(arg sim)">
+  <link
+    name="realsense_model_dummy_link">
+    <visual>
+        <origin xyz="0 0 0" rpy="0 0 0"/>
+        <geometry>
+            <mesh filename="$(arg realsense_meshfile)" />
+        </geometry>
+      </visual>
+  </link>
+  <joint name="realsense_model_joint" type="fixed">
+    <origin xyz="$(arg real_rgb_xyz)" rpy="0 0 0"/>
+    <parent link="realsense_link"/>
+    <child link="realsense_model_dummy_link"/>
+  </joint>
+</xacro:if>
   <!-- Links only needed in simulation, created by realsense software otherwise-->
 <xacro:if value="$(arg sim)">
