Commit message: Update camera frames

File: unicorn_description/urdf/unicorn_sim.urdf.xacro (robot description, xacro)
@@ -53,19 +53,4 @@
   <link
     name="chassis_link">
-    <!--
-    <inertial>
-      <origin
-        xyz="0 0 0"
-        rpy="0 0 0" />
-      <mass
-        value="15" />
-      <inertia
-        ixx="1"
-        ixy="0"
-        ixz="3"
-        iyy="3"
-        iyz="3"
-        izz="1" />
-    </inertial>-->
     <visual>
       <origin
@@ -82,19 +67,4 @@
       </material>
     </visual>
-    <!--
-    <collision>
-      <origin
-        xyz="0 0 0"
-        rpy="0 0 0" />
-      <geometry>
-        <mesh
-          filename="package://unicorn_description/meshes/chassis_link.STL" />
-        <surface>
-         <friction>
-           <ode><mu>0.4</mu><mu2>0.4</mu2></ode>
-         </friction>
-      </surface>
-      </geometry>
-    </collision>-->
   </link>
 <!-- Lift -->
@@ -336,24 +306,54 @@
   </joint>
   <!-- Zed Camera -->
-    <stereo_camera frame_rgb="zed_camera" frame_depth="zed_depth" cameraName="zed"  topic="pointcloud" robot_namespace="$(arg robot_namespace)"/>
-  <link name="zed_camera">
-    <visual>
-      <origin xyz="0 0 0" rpy="0 0 0"/>
-      <geometry>
-          <mesh filename="$(arg zed_meshfile)"/>
-      </geometry>
-    </visual>
-  </link>
-  <link name="zed_depth"></link>
-    <joint name="zed_camera_rgb_joint" type="fixed">
-      <origin xyz="$(arg zed_xyz)" rpy="$(arg zed_rpy)"/>
-      <parent link="chassis_link"/>
-      <child link="zed_camera"/>
-    </joint>
+<!-- Camera Center -->
+    <joint name="zed_camera_center_joint" type="fixed">
+        <parent link="chassis_link"/>
+        <child link="zed_camera_center"/>
+        <origin xyz="$(arg zed_xyz)" rpy="0 0 0" />
+    </joint>
+    <link name="zed_camera_center">
+        <visual>
+            <origin xyz="0 0 0" rpy="0 0 0"/>
+            <geometry>
+                <mesh filename="$(arg zed_meshfile)" />
+            </geometry>
+        </visual>
+    </link>
+<!-- Left Camera -->
+    <joint name="zed_left_camera_joint" type="fixed">
+        <parent link="zed_camera_center"/>
+        <child link="zed_left_camera_frame"/>
+        <origin xyz="0 6 0" rpy="0 0 0" />
+    </joint>
+    <link name="zed_left_camera_frame" />
+    <joint name="zed_left_camera_optical_joint" type="fixed">
+        <origin xyz="0 0 0" rpy="-${M_PI/2} 0.0 -${M_PI/2}"/>
+        <parent link="zed_left_camera_frame"/>
+        <child link="zed_left_camera_optical_frame"/>
+    </joint>
+    <link name="zed_left_camera_optical_frame"/>
+<!-- Right Camera -->
+    <joint name="zed_right_camera_joint" type="fixed">
+        <parent link="zed_camera_center"/>
+        <child link="zed_right_camera_frame"/>
+        <origin xyz="0 -6 0" rpy="0 0 0" />
+    </joint>
+    <link name="zed_right_camera_frame" />
+    <joint name="zed_right_camera_optical_joint" type="fixed">
+        <origin xyz="0 0 0" rpy="-${M_PI/2} 0.0 -${M_PI/2}"/>
+        <parent link="zed_right_camera_frame"/>
+        <child link="zed_right_camera_optical_frame"/>
+    </joint>
+    <link name="zed_right_camera_optical_frame"/>
+<!---->
+<xacro:if value="$(arg sim)">
+    <stereo_camera frame_rgb="zed_camera_center" frame_depth="zed_depth_dummy_frame_sim_only" cameraName="zed"  topic="pointcloud" robot_namespace="$(arg robot_namespace)"/>
+    <link name="zed_depth_dummy_frame_sim_only"></link>
     <joint name="zed_camera_depth_joint" type="fixed">
       <origin xyz="0 0 0" rpy="${-pi/2} 0 ${-pi/2}"/>
-      <parent link="zed_camera"/>
-      <child link="zed_depth"/>
-    </joint>
+      <parent link="zed_camera_center"/>
+      <child link="zed_depth_dummy_frame_sim_only"/>
+    </joint>
+</xacro:if>
   <!-- realsense Camera -->
 <!-- Links only needed in simulation, created by realsense software otherwise-->
@@ -373,7 +373,8 @@
   </joint>
 <xacro:if value="$(arg sim)">
-  <stereo_camera frame_rgb="realsense_color_frame" frame_depth="realsense_depth_frame" cameraName="realsense" topic="pointcloud" robot_namespace="$(arg robot_namespace)"/>
+  <stereo_camera frame_rgb="realsense_color_frame" frame_depth="realsense_depth_dummy_frame_sim_only" cameraName="realsense" topic="pointcloud" robot_namespace="$(arg robot_namespace)"/>
   <link name="realsense_color_frame"> </link>
   <link name="realsense_depth_frame"></link>
+   <link name="realsense_depth_dummy_frame_sim_only"></link>
   <link
     name="realsense_depth_optical_frame">
@@ -391,4 +392,9 @@
     <parent link="realsense_link"/>
     <child link="realsense_depth_frame"/>
+  </joint>
+  <joint name="realsense_depth_dummy_joint" type="fixed">
+    <origin xyz="$(arg real_depth_xyz)" rpy="-${M_PI/2} 0.0 -${M_PI/2}"/>
+    <parent link="realsense_link"/>
+    <child link="realsense_depth_dummy_frame_sim_only"/>
   </joint>
   <joint name="realsense_optical_color_joint" type="fixed">

File: unicorn_description/urdf/unicorn_target.urdf.xacro (robot description, xacro)
@@ -212,24 +212,54 @@
   </joint>
   <!-- Zed Camera -->
-    <stereo_camera frame_rgb="zed_camera" frame_depth="zed_depth" cameraName="zed"  topic="pointcloud" robot_namespace="$(arg robot_namespace)"/>
-  <link name="zed_camera">
-    <visual>
-      <origin xyz="0 0 0" rpy="0 0 0"/>
-      <geometry>
-          <mesh filename="$(arg zed_meshfile)"/>
-      </geometry>
-    </visual>
-  </link>
-  <link name="zed_depth"></link>
-    <joint name="zed_camera_rgb_joint" type="fixed">
-      <origin xyz="$(arg zed_xyz)" rpy="$(arg zed_rpy)"/>
-      <parent link="base_link"/>
-      <child link="zed_camera"/>
-    </joint>
+<!-- Camera Center -->
+    <joint name="zed_camera_center_joint" type="fixed">
+        <parent link="chassis_link"/>
+        <child link="zed_camera_center"/>
+        <origin xyz="$(arg zed_xyz)" rpy="0 0 0" />
+    </joint>
+    <link name="zed_camera_center">
+        <visual>
+            <origin xyz="0 0 0" rpy="0 0 0"/>
+            <geometry>
+                <mesh filename="$(arg zed_meshfile)" />
+            </geometry>
+        </visual>
+    </link>
+<!-- Left Camera -->
+    <joint name="zed_left_camera_joint" type="fixed">
+        <parent link="zed_camera_center"/>
+        <child link="zed_left_camera_frame"/>
+        <origin xyz="0 6 0" rpy="0 0 0" />
+    </joint>
+    <link name="zed_left_camera_frame" />
+    <joint name="zed_left_camera_optical_joint" type="fixed">
+        <origin xyz="0 0 0" rpy="-${M_PI/2} 0.0 -${M_PI/2}"/>
+        <parent link="zed_left_camera_frame"/>
+        <child link="zed_left_camera_optical_frame"/>
+    </joint>
+    <link name="zed_left_camera_optical_frame"/>
+<!-- Right Camera -->
+    <joint name="zed_right_camera_joint" type="fixed">
+        <parent link="zed_camera_center"/>
+        <child link="zed_right_camera_frame"/>
+        <origin xyz="0 -6 0" rpy="0 0 0" />
+    </joint>
+    <link name="zed_right_camera_frame" />
+    <joint name="zed_right_camera_optical_joint" type="fixed">
+        <origin xyz="0 0 0" rpy="-${M_PI/2} 0.0 -${M_PI/2}"/>
+        <parent link="zed_right_camera_frame"/>
+        <child link="zed_right_camera_optical_frame"/>
+    </joint>
+    <link name="zed_right_camera_optical_frame"/>
+<!---->
+<xacro:if value="$(arg sim)">
+    <stereo_camera frame_rgb="zed_camera_center" frame_depth="zed_depth_dummy_frame_sim_only" cameraName="zed"  topic="pointcloud" robot_namespace="$(arg robot_namespace)"/>
+    <link name="zed_depth_dummy_frame_sim_only"></link>
     <joint name="zed_camera_depth_joint" type="fixed">
       <origin xyz="0 0 0" rpy="${-pi/2} 0 ${-pi/2}"/>
-      <parent link="zed_camera"/>
-      <child link="zed_depth"/>
-    </joint>
+      <parent link="zed_camera_center"/>
+      <child link="zed_depth_dummy_frame_sim_only"/>
+    </joint>
+</xacro:if>
   <!-- realsense Camera -->
 <!-- Links only needed in simulation, created by realsense software otherwise-->
@@ -249,7 +279,8 @@
   </joint>
 <xacro:if value="$(arg sim)">
-  <stereo_camera frame_rgb="realsense_color_frame" frame_depth="realsense_depth_frame" cameraName="realsense" topic="pointcloud" robot_namespace="$(arg robot_namespace)"/>
+  <stereo_camera frame_rgb="realsense_color_frame" frame_depth="realsense_depth_dummy_frame_sim_only" cameraName="realsense" topic="pointcloud" robot_namespace="$(arg robot_namespace)"/>
   <link name="realsense_color_frame"> </link>
   <link name="realsense_depth_frame"></link>
+   <link name="realsense_depth_dummy_frame_sim_only"></link>
   <link
     name="realsense_depth_optical_frame">
@@ -267,4 +298,9 @@
     <parent link="realsense_link"/>
     <child link="realsense_depth_frame"/>
+  </joint>
+  <joint name="realsense_depth_dummy_joint" type="fixed">
+    <origin xyz="$(arg real_depth_xyz)" rpy="-${M_PI/2} 0.0 -${M_PI/2}"/>
+    <parent link="realsense_link"/>
+    <child link="realsense_depth_dummy_frame_sim_only"/>
   </joint>
   <joint name="realsense_optical_color_joint" type="fixed">

File: unicorn_description/urdf/unicorn_target_backwards.urdf.xacro (robot description, xacro)
@@ -176,24 +176,54 @@
   </joint>
   <!-- Zed Camera -->
-    <stereo_camera frame_rgb="zed_camera" frame_depth="zed_depth" cameraName="zed"  topic="pointcloud" robot_namespace="$(arg robot_namespace)"/>
-  <link name="zed_camera">
-    <visual>
-      <origin xyz="0 0 0" rpy="0 0 0"/>
-      <geometry>
-          <mesh filename="$(arg zed_meshfile)"/>
-      </geometry>
-    </visual>
-  </link>
-  <link name="zed_depth"></link>
-    <joint name="zed_camera_rgb_joint" type="fixed">
-      <origin xyz="$(arg zed_xyz)" rpy="$(arg zed_rpy)"/>
-      <parent link="chassis_link"/>
-      <child link="zed_camera"/>
-    </joint>
+<!-- Camera Center -->
+    <joint name="zed_camera_center_joint" type="fixed">
+        <parent link="chassis_link"/>
+        <child link="zed_camera_center"/>
+        <origin xyz="$(arg zed_xyz)" rpy="0 0 0" />
+    </joint>
+    <link name="zed_camera_center">
+        <visual>
+            <origin xyz="0 0 0" rpy="0 0 0"/>
+            <geometry>
+                <mesh filename="$(arg zed_meshfile)" />
+            </geometry>
+        </visual>
+    </link>
+<!-- Left Camera -->
+    <joint name="zed_left_camera_joint" type="fixed">
+        <parent link="zed_camera_center"/>
+        <child link="zed_left_camera_frame"/>
+        <origin xyz="0 6 0" rpy="0 0 0" />
+    </joint>
+    <link name="zed_left_camera_frame" />
+    <joint name="zed_left_camera_optical_joint" type="fixed">
+        <origin xyz="0 0 0" rpy="-${M_PI/2} 0.0 -${M_PI/2}"/>
+        <parent link="zed_left_camera_frame"/>
+        <child link="zed_left_camera_optical_frame"/>
+    </joint>
+    <link name="zed_left_camera_optical_frame"/>
+<!-- Right Camera -->
+    <joint name="zed_right_camera_joint" type="fixed">
+        <parent link="zed_camera_center"/>
+        <child link="zed_right_camera_frame"/>
+        <origin xyz="0 -6 0" rpy="0 0 0" />
+    </joint>
+    <link name="zed_right_camera_frame" />
+    <joint name="zed_right_camera_optical_joint" type="fixed">
+        <origin xyz="0 0 0" rpy="-${M_PI/2} 0.0 -${M_PI/2}"/>
+        <parent link="zed_right_camera_frame"/>
+        <child link="zed_right_camera_optical_frame"/>
+    </joint>
+    <link name="zed_right_camera_optical_frame"/>
+<!---->
+<xacro:if value="$(arg sim)">
+    <stereo_camera frame_rgb="zed_camera_center" frame_depth="zed_depth_dummy_frame_sim_only" cameraName="zed"  topic="pointcloud" robot_namespace="$(arg robot_namespace)"/>
+    <link name="zed_depth_dummy_frame_sim_only"></link>
     <joint name="zed_camera_depth_joint" type="fixed">
       <origin xyz="0 0 0" rpy="${-pi/2} 0 ${-pi/2}"/>
-      <parent link="zed_camera"/>
-      <child link="zed_depth"/>
-    </joint>
+      <parent link="zed_camera_center"/>
+      <child link="zed_depth_dummy_frame_sim_only"/>
+    </joint>
+</xacro:if>
   <!-- realsense Camera -->
 <!-- Links only needed in simulation, created by realsense software otherwise-->
@@ -213,7 +243,8 @@
   </joint>
 <xacro:if value="$(arg sim)">
-  <stereo_camera frame_rgb="realsense_color_frame" frame_depth="realsense_depth_frame" cameraName="realsense" topic="pointcloud" robot_namespace="$(arg robot_namespace)"/>
+  <stereo_camera frame_rgb="realsense_color_frame" frame_depth="realsense_depth_dummy_frame_sim_only" cameraName="realsense" topic="pointcloud" robot_namespace="$(arg robot_namespace)"/>
   <link name="realsense_color_frame"> </link>
   <link name="realsense_depth_frame"></link>
+   <link name="realsense_depth_dummy_frame_sim_only"></link>
   <link
     name="realsense_depth_optical_frame">
@@ -231,4 +262,9 @@
     <parent link="realsense_link"/>
     <child link="realsense_depth_frame"/>
+  </joint>
+  <joint name="realsense_depth_dummy_joint" type="fixed">
+    <origin xyz="$(arg real_depth_xyz)" rpy="-${M_PI/2} 0.0 -${M_PI/2}"/>
+    <parent link="realsense_link"/>
+    <child link="realsense_depth_dummy_frame_sim_only"/>
   </joint>
   <joint name="realsense_optical_color_joint" type="fixed">

Commit message: Change Zed meas

File: unicorn_description/urdf/unicorn_sim.urdf.xacro (robot description, xacro)
@@ -324,5 +324,5 @@
         <parent link="zed_camera_center"/>
         <child link="zed_left_camera_frame"/>
-        <origin xyz="0 6 0" rpy="0 0 0" />
+        <origin xyz="0 0.06 0" rpy="0 0 0" />
     </joint>
     <link name="zed_left_camera_frame" />
@@ -337,5 +337,5 @@
         <parent link="zed_camera_center"/>
         <child link="zed_right_camera_frame"/>
-        <origin xyz="0 -6 0" rpy="0 0 0" />
+        <origin xyz="0 -0.06 0" rpy="0 0 0" />
     </joint>
     <link name="zed_right_camera_frame" />

File: unicorn_description/urdf/unicorn_target.urdf.xacro (robot description, xacro)
@@ -230,5 +230,5 @@
         <parent link="zed_camera_center"/>
         <child link="zed_left_camera_frame"/>
-        <origin xyz="0 6 0" rpy="0 0 0" />
+        <origin xyz="0 0.06 0" rpy="0 0 0" />
     </joint>
     <link name="zed_left_camera_frame" />
@@ -243,5 +243,5 @@
         <parent link="zed_camera_center"/>
         <child link="zed_right_camera_frame"/>
-        <origin xyz="0 -6 0" rpy="0 0 0" />
+        <origin xyz="0 -0.06 0" rpy="0 0 0" />
     </joint>
     <link name="zed_right_camera_frame" />

File: unicorn_description/urdf/unicorn_target_backwards.urdf.xacro (robot description, xacro)
@@ -194,5 +194,5 @@
         <parent link="zed_camera_center"/>
         <child link="zed_left_camera_frame"/>
-        <origin xyz="0 6 0" rpy="0 0 0" />
+        <origin xyz="0 0.06 0" rpy="0 0 0" />
     </joint>
     <link name="zed_left_camera_frame" />
@@ -207,5 +207,5 @@
         <parent link="zed_camera_center"/>
         <child link="zed_right_camera_frame"/>
-        <origin xyz="0 -6 0" rpy="0 0 0" />
+        <origin xyz="0 -0.06 0" rpy="0 0 0" />
     </joint>
     <link name="zed_right_camera_frame" />

Commit message: Started adding joint controll motors

File: unicorn_description/urdf/unicorn_sim.urdf.xacro (robot description, xacro)
@@ -219,4 +219,12 @@
     </collision>
   </link>
+  <joint name="lift_horizontal_joint" type="prismatic">
+    <parent  link="lift_link" />
+    <child  link="lift_horizontal_link" />
+    <origin xyz="0.05 0 0.137" rpy="${M_PI2} 0 ${-M_PI2}" />
+    <axis xyz="0 0.0024714 -1" rpy="0 0 0"  />
+    <limit lower="0.17" upper="0" effort="100" velocity="100" />
+    <joint_properties damping="1000" friction="0.5" />
+  </joint>
   <joint
     name="lift_vertical_joint"
@@ -238,14 +246,4 @@
       <joint_properties damping="10" friction="0.5" />
   </joint>
-  <gazebo reference="lift_vertical_joint">
-      <mu1 value="10000.0" />
-      <mu2 value="10000.0" />
-      <kp value="100000.0" />
-      <kd value="10000.0" />
-      <dampingFactor value="0.5" />
-      <fdir1 value="1 0 0" />
-      <material>Gazebo/Black</material>
-      <turnGravityOff>false</turnGravityOff>
-  </gazebo>
   <wheel fb="back" lr="left" parent="lift_link"  translateY="0.24" translateX="0" translateZ="0.1225" wheel_radius="0.1225" wheel_height="0.032" flip="1"/>
   <wheel fb="back" lr="right" parent="lift_link" translateY="-0.24" translateX="0 " translateZ="0.1225" wheel_radius="0.1225" wheel_height="0.032" flip="1"/>
@@ -371,13 +369,14 @@
   </joint>
 </xacro:if>
-  <joint name="lift_horizontal_joint" type="prismatic">
-    <parent  link="lift_link" />
-    <child  link="lift_horizontal_link" />
-    <origin xyz="0.05 0 0.137" rpy="${M_PI2} 0 ${-M_PI2}" />
-    <axis xyz="0 0.0024714 -1" rpy="0 0 0"  />
-    <limit lower="0.17" upper="0" effort="100" velocity="100" />
-    <joint_properties damping="1000" friction="0.5" />
-  </joint>
-<<<<<<< HEAD
+  <gazebo reference="lift_vertical_joint">
+      <mu1 value="10000.0" />
+      <mu2 value="10000.0" />
+      <kp value="100000.0" />
+      <kd value="10000.0" />
+      <dampingFactor value="0.5" />
+      <fdir1 value="1 0 0" />
+      <material>Gazebo/Black</material>
+      <turnGravityOff>false</turnGravityOff>
+  </gazebo>
   <gazebo reference="lift_horizontal_joint">
       <mu1 value="10000.0" />
@@ -389,40 +388,30 @@
       <material>Gazebo/Black</material>
       <turnGravityOff>false</turnGravityOff>
-=======
-<xacro:if value="$(arg sim)">
-  <!-- Fake UWB -->
-  <gazebo>
-    <plugin name="p3d_base_controller" filename="libgazebo_ros_p3d.so">
-        <alwaysOn>true</alwaysOn>
-        <updateRate>50.0</updateRate>
-        <bodyName>chassis_link</bodyName>
-        <topicName>uwb/pose</topicName>
-        <gaussianNoise>0.1</gaussianNoise>
-        <frameName>map</frameName>
-        <xyzOffset>0 0 0</xyzOffset>
-        <rpyOffset>0 0 0</rpyOffset>
-      </plugin>
->>>>>>> c6a34eb1ea5167d43927d40b71a6c3829b7e0557
   </gazebo>
-  <transmission name="lift_horizontal_joint_trans">
+  <transmission name="lift_h_trans">
       <type>transmission_interface/SimpleTransmission</type>
       <joint name="lift_horizontal_joint">
-        <hardwareInterface>hardware_interface/EffortJointInterface</hardwareInterface>
+        <hardwareInterface>EffortJointInterface</hardwareInterface>
       </joint>
-      <actuator name="lift_horizontal_joint_motor">
-        <hardwareInterface>hardware_interface/EffortJointInterface</hardwareInterface>
+      <actuator name="lift_h_motor">
+        <hardwareInterface>EffortJointInterface</hardwareInterface>
         <mechanicalReduction>5</mechanicalReduction>
       </actuator>
   </transmission>
-  <transmission name="lift_vertical_joint_trans">
+  <transmission name="lift_v_trans">
       <type>transmission_interface/SimpleTransmission</type>
       <joint name="lift_vertical_joint">
-        <hardwareInterface>hardware_interface/EffortJointInterface</hardwareInterface>
+        <hardwareInterface>EffortJointInterface</hardwareInterface>
       </joint>
-      <actuator name="lift_vertical_joint_motor">
-        <hardwareInterface>hardware_interface/EffortJointInterface</hardwareInterface>
+      <actuator name="lift_v_motor">
+        <hardwareInterface>EffortJointInterface</hardwareInterface>
         <mechanicalReduction>5</mechanicalReduction>
       </actuator>
   </transmission>
+<gazebo>
+  <plugin name="gazebo_ros_control" filename="libgazebo_ros_control.so">
+    <robotNamespace>/unicorn</robotNamespace>
+  </plugin>
+</gazebo>
 <xacro:if value="$(arg sim)">
   <!-- GAZEBO STUFF -->
@@ -489,5 +478,7 @@
     </plugin>
     <!-- Joint controll plugin -->
-    <plugin name="gazebo_ros_control" filename="libgazebo_ros_control.so" />
+    <plugin name="gazebo_ros_control" filename="libgazebo_ros_control.so">
+      <robotNamespace>/unicorn</robotNamespace>
+    </plugin>
     <!-- gazebo wheel encoders -->
     <plugin name="am_gazebo_wheelencoder" filename="libam_gazebo_wheelencoder.so">

Commit message: Changed sim joint controller type and pid

File: unicorn_description/urdf/unicorn_sim.urdf.xacro (robot description, xacro)
@@ -224,6 +224,6 @@
     <origin xyz="0.05 0 0.137" rpy="${M_PI2} 0 ${-M_PI2}" />
     <axis xyz="0 0.0024714 -1" rpy="0 0 0"  />
-    <limit lower="0.17" upper="0" effort="100" velocity="100" />
-    <joint_properties damping="1000" friction="0.5" />
+    <limit lower="0.17" upper="0" effort="200" velocity="50" />
+    <joint_properties damping="1000" friction="100" />
   </joint>
   <joint
@@ -243,6 +243,6 @@
       upper="0.16"
       effort="100"
-      velocity="0.4" />
-      <joint_properties damping="10" friction="0.5" />
+      velocity="50" />
+      <joint_properties damping="1000" friction="10" />
   </joint>
   <wheel fb="back" lr="left" parent="lift_link"  translateY="0.24" translateX="0" translateZ="0.1225" wheel_radius="0.1225" wheel_height="0.032" flip="1"/>
@@ -374,5 +374,5 @@
       <kp value="100000.0" />
       <kd value="10000.0" />
-      <dampingFactor value="0.5" />
+      <dampingFactor value="10" />
       <fdir1 value="1 0 0" />
       <material>Gazebo/Black</material>
@@ -384,5 +384,5 @@
       <kp value="100000.0" />
       <kd value="10000.0" />
-      <dampingFactor value="0.5" />
+      <dampingFactor value="20" />
       <fdir1 value="1 0 0" />
       <material>Gazebo/Black</material>
@@ -396,5 +396,5 @@
       <actuator name="lift_h_motor">
         <hardwareInterface>EffortJointInterface</hardwareInterface>
-        <mechanicalReduction>5</mechanicalReduction>
+        <mechanicalReduction>500</mechanicalReduction>
       </actuator>
   </transmission>
@@ -406,11 +406,8 @@
       <actuator name="lift_v_motor">
         <hardwareInterface>EffortJointInterface</hardwareInterface>
-        <mechanicalReduction>5</mechanicalReduction>
+        <mechanicalReduction>500</mechanicalReduction>
       </actuator>
   </transmission>
 <gazebo>
-  <plugin name="gazebo_ros_control" filename="libgazebo_ros_control.so">
-    <robotNamespace>/unicorn</robotNamespace>
-  </plugin>
 </gazebo>
 <xacro:if value="$(arg sim)">
