Commit message: Changed Sim lift joint params

File: unicorn_description/urdf/unicorn_sim.urdf.xacro (robot description, xacro)
@@ -53,4 +53,18 @@
   <link
     name="chassis_link">
+    <inertial>
+      <origin
+        xyz="0 0 0"
+        rpy="0 0 0" />
+      <mass
+        value="15" />
+      <inertia
+        ixx="1"
+        ixy="0"
+        ixz="3"
+        iyy="3"
+        iyz="3"
+        izz="1" />
+    </inertial>
     <visual>
       <origin
@@ -67,4 +81,21 @@
       </material>
     </visual>
+    <surface>
+      <friction>
+        <ode>
+          <mu>0.8</mu>
+          <mu2>0.8</mu2>
+        </ode>
+      </friction>
+    </surface>
+  <collision>
+    <origin
+      xyz="0 0 0"
+      rpy="0 0 0" />
+    <geometry>
+      <mesh
+        filename="package://unicorn_description/meshes/chassis_link.STL" />
+    </geometry>
+  </collision>
   </link>
 <!-- Lift -->
@@ -102,6 +133,6 @@
         <friction>
           <ode>
-            <mu>0.5</mu>
-            <mu2>0.5</mu2>
+            <mu>0.8</mu>
+            <mu2>0.8</mu2>
           </ode>
         </friction>
@@ -150,6 +181,6 @@
         <friction>
           <ode>
-            <mu>0.5</mu>
-            <mu2>0.5</mu2>
+            <mu>0.8</mu>
+            <mu2>0.8</mu2>
           </ode>
         </friction>
@@ -209,4 +240,12 @@
       </material>
     </visual>
+    <surface>
+      <friction>
+        <ode>
+          <mu>0.8</mu>
+          <mu2>0.8</mu2>
+        </ode>
+      </friction>
+    </surface>
     <collision>
       <origin
@@ -223,26 +262,15 @@
     <child  link="lift_horizontal_link" />
     <origin xyz="0.05 0 0.137" rpy="${M_PI2} 0 ${-M_PI2}" />
-    <axis xyz="0 0.0024714 -1" rpy="0 0 0"  />
-    <limit lower="0.17" upper="0" effort="200" velocity="50" />
-    <joint_properties damping="1000" friction="100" />
-  </joint>
-  <joint
-    name="lift_vertical_joint"
-    type="prismatic">
-    <origin
-      xyz="0 -0.16 0"
-      rpy="0 0 0" />
-    <parent
-      link="lift_horizontal_link" />
-    <child
-      link="lift_vertical_link" />
-    <axis
-      xyz="0 1 0" />
-    <limit
-      lower="0"
-      upper="0.16"
-      effort="100"
-      velocity="50" />
-      <joint_properties damping="1000" friction="10" />
+    <axis xyz="0 0 -1" rpy="0 0 0"  />
+    <limit lower="0.17" upper="0" effort="100" velocity="0" />
+    <joint_properties damping="1000" friction="1000" />
+  </joint>
+  <joint name="lift_vertical_joint" type="prismatic">
+    <origin xyz="0 -0.16 0" rpy="0 0 0" />
+    <parent link="lift_horizontal_link" />
+    <child link="lift_vertical_link" />
+    <axis xyz="0 1 0" />
+    <limit lower="0" upper="0.16" effort="50" velocity="0" />
+    <joint_properties damping="1000" friction="1000" />
   </joint>
   <wheel fb="back" lr="left" parent="lift_link"  translateY="0.24" translateX="0" translateZ="0.1225" wheel_radius="0.1225" wheel_height="0.032" flip="1"/>
@@ -374,8 +402,8 @@
       <kp value="100000.0" />
       <kd value="10000.0" />
-      <dampingFactor value="10" />
+      <dampingFactor value="100" />
       <fdir1 value="1 0 0" />
       <material>Gazebo/Black</material>
-      <turnGravityOff>false</turnGravityOff>
+      <turnGravityOff>true</turnGravityOff>
   </gazebo>
   <gazebo reference="lift_horizontal_joint">
@@ -392,8 +420,8 @@
       <type>transmission_interface/SimpleTransmission</type>
       <joint name="lift_horizontal_joint">
-        <hardwareInterface>EffortJointInterface</hardwareInterface>
+        <hardwareInterface>hardware_interface/EffortJointInterface</hardwareInterface>
       </joint>
       <actuator name="lift_h_motor">
-        <hardwareInterface>EffortJointInterface</hardwareInterface>
+        <hardwareInterface>hardware_interface/EffortJointInterface</hardwareInterface>
         <mechanicalReduction>500</mechanicalReduction>
       </actuator>
@@ -402,8 +430,8 @@
       <type>transmission_interface/SimpleTransmission</type>
       <joint name="lift_vertical_joint">
-        <hardwareInterface>EffortJointInterface</hardwareInterface>
+        <hardwareInterface>hardware_interface/EffortJointInterface</hardwareInterface>
       </joint>
       <actuator name="lift_v_motor">
-        <hardwareInterface>EffortJointInterface</hardwareInterface>
+        <hardwareInterface>hardware_interface/EffortJointInterface</hardwareInterface>
         <mechanicalReduction>500</mechanicalReduction>
       </actuator>

Commit message: Somewhat working sim lift controllers and urdf params

File: unicorn_description/urdf/unicorn_sim.urdf.xacro (robot description, xacro)
@@ -264,5 +264,5 @@
     <axis xyz="0 0 -1" rpy="0 0 0"  />
     <limit lower="0.17" upper="0" effort="100" velocity="0" />
-    <joint_properties damping="1000" friction="1000" />
+    <joint_properties damping="1000" friction="100" />
   </joint>
   <joint name="lift_vertical_joint" type="prismatic">
@@ -271,6 +271,6 @@
     <child link="lift_vertical_link" />
     <axis xyz="0 1 0" />
-    <limit lower="0" upper="0.16" effort="50" velocity="0" />
-    <joint_properties damping="1000" friction="1000" />
+    <limit lower="0" upper="0.16" effort="100" velocity="0" />
+    <joint_properties damping="1000" friction="100" />
   </joint>
   <wheel fb="back" lr="left" parent="lift_link"  translateY="0.24" translateX="0" translateZ="0.1225" wheel_radius="0.1225" wheel_height="0.032" flip="1"/>
@@ -402,8 +402,8 @@
       <kp value="100000.0" />
       <kd value="10000.0" />
-      <dampingFactor value="100" />
+      <dampingFactor value="50" />
       <fdir1 value="1 0 0" />
       <material>Gazebo/Black</material>
-      <turnGravityOff>true</turnGravityOff>
+      <turnGravityOff>false</turnGravityOff>
   </gazebo>
   <gazebo reference="lift_horizontal_joint">

Commit message: Added color to gazebo model

File: unicorn_description/urdf/unicorn_sim.urdf.xacro (robot description, xacro)
@@ -258,5 +258,5 @@
     </collision>
   </link>
-  <joint name="lift_horizontal_joint" type="prismatic">
+  <joint name="lift_horizontal_joint" type="fixed"> <!-- type="prismatic" -->
     <parent  link="lift_link" />
     <child  link="lift_horizontal_link" />
@@ -266,5 +266,5 @@
     <joint_properties damping="10000" friction="1000" />
   </joint>
-  <joint name="lift_vertical_joint" type="prismatic">
+  <joint name="lift_vertical_joint" type="fixed"> <!-- type="prismatic" -->
     <origin xyz="0 -0.16 0" rpy="0 0 0" />
     <parent link="lift_horizontal_link" />
@@ -397,24 +397,60 @@
   </joint>
 </xacro:if>
+<!-- Set Color for nodes -->
+    <gazebo reference="chassis_link">
+      <material>Gazebo/Grey</material>
+      <turnGravityOff>false</turnGravityOff>
+    </gazebo>
+    <gazebo reference="lift_link">
+      <material>Gazebo/Grey</material>
+      <turnGravityOff>false</turnGravityOff>
+    </gazebo>
+    <gazebo reference="base_laser">
+      <material>Gazebo/RedBright</material>
+      <turnGravityOff>false</turnGravityOff>
+    </gazebo>
+    <gazebo reference="rear_laser">
+      <material>Gazebo/DarkGrey</material>
+      <turnGravityOff>false</turnGravityOff>
+    </gazebo>
+    <gazebo reference="zed_camera_center">
+      <material>Gazebo/FlatBlack</material>
+      <turnGravityOff>false</turnGravityOff>
+    </gazebo>
+    <gazebo reference="realsense_link">
+      <material>Gazebo/Grey</material>
+      <turnGravityOff>false</turnGravityOff>
+    </gazebo>
+    <gazebo reference="lift_vertical_link">
+      <material>Gazebo/White</material>
+      <turnGravityOff>false</turnGravityOff>
+    </gazebo>
+    <gazebo reference="lift_horizontal_link">
+      <material>Gazebo/White</material>
+      <turnGravityOff>false</turnGravityOff>
+    </gazebo>
+<!-- Used for Simulating Lift movment, removed due to problems with controllers -->
+ <!--
   <gazebo reference="lift_vertical_joint">
-      <mu1 value="10000.0" />
-      <mu2 value="10000.0" />
+      <mu1 value="0.8" />
+      <mu2 value="0.8" />
       <kp value="100000.0" />
       <kd value="10000.0" />
-      <dampingFactor value="50" />
+      <dampingFactor value="0.9" />
       <fdir1 value="1 0 0" />
-      <material>Gazebo/Black</material>
+      <material>Gazebo/Gold</material>
       <turnGravityOff>false</turnGravityOff>
   </gazebo>
   <gazebo reference="lift_horizontal_joint">
-      <mu1 value="10000.0" />
-      <mu2 value="10000.0" />
+      <mu1 value="0.8" />
+      <mu2 value="0.8" />
       <kp value="100000.0" />
       <kd value="10000.0" />
-      <dampingFactor value="100" />
+      <dampingFactor value="0.9" />
       <fdir1 value="1 0 0" />
-      <material>Gazebo/Black</material>
+      <material>Gazebo/Grey</material>
       <turnGravityOff>false</turnGravityOff>
   </gazebo>
+-->
   <transmission name="lift_h_trans">
       <type>transmission_interface/SimpleTransmission</type>
