Commit message: Added Base link for simulator so that same frame standard can be used for both simulator and robot

File: unicorn_description/urdf/unicorn_sim.urdf.xacro (robot description, xacro)
@@ -3,4 +3,7 @@
   <xacro:arg name="robot_namespace" default="/" />
   <xacro:arg name="sim" default="true" />
+  <!-- Define Constants -->
+  <xacro:property name="M_PI" value="3.1415926535897931" />
+  <xacro:property name="M_PI2" value="1.57079632679" />
     <!-- Swivel wheel -->
   <xacro:include filename="$(find unicorn_description)/urdf/swivel_wheel.urdf.xacro" />
@@ -11,17 +14,17 @@
    <!-- lidar pack-->
   <xacro:include filename="$(find unicorn_description)/urdf/lidar_gazebo.urdf.xacro" />
-  <xacro:property name="M_PI" value="3.1415926535897931" />
-  <xacro:property name="M_PI2" value="1.57079632679" />
-  <!-- base --><!--
-    <xacro:property name="base_x_size" value="0.72" />
-  <xacro:property name="base_y_size" value="0.55" />
-  <xacro:property name="base_z_size" value="0.6" />
-  <xacro:property name="base_mass" value="21.446" /> 21.446 in kg-->
-    <!-- Main Body-base -->
+  <!-- Main Body-base -->
   <xacro:property name="base_x_size" value="0.72" />
   <xacro:property name="base_y_size" value="0.55" />
   <xacro:property name="base_z_size" value="0.23" />
   <xacro:property name="base_mass" value="15" /> <!-- in kg-->
-    <!--Inertial macros for the box and cylinder. Units are kg*m^2-->
+  <!-- Base Link Rotation -->
+  <xacro:if value="$(arg sim)">
+    <xacro:arg name="base_link_rpy" default="0 0 0" />
+  </xacro:if>
+  <xacro:unless value="$(arg sim)">
+    <xacro:arg name="base_link_rpy" default="0 0 ${M_PI}" />
+  </xacro:unless>
+  <!--Inertial macros for the box and cylinder. Units are kg*m^2-->
   <xacro:macro name="box_inertia" params="m x y z">
     <inertia ixx="${m*(y*y+z*z)/12}" ixy="0" ixz="0"
@@ -33,5 +36,5 @@
   <xacro:arg name="laser_rpy" default="0 0 0" />
   <xacro:arg name="frontlidar_meshfile" default="package://unicorn_description/meshes/base_laser.STL" />
-<!-- Rear Lidar  -->
+  <!-- Rear Lidar  -->
   <xacro:arg name="rear_laser_xyz" default="-0.42145 -0.00645 0.28652" />
   <xacro:arg name="rear_laser_rpy" default="0 0 ${M_PI}" />
@@ -49,34 +52,25 @@
   <xacro:arg name="real_depth_rpy" default="${-M_PI2} 0 ${-M_PI2}" />
   <xacro:arg name="realsense_meshfile" default="package://unicorn_description/meshes/real_sense.STL" />
-  <!-- Lift -->
  <!-- Main Body-base -->
+  <link name="base_link" />
+  <joint name="chassis_joint" type="fixed">
+    <parent link="base_link"/>
+    <child link="chassis_link" />
+  <origin xyz="0 0.0 0" rpy="$(arg base_link_rpy)" />
+  </joint>
   <link
     name="chassis_link">
     <inertial>
-      <origin
-        xyz="0 0 0"
-        rpy="0 0 0" />
-      <mass
-        value="15" />
-      <inertia
-        ixx="1"
-        ixy="0"
-        ixz="3"
-        iyy="3"
-        iyz="3"
-        izz="1" />
+      <origin xyz="0 0 0" rpy="0 0 0" />
+      <mass value="15" />
+      <inertia ixx="1" ixy="0" ixz="3" iyy="3" iyz="3" izz="1" />
     </inertial>
     <visual>
-      <origin
-        xyz="0 0 0"
-        rpy="0 0 0" />
-      <geometry>
-        <mesh
-          filename="package://unicorn_description/meshes/chassis_link.STL" />
-      </geometry>
-      <material
-        name="">
-        <color
-          rgba="0.792156862745098 0.819607843137255 0.933333333333333 1" />
+      <origin xyz="0 0 0" rpy="0 0 0" />
+      <geometry>
+        <mesh filename="package://unicorn_description/meshes/chassis_link.STL" />
+      </geometry>
+      <material name="">
+        <color rgba="0.792156862745098 0.819607843137255 0.933333333333333 1" />
       </material>
     </visual>
@@ -90,10 +84,7 @@
     </surface>
   <collision>
-    <origin
-      xyz="0 0 0"
-      rpy="0 0 0" />
+    <origin xyz="0 0 0" rpy="0 0 0" />
     <geometry>
-      <mesh
-        filename="package://unicorn_description/meshes/chassis_link.STL" />
+      <mesh filename="package://unicorn_description/meshes/chassis_link.STL" />
     </geometry>
   </collision>
@@ -103,29 +94,15 @@
     name="lift_link">
     <inertial>
-      <origin
-        xyz="0 0 0"
-        rpy="0 0 0" />
-      <mass
-        value="10" />
-      <inertia
-        ixx="1"
-        ixy="0"
-        ixz="3"
-        iyy="3"
-        iyz="3"
-        izz="1" />
-    </inertial>-
+      <origin xyz="0 0 0" rpy="0 0 0" />
+      <mass value="10" />
+      <inertia ixx="1" ixy="0" ixz="3" iyy="3" iyz="3" izz="1" />
+    </inertial>
     <visual>
-      <origin
-        xyz="0 0 0"
-        rpy="0 0 ${M_PI}" />
-      <geometry>
-        <mesh
-          filename="package://unicorn_description/meshes/lift_link.STL" />
-      </geometry>
-      <material
-        name="">
-        <color
-          rgba="0.752941176470588 0.752941176470588 0.752941176470588 1" />
+      <origin xyz="0 0 0" rpy="0 0 ${M_PI}" />
+      <geometry>
+        <mesh filename="package://unicorn_description/meshes/lift_link.STL" />
+      </geometry>
+      <material name="">
+        <color rgba="0.752941176470588 0.752941176470588 0.752941176470588 1" />
       </material>
     </visual>
@@ -139,25 +116,15 @@
       </surface>
     <collision>
-      <origin
-        xyz="0 0 0"
-        rpy="0 0 ${M_PI}" />
-      <geometry>
-        <mesh
-          filename="package://unicorn_description/meshes/lift_link.STL" />
+      <origin xyz="0 0 0" rpy="0 0 ${M_PI}" />
+      <geometry>
+        <mesh filename="package://unicorn_description/meshes/lift_link.STL" />
       </geometry>
     </collision>
   </link>
-  <joint
-    name="lift_joint"
-    type="fixed">
-    <origin
-      xyz="0 0 0"
-      rpy="0 0 ${M_PI}" />
-    <parent
-      link="chassis_link" />
-    <child
-      link="lift_link" />
-    <axis
-      xyz="0 0 0" />
+  <joint name="lift_joint" type="fixed">
+    <origin xyz="0 0 0" rpy="0 0 ${M_PI}" />
+    <parent link="chassis_link" />
+    <child link="lift_link" />
+    <axis xyz="0 0 0" />
     <joint_properties damping="1" friction="0.5" />
   </joint>
@@ -166,15 +133,10 @@
     name="lift_horizontal_link">
     <visual>
-      <origin
-        xyz="0 0 0"
-        rpy="0 0 0" />
-      <geometry>
-        <mesh
-          filename="package://unicorn_description/meshes/lift_horizontal_link.STL" />
-      </geometry>
-      <material
-        name="">
-        <color
-          rgba="0.898039215686275 0.917647058823529 0.929411764705882 1" />
+      <origin xyz="0 0 0" rpy="0 0 0" />
+      <geometry>
+        <mesh filename="package://unicorn_description/meshes/lift_horizontal_link.STL" />
+      </geometry>
+      <material name="">
+        <color rgba="0.898039215686275 0.917647058823529 0.929411764705882 1" />
       </material>
     </visual>
@@ -188,25 +150,13 @@
       </surface>
     <collision>
-      <origin
-        xyz="0 0 0"
-        rpy="0 0 0" />
-      <geometry>
-        <mesh
-          filename="package://unicorn_description/meshes/lift_horizontal_link.STL" />
+      <origin xyz="0 0 0" rpy="0 0 0" />
+      <geometry>
+        <mesh filename="package://unicorn_description/meshes/lift_horizontal_link.STL" />
       </geometry>
     </collision>
     <inertial>
-      <origin
-        xyz="0 0 0"
-        rpy="0 0 0" />
-      <mass
-        value="1.50791731426345" />
-      <inertia
-        ixx="0.00998369504134607"
-        ixy="1.05918049885466E-06"
-        ixz="3.20101525315815E-06"
-        iyy="0.0148024039374132"
-        iyz="1.02762580499191E-05"
-        izz="0.0197484509547163" />
+      <origin xyz="0 0 0" rpy="0 0 0" />
+      <mass value="1.50791731426345" />
+      <inertia ixx="0.00998369504134607" ixy="1.05918049885466E-06" ixz="3.20101525315815E-06" iyy="0.0148024039374132" iyz="1.02762580499191E-05" izz="0.0197484509547163" />
     </inertial>
   </link>
@@ -214,29 +164,15 @@
     name="lift_vertical_link">
     <inertial>
-      <origin
-        xyz="-0.0046764 0.62992 -0.22573"
-        rpy="0 0 0" />
-      <mass
-        value="0.61742" />
-      <inertia
-        ixx="0.00029455"
-        ixy="9.8754E-10"
-        ixz="2.0681E-19"
-        iyy="0.00411"
-        iyz="3.0422E-05"
-        izz="0.0043679" />
+      <origin xyz="-0.0046764 0.62992 -0.22573" rpy="0 0 0" />
+      <mass value="0.61742" />
+      <inertia ixx="0.00029455" ixy="9.8754E-10" ixz="2.0681E-19" iyy="0.00411" iyz="3.0422E-05" izz="0.0043679" />
     </inertial>
     <visual>
-      <origin
-        xyz="0 0 0"
-        rpy="0 0 0" />
-      <geometry>
-        <mesh
-          filename="package://unicorn_description/meshes/lift_vertical_link.STL" />
-      </geometry>
-      <material
-        name="">
-        <color
-          rgba="1 0.69412 0.27843 1" />
+      <origin xyz="0 0 0" rpy="0 0 0" />
+      <geometry>
+        <mesh filename="package://unicorn_description/meshes/lift_vertical_link.STL" />
+      </geometry>
+      <material name="">
+        <color rgba="1 0.69412 0.27843 1" />
       </material>
     </visual>
@@ -250,10 +186,7 @@
     </surface>
     <collision>
-      <origin
-        xyz="0 0 0"
-        rpy="0 0 0" />
-      <geometry>
-        <mesh
-          filename="package://unicorn_description/meshes/lift_vertical_link.STL" />
+      <origin xyz="0 0 0" rpy="0 0 0" />
+      <geometry>
+        <mesh filename="package://unicorn_description/meshes/lift_vertical_link.STL" />
       </geometry>
     </collision>
@@ -275,10 +208,31 @@
     <joint_properties damping="1000" friction="1000" />
   </joint>
-  <wheel fb="back" lr="left" parent="lift_link"  translateY="0.24" translateX="0" translateZ="0.1225" wheel_radius="0.1225" wheel_height="0.032" flip="1"/>
-  <wheel fb="back" lr="right" parent="lift_link" translateY="-0.24" translateX="0 " translateZ="0.1225" wheel_radius="0.1225" wheel_height="0.032" flip="1"/>
-  <!-- others wheels -->
+<!-- Front Wheels -->
+<!-- Dummy Link for simulation, used to Correct back motion from HRP drivers -->
+  <xacro:if value="$(arg sim)">
+    <link name="dummy_wheel_link" >
+      <inertial>
+        <origin xyz="0 0 0" rpy="0 0 0" />
+        <mass value="0.01" />
+        <box_inertia  m="${5*0.01}" x="${base_x_size}" y="${base_y_size}" z="${base_z_size}"/>
+      </inertial>
+    </link>
+    <joint name="dummy_wheel_joint" type="fixed">
+      <origin xyz="0 0.0 0" rpy="0 0 ${M_PI}" />
+      <parent link="chassis_link"/>
+      <child link="dummy_wheel_link"/>
+    </joint>
+    <wheel fb="back" lr="left" parent="dummy_wheel_link"  translateY="0.24" translateX="0" translateZ="0.1225" wheel_radius="0.1225" wheel_height="0.032" flip="1"/>
+    <wheel fb="back" lr="right" parent="dummy_wheel_link" translateY="-0.24" translateX="0 " translateZ="0.1225" wheel_radius="0.1225" wheel_height="0.032" flip="1"/>
+  </xacro:if>
+  <!-- For real Platform -->
+  <xacro:unless value="$(arg sim)">
+    <wheel fb="back" lr="left" parent="chassis_link"  translateY="0.24" translateX="0" translateZ="0.1225" wheel_radius="0.1225" wheel_height="0.032" flip="1"/>
+    <wheel fb="back" lr="right" parent="chassis_link" translateY="-0.24" translateX="0 " translateZ="0.1225" wheel_radius="0.1225" wheel_height="0.032" flip="1"/>
+  </xacro:unless>
+  <!-- Swivel back wheels - Should be changed to omniwheels-->
   <swivel_wheel fb="front" lr="left" parent="chassis_link" translateY="0.16" translateX="-0.355" translateZ="0.1531" wheel_radius="0.05" wheel_height="0.05" flip="0"/>
   <swivel_wheel fb="front" lr="right" parent="chassis_link" translateY="-0.16" translateX="-0.355" translateZ="0.1531" wheel_radius="0.05" wheel_height="0.05" flip="0"/>
- <!-- Front Lidar -->
+  <!-- Front Lidar -->
   <lidar_gazebo frame="base_laser" topic="frontLidar/scan" simulation="$(arg sim)" sample_size="800" min_angle="-2.35619" max_angle="2.35619" robot_namespace="$(arg robot_namespace)" filename="$(arg frontlidar_meshfile)" />
   <joint name="laser_mount_joint" type="fixed">
@@ -295,56 +249,52 @@
   </joint>
   <!-- Zed Camera -->
-<!-- Camera Center -->
-    <joint name="zed_camera_center_joint" type="fixed">
-        <parent link="chassis_link"/>
-        <child link="zed_camera_center"/>
-        <origin xyz="$(arg zed_xyz)" rpy="0 0 0" />
-    </joint>
-    <link name="zed_camera_center">
-        <visual>
-            <origin xyz="0 0 0" rpy="0 0 0"/>
-            <geometry>
-                <mesh filename="$(arg zed_meshfile)" />
-            </geometry>
-        </visual>
-    </link>
-<!-- Left Camera -->
-    <joint name="zed_left_camera_joint" type="fixed">
+  <link name="zed_camera_center">
+      <visual>
+          <origin xyz="0 0 0" rpy="0 0 0"/>
+          <geometry>
+              <mesh filename="$(arg zed_meshfile)" />
+          </geometry>
+      </visual>
+  </link>
+  <link name="zed_right_camera_frame" />
+  <link name="zed_right_camera_optical_frame"/>
+  <link name="zed_left_camera_optical_frame"/>
+  <link name="zed_left_camera_frame" />
+  <joint name="zed_camera_center_joint" type="fixed">
+      <parent link="chassis_link"/>
+      <child link="zed_camera_center"/>
+      <origin xyz="$(arg zed_xyz)" rpy="0 0 0" />
+  </joint>
+  <joint name="zed_left_camera_joint" type="fixed">
+      <parent link="zed_camera_center"/>
+      <child link="zed_left_camera_frame"/>
+      <origin xyz="0 0.06 0" rpy="0 0 0" />
+  </joint>
+  <joint name="zed_left_camera_optical_joint" type="fixed">
+      <origin xyz="0 0 0" rpy="-${M_PI/2} 0.0 -${M_PI/2}"/>
+      <parent link="zed_left_camera_frame"/>
+      <child link="zed_left_camera_optical_frame"/>
+  </joint>
+  <joint name="zed_right_camera_joint" type="fixed">
+      <parent link="zed_camera_center"/>
+      <child link="zed_right_camera_frame"/>
+      <origin xyz="0 -0.06 0" rpy="0 0 0" />
+  </joint>
+  <joint name="zed_right_camera_optical_joint" type="fixed">
+      <origin xyz="0 0 0" rpy="-${M_PI/2} 0.0 -${M_PI/2}"/>
+      <parent link="zed_right_camera_frame"/>
+      <child link="zed_right_camera_optical_frame"/>
+  </joint>
+  <!-- Simulated Zed Camera-->
+  <xacro:if value="$(arg sim)">
+      <stereo_camera frame_rgb="zed_camera_center" frame_depth="zed_depth_dummy_frame_sim_only" cameraName="zed"  topic="pointcloud" robot_namespace="$(arg robot_namespace)"/>
+      <link name="zed_depth_dummy_frame_sim_only" />
+      <joint name="zed_camera_depth_joint" type="fixed">
+        <origin xyz="0 0 0" rpy="${-pi/2} 0 ${-pi/2}"/>
         <parent link="zed_camera_center"/>
-        <child link="zed_left_camera_frame"/>
-        <origin xyz="0 0.06 0" rpy="0 0 0" />
-    </joint>
-    <link name="zed_left_camera_frame" />
-    <joint name="zed_left_camera_optical_joint" type="fixed">
-        <origin xyz="0 0 0" rpy="-${M_PI/2} 0.0 -${M_PI/2}"/>
-        <parent link="zed_left_camera_frame"/>
-        <child link="zed_left_camera_optical_frame"/>
-    </joint>
-    <link name="zed_left_camera_optical_frame"/>
-<!-- Right Camera -->
-    <joint name="zed_right_camera_joint" type="fixed">
-        <parent link="zed_camera_center"/>
-        <child link="zed_right_camera_frame"/>
-        <origin xyz="0 -0.06 0" rpy="0 0 0" />
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