Commit message: push from roboto

File: unicorn_description/urdf/unicorn_target.urdf.xacro (robot description, xacro)
@@ -125,5 +125,5 @@
   </gazebo>
   <joint name="base_chassis_joint" type="fixed">
-    <parent link="base_link"/>
+    <parent link="base_link"/> <!-- Switched -->
     <child link="chassis_link" />
   <origin xyz="0 0.0 0" rpy="0 0 ${M_PI}" />
@@ -186,5 +186,6 @@
     </joint> -->
     <joint name="chassis_zed_joint" type="fixed">
-      <parent link="chassis_link"/>
+      <!--parent link="chassis_link"/-->
+      <parent link="base_link"/>
       <child link="zed_center"/>
      <origin xyz="-0.14 0.0 0.11" rpy="0 0 ${-M_PI}"/>
@@ -218,5 +219,6 @@
   <link name="camera_rgb_optical_frame" />
   <joint name="chassis_orbbec_joint" type="fixed">
-    <parent link="chassis_link"/>
+    <!--parent link="chassis_link"/-->
+    <parent link="base_link"/>
     <child link="camera_link"/>
     <origin xyz="0.2 0 0.3" rpy="0 0 ${M_PI}"/>
@@ -242,8 +244,12 @@
     <origin xyz="0 0 0" rpy="0 0 0" />
   </joint>
-  <wheel fb="back" lr="left" parent="chassis_link" translateY="-0.24" translateX="0.0" translateZ="-0.006" wheel_radius="0.1225" wheel_height="0.032" flip="1"/>
-  <wheel fb="back" lr="right" parent="chassis_link" translateY="0.24" translateX="0.0" translateZ="-0.006" wheel_radius="0.1225" wheel_height="0.032" flip="1"/>
-  <swivel_wheel fb="front" lr="left" parent="chassis_link" translateY="-0.16" translateX="0.355" translateZ="0.03" wheel_radius="0.05" wheel_height="0.05" flip="0"/>
-  <swivel_wheel fb="front" lr="right" parent="chassis_link" translateY="0.16" translateX="0.355" translateZ="0.03" wheel_radius="0.05" wheel_height="0.05" flip="0"/>
+  <!--wheel fb="back" lr="left" parent="chassis_link" translateY="-0.24" translateX="0.0" translateZ="-0.006" wheel_radius="0.1225" wheel_height="0.032" flip="1"/-->
+  <wheel fb="back" lr="left" parent="base_link" translateY="-0.24" translateX="0.0" translateZ="-0.006" wheel_radius="0.1225" wheel_height="0.032" flip="1"/>
+  <!--wheel fb="back" lr="right" parent="chassis_link" translateY="0.24" translateX="0.0" translateZ="-0.006" wheel_radius="0.1225" wheel_height="0.032" flip="1"/-->
+  <wheel fb="back" lr="right" parent="base_link" translateY="0.24" translateX="0.0" translateZ="-0.006" wheel_radius="0.1225" wheel_height="0.032" flip="1"/>
+  <!--swivel_wheel fb="front" lr="left" parent="chassis_link" translateY="-0.16" translateX="0.355" translateZ="0.03" wheel_radius="0.05" wheel_height="0.05" flip="0"/-->
+  <swivel_wheel fb="front" lr="left" parent="base_link" translateY="-0.16" translateX="0.355" translateZ="0.03" wheel_radius="0.05" wheel_height="0.05" flip="0"/>
+  <!--swivel_wheel fb="front" lr="right" parent="chassis_link" translateY="0.16" translateX="0.355" translateZ="0.03" wheel_radius="0.05" wheel_height="0.05" flip="0"/-->
+  <swivel_wheel fb="front" lr="right" parent="base_link" translateY="0.16" translateX="0.355" translateZ="0.03" wheel_radius="0.05" wheel_height="0.05" flip="0"/>
   <!--ultrasonic_sensor frame="base_ultrasonic_br" topic="br" robot_namespace="$(arg robot_namespace)"/>
   <joint name="ultrasonic_mount_joint_br" type="fixed">
@@ -306,5 +312,6 @@
    <joint name="laser_mount_joint" type="fixed">
       <origin xyz="$(arg laser_xyz)" rpy="$(arg laser_rpy)" />
-      <parent link="chassis_link" />
+      <!--parent link="chassis_link" /-->
+      <parent link="base_link" />
       <child link="base_laser" />
    </joint>

Commit message: Added baselink for target to fix reverse issue

File: unicorn_description/urdf/unicorn_target.urdf.xacro (robot description, xacro)
@@ -48,5 +48,5 @@
  <!-- Main Body-base -->
   <link
-    name="chassis_link">
+    name="base_link">
     <inertial>
       <origin
@@ -69,5 +69,5 @@
       <geometry>
         <mesh
-          filename="package://unicorn_description/meshes/chassis_link.STL" />
+          filename="package://unicorn_description/meshes/base_link.STL" />
       </geometry>
       <material
@@ -83,5 +83,5 @@
       <geometry>
         <mesh
-          filename="package://unicorn_description/meshes/chassis_link.STL" />
+          filename="package://unicorn_description/meshes/base_link.STL" />
         <surface>
          <friction>
@@ -140,5 +140,5 @@
       rpy="0 0 ${M_PI}" />
     <parent
-      link="chassis_link" />
+      link="base_link" />
     <child
       link="lift_link" />
@@ -147,7 +147,6 @@
     <joint_properties damping="0.0" friction="0.0" />
   </joint>
-<!--
   <link
-    name="wheel_link">
+    name="chassis_link">
     <inertial>
       <origin
@@ -176,4 +175,49 @@
         rpy="0 0 0" />
       <geometry>
+        <!-- <mesh
+          filename="package://unicorn_description/meshes/base_link.STL" /> -->
+          <box size="0.01 0.01 0.01"/>
+      </geometry>
+      <!-- <surface>
+         <friction>
+           <ode><mu>0</mu><mu2>0</mu2></ode>
+         </friction>
+      </surface> -->
+    </collision>
+  </link>
+  <joint name="chassis_link_joint" type="fixed">
+    <parent link="base_link"/> <!-- Switched -->
+    <child link="chassis_link" />
+  <origin xyz="0 0.0 0" rpy="0 0 ${M_PI}" />
+  </joint>
+<!--
+  <link
+    name="wheel_link">
+    <inertial>
+      <origin
+        xyz="0 0 0"
+        rpy="0 0 0" />
+      <mass
+        value="0.01" />
+      <box_inertia  m="${5*0.01}" x="${base_x_size}" y="${base_y_size}" z="${base_z_size}"/>
+    </inertial>
+    <visual>
+      <origin
+        xyz="0 0 0"
+        rpy="0 0 0" />
+      <geometry>
+        <box size="0.01 0.01 0.01"/>
+      </geometry>
+      <material
+        name="">
+        <color
+          rgba="0.79216 0.81961 0.93333 1" />
+      </material>
+    </visual>
+    <collision>
+      <origin
+        xyz="0 0 0"
+        rpy="0 0 0" />
+      <geometry>
           <box size="0.01 0.01 0.01"/>
       </geometry>
@@ -185,22 +229,22 @@
   </gazebo>
   <joint name="base_chassis_joint" type="fixed">
-    <parent link="chassis_link"/>
+    <parent link="base_link"/>
     <child link="wheel_link" />
   <origin xyz="0 0.0 0" rpy="0 0 ${M_PI}" />
   </joint>-->
   <!-- driving wheels
-  <wheel fb="back" lr="left" parent="chassis_link" rotationZ="3.14159" translateY="0.23" translateX="0" translateZ="0.1225" wheel_radius="0.1225" wheel_height="0.032" flip="1"/>
-  <wheel fb="back" lr="right" parent="chassis_link" rotationZ="0" translateY="-0.23" translateX="0 " translateZ="0.1225" wheel_radius="0.1225" wheel_height="0.032" flip="1"/>
+  <wheel fb="back" lr="left" parent="base_link" rotationZ="3.14159" translateY="0.23" translateX="0" translateZ="0.1225" wheel_radius="0.1225" wheel_height="0.032" flip="1"/>
+  <wheel fb="back" lr="right" parent="base_link" rotationZ="0" translateY="-0.23" translateX="0 " translateZ="0.1225" wheel_radius="0.1225" wheel_height="0.032" flip="1"/>
   -->
   <wheel fb="back" lr="left" parent="lift_link"  translateY="0.24" translateX="0" translateZ="0.1225" wheel_radius="0.1225" wheel_height="0.032" flip="1"/>
   <wheel fb="back" lr="right" parent="lift_link" translateY="-0.24" translateX="0 " translateZ="0.1225" wheel_radius="0.1225" wheel_height="0.032" flip="1"/>
   <!-- others wheels -->
-  <swivel_wheel fb="front" lr="left" parent="chassis_link" translateY="0.16" translateX="-0.355" translateZ="0.1531" wheel_radius="0.05" wheel_height="0.05" flip="0"/>
-  <swivel_wheel fb="front" lr="right" parent="chassis_link" translateY="-0.16" translateX="-0.355" translateZ="0.1531" wheel_radius="0.05" wheel_height="0.05" flip="0"/>
+  <swivel_wheel fb="front" lr="left" parent="base_link" translateY="0.16" translateX="-0.355" translateZ="0.1531" wheel_radius="0.05" wheel_height="0.05" flip="0"/>
+  <swivel_wheel fb="front" lr="right" parent="base_link" translateY="-0.16" translateX="-0.355" translateZ="0.1531" wheel_radius="0.05" wheel_height="0.05" flip="0"/>
  <!-- Front Lidar -->
   <lidar_gazebo frame="base_laser" topic="frontLidar/scan" simulation="$(arg sim)" sample_size="800" min_angle="-2.35619" max_angle="2.35619" robot_namespace="$(arg robot_namespace)" filename="$(arg frontlidar_meshfile)" />
   <joint name="laser_mount_joint" type="fixed">
     <origin xyz="$(arg laser_xyz)" rpy="$(arg laser_rpy)" />
-    <parent link="chassis_link" />
+    <parent link="base_link" />
     <child link="base_laser" />
   </joint>
@@ -209,5 +253,5 @@
   <joint name="rear_laser_mount_joint" type="fixed">
     <origin xyz="$(arg rear_laser_xyz)" rpy="$(arg rear_laser_rpy)" />
-    <parent link="chassis_link" />
+    <parent link="base_link" />
     <child link="rear_laser" />
   </joint>
@@ -216,5 +260,5 @@
     <joint name="zed_camera_rgb_joint" type="fixed">
       <origin xyz="$(arg zed_xyz)" rpy="$(arg zed_rpy)"/>
-      <parent link="chassis_link"/>
+      <parent link="base_link"/>
       <child link="zed_camera"/>
     </joint>
@@ -228,5 +272,5 @@
     <joint name="realsense_gb_joint" type="fixed">
       <origin xyz="$(arg real_rgb_xyz)" rpy="$(arg real_rpy)"/>
-      <parent link="chassis_link"/>
+      <parent link="base_link"/>
       <child link="realsense_camera"/>
     </joint>
@@ -243,5 +287,5 @@
       <updateRate>5</updateRate>
       <frameId>odom_chassis</frameId>
-      <bodyName>chassis_link</bodyName>
+      <bodyName>base_link</bodyName>
       <topicName>gps</topicName>
       <velocityTopicName>gps_velocity</velocityTopicName>
@@ -267,5 +311,5 @@
       <odometryTopic>wheel_encoder/odom</odometryTopic>
       <odometryFrame>odom_chassis_dont_use</odometryFrame>
-      <robotBaseFrame>chassis_link</robotBaseFrame>
+      <robotBaseFrame>base_link</robotBaseFrame>
       <publishWheelTF>false</publishWheelTF>
       <publishWheelJointState>false</publishWheelJointState>

Commit message: Added baselink for target to fix reverse issue

File: unicorn_description/urdf/unicorn_target.urdf.xacro (robot description, xacro)
@@ -147,4 +147,5 @@
     <joint_properties damping="0.0" friction="0.0" />
   </joint>
+<!-- Dummy frame to fix reverse issue -->
   <link
     name="chassis_link">
@@ -175,13 +176,6 @@
         rpy="0 0 0" />
       <geometry>
-        <!-- <mesh
-          filename="package://unicorn_description/meshes/base_link.STL" /> -->
           <box size="0.01 0.01 0.01"/>
       </geometry>
-      <!-- <surface>
-         <friction>
-           <ode><mu>0</mu><mu2>0</mu2></ode>
-         </friction>
-      </surface> -->
     </collision>
   </link>

Commit message: Added baselink for target to fix reverse issue

File: unicorn_description/urdf/unicorn_target.urdf.xacro (robot description, xacro)
@@ -180,5 +180,5 @@
     </collision>
   </link>
-  <joint name="chassis_link_joint" type="fixed">
+  <joint name="chassis_joint" type="fixed">
     <parent link="base_link"/> <!-- Switched -->
     <child link="chassis_link" />

Commit message: Fix wrong frames and topics

File: unicorn_description/urdf/unicorn_target.urdf.xacro (robot description, xacro)
@@ -181,6 +181,6 @@
   </link>
   <joint name="chassis_joint" type="fixed">
-    <parent link="base_link"/> <!-- Switched -->
-    <child link="chassis_link" />
+    <parent link="chassis_link"/> <!-- Switched -->
+    <child link="base_link" />
   <origin xyz="0 0.0 0" rpy="0 0 ${M_PI}" />
   </joint>

Commit message: rotated zed frame in target

File: unicorn_description/urdf/unicorn_target.urdf.xacro (robot description, xacro)
@@ -214,5 +214,5 @@
 <!-- Camera Center -->
     <joint name="zed_camera_center_joint" type="fixed">
-        <parent link="chassis_link"/>
+        <parent link="base_link"/>
         <child link="zed_camera_center"/>
         <origin xyz="$(arg zed_xyz)" rpy="0 0 0" />
