Commit message: Uppdated Robot URDF to be more compact and similar to simulation

File: unicorn_description/urdf/unicorn_target.urdf.xacro (robot description, xacro)
@@ -3,25 +3,28 @@
   <xacro:arg name="robot_namespace" default="/" />
   <xacro:arg name="sim" default="false" />
+  <!-- Define Constants -->
+  <xacro:property name="M_PI" value="3.1415926535897931" />
+  <xacro:property name="M_PI2" value="1.57079632679" />
     <!-- Swivel wheel -->
-  <xacro:include filename="$(find am_description)/urdf/swivel_wheel.urdf.xacro" />
+  <xacro:include filename="$(find unicorn_description)/urdf/swivel_wheel.urdf.xacro" />
     <!-- Wheel -->
-  <xacro:include filename="$(find am_description)/urdf/wheel.urdf.xacro" />
+  <xacro:include filename="$(find unicorn_description)/urdf/wheel.urdf.xacro" />
     <!-- camera pack-->
   <xacro:include filename="$(find unicorn_description)/urdf/stereo_camera_gazebo.urdf.xacro" />
    <!-- lidar pack-->
   <xacro:include filename="$(find unicorn_description)/urdf/lidar_gazebo.urdf.xacro" />
-  <xacro:property name="M_PI" value="3.1415926535897931" />
-  <xacro:property name="M_PI2" value="1.57079632679" />
-  <!-- base --><!--
-    <xacro:property name="base_x_size" value="0.72" />
-  <xacro:property name="base_y_size" value="0.55" />
-  <xacro:property name="base_z_size" value="0.6" />
-  <xacro:property name="base_mass" value="21.446" /> 21.446 in kg-->
-    <!-- Main Body-base -->
+  <!-- Main Body-base -->
   <xacro:property name="base_x_size" value="0.72" />
   <xacro:property name="base_y_size" value="0.55" />
   <xacro:property name="base_z_size" value="0.23" />
   <xacro:property name="base_mass" value="15" /> <!-- in kg-->
-    <!--Inertial macros for the box and cylinder. Units are kg*m^2-->
+  <!-- Base Link Rotation -->
+  <xacro:if value="$(arg sim)">
+    <xacro:arg name="base_link_rpy" default="0 0 0" />
+  </xacro:if>
+  <xacro:unless value="$(arg sim)">
+    <xacro:arg name="base_link_rpy" default="0 0 ${M_PI}" />
+  </xacro:unless>
+  <!--Inertial macros for the box and cylinder. Units are kg*m^2-->
   <xacro:macro name="box_inertia" params="m x y z">
     <inertia ixx="${m*(y*y+z*z)/12}" ixy="0" ixz="0"
@@ -33,5 +36,5 @@
   <xacro:arg name="laser_rpy" default="0 0 0" />
   <xacro:arg name="frontlidar_meshfile" default="package://unicorn_description/meshes/base_laser.STL" />
-<!-- Rear Lidar  -->
+  <!-- Rear Lidar  -->
   <xacro:arg name="rear_laser_xyz" default="-0.42145 -0.00645 0.28652" />
   <xacro:arg name="rear_laser_rpy" default="0 0 ${M_PI}" />
@@ -50,48 +53,40 @@
   <xacro:arg name="realsense_meshfile" default="package://unicorn_description/meshes/real_sense.STL" />
  <!-- Main Body-base -->
+  <link name="base_link" />
+  <joint name="chassis_joint" type="fixed">
+    <parent link="base_link"/>
+    <child link="chassis_link" />
+  <origin xyz="0 0.0 0" rpy="$(arg base_link_rpy)" />
+  </joint>
   <link
-    name="base_link">
+    name="chassis_link">
     <inertial>
-      <origin
-        xyz="0 0 0"
-        rpy="0 0 0" />
-      <mass
-        value="10" />
-      <inertia
-        ixx="1"
-        ixy="0"
-        ixz="3"
-        iyy="3"
-        iyz="3"
-        izz="1" />
+      <origin xyz="0 0 0" rpy="0 0 0" />
+      <mass value="15" />
+      <inertia ixx="1" ixy="0" ixz="3" iyy="3" iyz="3" izz="1" />
     </inertial>
     <visual>
-      <origin
-        xyz="0 0 0"
-        rpy="0 0 0" />
-      <geometry>
-        <mesh
-          filename="package://unicorn_description/meshes/chassis_link.STL" />
-      </geometry>
-      <material
-        name="">
-        <color
-          rgba="0.792156862745098 0.819607843137255 0.933333333333333 1" />
+      <origin xyz="0 0 0" rpy="0 0 0" />
+      <geometry>
+        <mesh filename="package://unicorn_description/meshes/chassis_link.STL" />
+      </geometry>
+      <material name="">
+        <color rgba="0.792156862745098 0.819607843137255 0.933333333333333 1" />
       </material>
     </visual>
-    <collision>
-      <origin
-        xyz="0 0 0"
-        rpy="0 0 0" />
-      <geometry>
-        <mesh
-          filename="package://unicorn_description/meshes/chassis_link.STL" />
-        <surface>
-         <friction>
-           <ode><mu>0.4</mu><mu2>0.4</mu2></ode>
-         </friction>
-      </surface>
-      </geometry>
-    </collision>
+    <surface>
+      <friction>
+        <ode>
+          <mu>0.8</mu>
+          <mu2>0.8</mu2>
+        </ode>
+      </friction>
+    </surface>
+  <collision>
+    <origin xyz="0 0 0" rpy="0 0 0" />
+    <geometry>
+      <mesh filename="package://unicorn_description/meshes/chassis_link.STL" />
+    </geometry>
+  </collision>
   </link>
 <!-- Lift -->
@@ -99,169 +94,207 @@
     name="lift_link">
     <inertial>
-      <origin
-        xyz="0 0 0"
-        rpy="0 0 0" />
-      <mass
-        value="4" />
-      <inertia
-        ixx="1"
-        ixy="0"
-        ixz="3"
-        iyy="3"
-        iyz="3"
-        izz="1" />
+      <origin xyz="0 0 0" rpy="0 0 0" />
+      <mass value="10" />
+      <inertia ixx="1" ixy="0" ixz="3" iyy="3" iyz="3" izz="1" />
     </inertial>
     <visual>
-      <origin
-        xyz="0 0 0"
-        rpy="0 0 ${M_PI}" />
-      <geometry>
-        <mesh
-          filename="package://unicorn_description/meshes/lift_link.STL" />
-      </geometry>
-      <material
-        name="">
-        <color
-          rgba="0.752941176470588 0.752941176470588 0.752941176470588 1" />
+      <origin xyz="0 0 0" rpy="0 0 ${M_PI}" />
+      <geometry>
+        <mesh filename="package://unicorn_description/meshes/lift_link.STL" />
+      </geometry>
+      <material name="">
+        <color rgba="0.752941176470588 0.752941176470588 0.752941176470588 1" />
       </material>
     </visual>
+      <surface>
+        <friction>
+          <ode>
+            <mu>0.8</mu>
+            <mu2>0.8</mu2>
+          </ode>
+        </friction>
+      </surface>
     <collision>
-      <origin
-        xyz="0 0 0"
-        rpy="0 0 ${M_PI}" />
-      <geometry>
-        <mesh
-          filename="package://unicorn_description/meshes/lift_link.STL" />
+      <origin xyz="0 0 0" rpy="0 0 ${M_PI}" />
+      <geometry>
+        <mesh filename="package://unicorn_description/meshes/lift_link.STL" />
       </geometry>
     </collision>
   </link>
-  <joint
-    name="lift_joint"
-    type="fixed">
-    <origin
-      xyz="0 0 0"
-      rpy="0 0 ${M_PI}" />
-    <parent
-      link="base_link" />
-    <child
-      link="lift_link" />
-    <axis
-      xyz="0 0 0" />
-    <joint_properties damping="0.0" friction="0.0" />
-  </joint>
-<!-- Dummy frame to fix reverse issue -->
+  <joint name="lift_joint" type="fixed">
+    <origin xyz="0 0 0" rpy="0 0 ${M_PI}" />
+    <parent link="chassis_link" />
+    <child link="lift_link" />
+    <axis xyz="0 0 0" />
+    <joint_properties damping="1" friction="0.5" />
+  </joint>
+<!-- Lift links-->
   <link
-    name="chassis_link">
+    name="lift_horizontal_link">
+    <visual>
+      <origin xyz="0 0 0" rpy="0 0 0" />
+      <geometry>
+        <mesh filename="package://unicorn_description/meshes/lift_horizontal_link.STL" />
+      </geometry>
+      <material name="">
+        <color rgba="0.898039215686275 0.917647058823529 0.929411764705882 1" />
+      </material>
+    </visual>
+      <surface>
+        <friction>
+          <ode>
+            <mu>0.8</mu>
+            <mu2>0.8</mu2>
+          </ode>
+        </friction>
+      </surface>
+    <collision>
+      <origin xyz="0 0 0" rpy="0 0 0" />
+      <geometry>
+        <mesh filename="package://unicorn_description/meshes/lift_horizontal_link.STL" />
+      </geometry>
+    </collision>
     <inertial>
-      <origin
-        xyz="0 0 0"
-        rpy="0 0 0" />
-      <mass
-        value="0.01" />
-      <box_inertia  m="${5*0.01}" x="${base_x_size}" y="${base_y_size}" z="${base_z_size}"/>
+      <origin xyz="0 0 0" rpy="0 0 0" />
+      <mass value="1.50791731426345" />
+      <inertia ixx="0.00998369504134607" ixy="1.05918049885466E-06" ixz="3.20101525315815E-06" iyy="0.0148024039374132" iyz="1.02762580499191E-05" izz="0.0197484509547163" />
+    </inertial>
+  </link>
+  <link
+    name="lift_vertical_link">
+    <inertial>
+      <origin xyz="-0.0046764 0.62992 -0.22573" rpy="0 0 0" />
+      <mass value="0.61742" />
+      <inertia ixx="0.00029455" ixy="9.8754E-10" ixz="2.0681E-19" iyy="0.00411" iyz="3.0422E-05" izz="0.0043679" />
     </inertial>
     <visual>
-      <origin
-        xyz="0 0 0"
-        rpy="0 0 0" />
-      <geometry>
-        <box size="0.01 0.01 0.01"/>
-      </geometry>
-      <material
-        name="">
-        <color
-          rgba="0.79216 0.81961 0.93333 1" />
+      <origin xyz="0 0 0" rpy="0 0 0" />
+      <geometry>
+        <mesh filename="package://unicorn_description/meshes/lift_vertical_link.STL" />
+      </geometry>
+      <material name="">
+        <color rgba="1 0.69412 0.27843 1" />
       </material>
     </visual>
+    <surface>
+      <friction>
+        <ode>
+          <mu>0.8</mu>
+          <mu2>0.8</mu2>
+        </ode>
+      </friction>
+    </surface>
     <collision>
-      <origin
-        xyz="0 0 0"
-        rpy="0 0 0" />
-      <geometry>
-          <box size="0.01 0.01 0.01"/>
+      <origin xyz="0 0 0" rpy="0 0 0" />
+      <geometry>
+        <mesh filename="package://unicorn_description/meshes/lift_vertical_link.STL" />
       </geometry>
     </collision>
   </link>
-  <joint name="chassis_joint" type="fixed">
-    <parent link="chassis_link"/> <!-- Switched -->
-    <child link="base_link" />
-  <origin xyz="0 0.0 0" rpy="0 0 ${M_PI}" />
-  </joint>
-  <!-- driving wheels
-  <wheel fb="back" lr="left" parent="base_link" rotationZ="3.14159" translateY="0.23" translateX="0" translateZ="0.1225" wheel_radius="0.1225" wheel_height="0.032" flip="1"/>
-  <wheel fb="back" lr="right" parent="base_link" rotationZ="0" translateY="-0.23" translateX="0 " translateZ="0.1225" wheel_radius="0.1225" wheel_height="0.032" flip="1"/>
-  -->
-  <wheel fb="back" lr="left" parent="lift_link"  translateY="0.24" translateX="0" translateZ="0.1225" wheel_radius="0.1225" wheel_height="0.032" flip="1"/>
-  <wheel fb="back" lr="right" parent="lift_link" translateY="-0.24" translateX="0 " translateZ="0.1225" wheel_radius="0.1225" wheel_height="0.032" flip="1"/>
-  <!-- others wheels -->
-  <swivel_wheel fb="front" lr="left" parent="base_link" translateY="0.16" translateX="-0.355" translateZ="0.1531" wheel_radius="0.05" wheel_height="0.05" flip="0"/>
-  <swivel_wheel fb="front" lr="right" parent="base_link" translateY="-0.16" translateX="-0.355" translateZ="0.1531" wheel_radius="0.05" wheel_height="0.05" flip="0"/>
- <!-- Front Lidar -->
+  <joint name="lift_horizontal_joint" type="fixed"> <!-- type="prismatic" -->
+    <parent  link="lift_link" />
+    <child  link="lift_horizontal_link" />
+    <origin xyz="0.05 0 0.137" rpy="${M_PI2} 0 ${-M_PI2}" />
+    <axis xyz="0 0 -1" rpy="0 0 0"  />
+    <limit lower="0.17" upper="0" effort="100" velocity="0" />
+    <joint_properties damping="10000" friction="1000" />
+  </joint>
+  <joint name="lift_vertical_joint" type="fixed"> <!-- type="prismatic" -->
+    <origin xyz="0 -0.16 0" rpy="0 0 0" />
+    <parent link="lift_horizontal_link" />
+    <child link="lift_vertical_link" />
+    <axis xyz="0 1 0" />
+    <limit lower="0" upper="0.16" effort="100" velocity="0" />
+    <joint_properties damping="1000" friction="1000" />
+  </joint>
+<!-- Front Wheels -->
+<!-- Dummy Link for simulation, used to Correct back motion from HRP drivers -->
+  <xacro:if value="$(arg sim)">
+    <link name="dummy_wheel_link" >
+      <inertial>
+        <origin xyz="0 0 0" rpy="0 0 0" />
+        <mass value="0.01" />
+        <box_inertia  m="${5*0.01}" x="${base_x_size}" y="${base_y_size}" z="${base_z_size}"/>
+      </inertial>
+    </link>
+    <joint name="dummy_wheel_joint" type="fixed">
+      <origin xyz="0 0.0 0" rpy="0 0 ${M_PI}" />
+      <parent link="chassis_link"/>
+      <child link="dummy_wheel_link"/>
+    </joint>
+    <wheel fb="back" lr="left" parent="dummy_wheel_link"  translateY="0.24" translateX="0" translateZ="0.1225" wheel_radius="0.1225" wheel_height="0.032" flip="1"/>
+    <wheel fb="back" lr="right" parent="dummy_wheel_link" translateY="-0.24" translateX="0 " translateZ="0.1225" wheel_radius="0.1225" wheel_height="0.032" flip="1"/>
+  </xacro:if>
+  <!-- For real Platform -->
+  <xacro:unless value="$(arg sim)">
+    <wheel fb="back" lr="left" parent="chassis_link"  translateY="0.24" translateX="0" translateZ="0.1225" wheel_radius="0.1225" wheel_height="0.032" flip="1"/>
+    <wheel fb="back" lr="right" parent="chassis_link" translateY="-0.24" translateX="0 " translateZ="0.1225" wheel_radius="0.1225" wheel_height="0.032" flip="1"/>
+  </xacro:unless>
+  <!-- Swivel back wheels - Should be changed to omniwheels-->
+  <swivel_wheel fb="front" lr="left" parent="chassis_link" translateY="0.16" translateX="-0.355" translateZ="0.1531" wheel_radius="0.05" wheel_height="0.05" flip="0"/>
+  <swivel_wheel fb="front" lr="right" parent="chassis_link" translateY="-0.16" translateX="-0.355" translateZ="0.1531" wheel_radius="0.05" wheel_height="0.05" flip="0"/>
+  <!-- Front Lidar -->
   <lidar_gazebo frame="base_laser" topic="frontLidar/scan" simulation="$(arg sim)" sample_size="800" min_angle="-2.35619" max_angle="2.35619" robot_namespace="$(arg robot_namespace)" filename="$(arg frontlidar_meshfile)" />
   <joint name="laser_mount_joint" type="fixed">
     <origin xyz="$(arg laser_xyz)" rpy="$(arg laser_rpy)" />
-    <parent link="base_link" />
+    <parent link="chassis_link" />
     <child link="base_laser" />
   </joint>
    <!-- Back Lidar -->
-  <lidar_gazebo frame="rear_laser" topic="rearLidar/scan" simulation="$(arg sim)" sample_size="11" min_angle="-0.767944871" max_angle="0.767944871" robot_namespace="$(arg robot_namespace)" filename="$(arg rearlidar_meshfile)"/>
+  <lidar_gazebo frame="rear_laser" topic="rearLidar/scan" simulation="$(arg sim)" sample_size="11" min_angle="-0.698131701" max_angle="0.698131701" robot_namespace="$(arg robot_namespace)" filename="$(arg rearlidar_meshfile)"/>
   <joint name="rear_laser_mount_joint" type="fixed">
     <origin xyz="$(arg rear_laser_xyz)" rpy="$(arg rear_laser_rpy)" />
-    <parent link="base_link" />
+    <parent link="chassis_link" />
     <child link="rear_laser" />
   </joint>
   <!-- Zed Camera -->
-<!-- Camera Center -->
-    <joint name="zed_camera_center_joint" type="fixed">
-        <parent link="base_link"/>
-        <child link="zed_camera_center"/>
-        <origin xyz="$(arg zed_xyz)" rpy="0 0 0" />
-    </joint>
-    <link name="zed_camera_center">
-        <visual>
-            <origin xyz="0 0 0" rpy="0 0 0"/>
-            <geometry>
-                <mesh filename="$(arg zed_meshfile)" />
-            </geometry>
-        </visual>
-    </link>
-<!-- Left Camera -->
-    <joint name="zed_left_camera_joint" type="fixed">
+  <link name="zed_camera_center">
+      <visual>
+          <origin xyz="0 0 0" rpy="0 0 0"/>
+          <geometry>
+              <mesh filename="$(arg zed_meshfile)" />
+          </geometry>
+      </visual>
+  </link>
+  <link name="zed_right_camera_frame" />
+  <link name="zed_right_camera_optical_frame"/>
+  <link name="zed_left_camera_optical_frame"/>
+  <link name="zed_left_camera_frame" />
+  <joint name="zed_camera_center_joint" type="fixed">
+      <parent link="chassis_link"/>
+      <child link="zed_camera_center"/>
+      <origin xyz="$(arg zed_xyz)" rpy="0 0 0" />
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