Commit message: Changed friction for wheels in sim

File: unicorn_description/urdf/swivel_wheel.urdf.xacro (robot description, xacro)
@@ -85,6 +85,6 @@
           <friction>
             <ode>
-              <mu>0.4</mu>
-              <mu2>0.4</mu2>
+              <mu>0.8</mu>
+              <mu2>0.8</mu2>
             </ode>
           </friction>

File: unicorn_description/urdf/unicorn_sim.urdf.xacro (robot description, xacro)
@@ -179,4 +179,196 @@
     </inertial>
   </link>
+  <link
+    name="lift_vertical_link">
+    <inertial>
+      <origin
+        xyz="-0.0046764 0.62992 -0.22573"
+        rpy="0 0 0" />
+      <mass
+        value="0.61742" />
+      <inertia
+        ixx="0.00029455"
+        ixy="9.8754E-10"
+        ixz="2.0681E-19"
+        iyy="0.00411"
+        iyz="3.0422E-05"
+        izz="0.0043679" />
+    </inertial>
+    <visual>
+      <origin
+        xyz="0 0 0"
+        rpy="0 0 0" />
+      <geometry>
+        <mesh
+          filename="package://unicorn_description/meshes/lift_vertical_link.STL" />
+      </geometry>
+      <material
+        name="">
+        <color
+          rgba="1 0.69412 0.27843 1" />
+      </material>
+    </visual>
+    <collision>
+      <origin
+        xyz="0 0 0"
+        rpy="0 0 0" />
+      <geometry>
+        <mesh
+          filename="package://unicorn_description/meshes/lift_vertical_link.STL" />
+      </geometry>
+    </collision>
+  </link>
+  <joint
+    name="lift_vertical_joint"
+    type="prismatic">
+    <origin
+      xyz="0 -0.16 0"
+      rpy="0 0 0" />
+    <parent
+      link="lift_horizontal_link" />
+    <child
+      link="lift_vertical_link" />
+    <axis
+      xyz="0 1 0" />
+    <limit
+      lower="0"
+      upper="0.16"
+      effort="100"
+      velocity="0.4" />
+      <joint_properties damping="10" friction="0.5" />
+  </joint>
+  <gazebo reference="lift_vertical_joint">
+      <mu1 value="10000.0" />
+      <mu2 value="10000.0" />
+      <kp value="100000.0" />
+      <kd value="10000.0" />
+      <dampingFactor value="0.5" />
+      <fdir1 value="1 0 0" />
+      <material>Gazebo/Black</material>
+      <turnGravityOff>false</turnGravityOff>
+  </gazebo>
+  <wheel fb="back" lr="left" parent="lift_link"  translateY="0.24" translateX="0" translateZ="0.1225" wheel_radius="0.1225" wheel_height="0.032" flip="1"/>
+  <wheel fb="back" lr="right" parent="lift_link" translateY="-0.24" translateX="0 " translateZ="0.1225" wheel_radius="0.1225" wheel_height="0.032" flip="1"/>
+  <!-- others wheels -->
+  <swivel_wheel fb="front" lr="left" parent="chassis_link" translateY="0.16" translateX="-0.355" translateZ="0.1531" wheel_radius="0.05" wheel_height="0.05" flip="0"/>
+  <swivel_wheel fb="front" lr="right" parent="chassis_link" translateY="-0.16" translateX="-0.355" translateZ="0.1531" wheel_radius="0.05" wheel_height="0.05" flip="0"/>
+ <!-- Front Lidar -->
+  <lidar_gazebo frame="base_laser" topic="frontLidar/scan" simulation="$(arg sim)" sample_size="800" min_angle="-2.35619" max_angle="2.35619" robot_namespace="$(arg robot_namespace)" filename="$(arg frontlidar_meshfile)" />
+  <joint name="laser_mount_joint" type="fixed">
+    <origin xyz="$(arg laser_xyz)" rpy="$(arg laser_rpy)" />
+    <parent link="chassis_link" />
+    <child link="base_laser" />
+  </joint>
+   <!-- Back Lidar -->
+  <lidar_gazebo frame="rear_laser" topic="rearLidar/scan" simulation="$(arg sim)" sample_size="11" min_angle="-0.767944871" max_angle="0.767944871" robot_namespace="$(arg robot_namespace)" filename="$(arg rearlidar_meshfile)"/>
+  <joint name="rear_laser_mount_joint" type="fixed">
+    <origin xyz="$(arg rear_laser_xyz)" rpy="$(arg rear_laser_rpy)" />
+    <parent link="chassis_link" />
+    <child link="rear_laser" />
+  </joint>
+  <!-- Zed Camera -->
+<!-- Camera Center -->
+    <joint name="zed_camera_center_joint" type="fixed">
+        <parent link="chassis_link"/>
+        <child link="zed_camera_center"/>
+        <origin xyz="$(arg zed_xyz)" rpy="0 0 0" />
+    </joint>
+    <link name="zed_camera_center">
+        <visual>
+            <origin xyz="0 0 0" rpy="0 0 0"/>
+            <geometry>
+                <mesh filename="$(arg zed_meshfile)" />
+            </geometry>
+        </visual>
+    </link>
+<!-- Left Camera -->
+    <joint name="zed_left_camera_joint" type="fixed">
+        <parent link="zed_camera_center"/>
+        <child link="zed_left_camera_frame"/>
+        <origin xyz="0 0.06 0" rpy="0 0 0" />
+    </joint>
+    <link name="zed_left_camera_frame" />
+    <joint name="zed_left_camera_optical_joint" type="fixed">
+        <origin xyz="0 0 0" rpy="-${M_PI/2} 0.0 -${M_PI/2}"/>
+        <parent link="zed_left_camera_frame"/>
+        <child link="zed_left_camera_optical_frame"/>
+    </joint>
+    <link name="zed_left_camera_optical_frame"/>
+<!-- Right Camera -->
+    <joint name="zed_right_camera_joint" type="fixed">
+        <parent link="zed_camera_center"/>
+        <child link="zed_right_camera_frame"/>
+        <origin xyz="0 -0.06 0" rpy="0 0 0" />
+    </joint>
+    <link name="zed_right_camera_frame" />
+    <joint name="zed_right_camera_optical_joint" type="fixed">
+        <origin xyz="0 0 0" rpy="-${M_PI/2} 0.0 -${M_PI/2}"/>
+        <parent link="zed_right_camera_frame"/>
+        <child link="zed_right_camera_optical_frame"/>
+    </joint>
+    <link name="zed_right_camera_optical_frame"/>
+<!---->
+<xacro:if value="$(arg sim)">
+    <stereo_camera frame_rgb="zed_camera_center" frame_depth="zed_depth_dummy_frame_sim_only" cameraName="zed"  topic="pointcloud" robot_namespace="$(arg robot_namespace)"/>
+    <link name="zed_depth_dummy_frame_sim_only"></link>
+    <joint name="zed_camera_depth_joint" type="fixed">
+      <origin xyz="0 0 0" rpy="${-pi/2} 0 ${-pi/2}"/>
+      <parent link="zed_camera_center"/>
+      <child link="zed_depth_dummy_frame_sim_only"/>
+    </joint>
+</xacro:if>
+  <!-- realsense Camera -->
+<!-- Links only needed in simulation, created by realsense software otherwise-->
+  <link
+    name="realsense_link">
+      <visual>
+      <origin xyz="0 0 0" rpy="0 0 0"/>
+      <geometry>
+          <mesh filename="$(arg realsense_meshfile)" />
+      </geometry>
+    </visual>
+  </link>
+  <joint name="realsense_joint" type="fixed">
+    <origin xyz="$(arg real_base)" rpy="$(arg real_rpy)"/>
+    <parent link="chassis_link"/>
+    <child link="realsense_link"/>
+  </joint>
+<xacro:if value="$(arg sim)">
+  <stereo_camera frame_rgb="realsense_color_frame" frame_depth="realsense_depth_dummy_frame_sim_only" cameraName="realsense" topic="pointcloud" robot_namespace="$(arg robot_namespace)"/>
+  <link name="realsense_color_frame"> </link>
+  <link name="realsense_depth_frame"></link>
+   <link name="realsense_depth_dummy_frame_sim_only"></link>
+  <link
+    name="realsense_depth_optical_frame">
+  </link>
+  <link
+    name="realsense_color_optical_frame">
+  </link>
+  <joint name="realsense_gb_joint" type="fixed">
+    <origin xyz="$(arg real_rgb_xyz)" rpy="0 0 0"/>
+    <parent link="realsense_link"/>
+    <child link="realsense_color_frame"/>
+  </joint>
+  <joint name="realsense_depth_joint" type="fixed">
+    <origin xyz="$(arg real_depth_xyz)" rpy="0 0 0"/>
+    <parent link="realsense_link"/>
+    <child link="realsense_depth_frame"/>
+  </joint>
+  <joint name="realsense_depth_dummy_joint" type="fixed">
+    <origin xyz="$(arg real_depth_xyz)" rpy="-${M_PI/2} 0.0 -${M_PI/2}"/>
+    <parent link="realsense_link"/>
+    <child link="realsense_depth_dummy_frame_sim_only"/>
+  </joint>
+  <joint name="realsense_optical_color_joint" type="fixed">
+    <origin xyz="0 0 0" rpy="$(arg real_optical_rpy)"/>
+    <parent link="realsense_color_frame"/>
+    <child link="realsense_color_optical_frame"/>
+  </joint>
+  <joint name="realsense_optical_depth_joint" type="fixed">
+    <origin xyz="0 0 0" rpy="$(arg real_depth_rpy)"/>
+    <parent link="realsense_depth_frame"/>
+    <child link="realsense_depth_optical_frame"/>
+  </joint>
+</xacro:if>
   <joint name="lift_horizontal_joint" type="prismatic">
     <parent  link="lift_link" />
@@ -207,73 +399,4 @@
       </actuator>
   </transmission>
-  <link
-    name="lift_vertical_link">
-    <inertial>
-      <origin
-        xyz="-0.0046764 0.62992 -0.22573"
-        rpy="0 0 0" />
-      <mass
-        value="0.61742" />
-      <inertia
-        ixx="0.00029455"
-        ixy="9.8754E-10"
-        ixz="2.0681E-19"
-        iyy="0.00411"
-        iyz="3.0422E-05"
-        izz="0.0043679" />
-    </inertial>
-    <visual>
-      <origin
-        xyz="0 0 0"
-        rpy="0 0 0" />
-      <geometry>
-        <mesh
-          filename="package://unicorn_description/meshes/lift_vertical_link.STL" />
-      </geometry>
-      <material
-        name="">
-        <color
-          rgba="1 0.69412 0.27843 1" />
-      </material>
-    </visual>
-    <collision>
-      <origin
-        xyz="0 0 0"
-        rpy="0 0 0" />
-      <geometry>
-        <mesh
-          filename="package://unicorn_description/meshes/lift_vertical_link.STL" />
-      </geometry>
-    </collision>
-  </link>
-  <joint
-    name="lift_vertical_joint"
-    type="prismatic">
-    <origin
-      xyz="0 -0.16 0"
-      rpy="0 0 0" />
-    <parent
-      link="lift_horizontal_link" />
-    <child
-      link="lift_vertical_link" />
-    <axis
-      xyz="0 1 0" />
-    <limit
-      lower="0"
-      upper="0.16"
-      effort="100"
-      velocity="0.4" />
-      <joint_properties damping="10" friction="0.5" />
-  </joint>
-  <gazebo reference="lift_vertical_joint">
-      <mu1 value="10000.0" />
-      <mu2 value="10000.0" />
-      <kp value="100000.0" />
-      <kd value="10000.0" />
-      <dampingFactor value="0.5" />
-      <fdir1 value="1 0 0" />
-      <material>Gazebo/Black</material>
-      <turnGravityOff>false</turnGravityOff>
-  </gazebo>
   <transmission name="lift_vertical_joint_trans">
       <type>transmission_interface/SimpleTransmission</type>
@@ -286,145 +409,8 @@
       </actuator>
   </transmission>
-  <wheel fb="back" lr="left" parent="lift_link"  translateY="0.24" translateX="0" translateZ="0.1225" wheel_radius="0.1225" wheel_height="0.032" flip="1"/>
-  <wheel fb="back" lr="right" parent="lift_link" translateY="-0.24" translateX="0 " translateZ="0.1225" wheel_radius="0.1225" wheel_height="0.032" flip="1"/>
-  <!-- others wheels -->
-  <swivel_wheel fb="front" lr="left" parent="chassis_link" translateY="0.16" translateX="-0.355" translateZ="0.1531" wheel_radius="0.05" wheel_height="0.05" flip="0"/>
-  <swivel_wheel fb="front" lr="right" parent="chassis_link" translateY="-0.16" translateX="-0.355" translateZ="0.1531" wheel_radius="0.05" wheel_height="0.05" flip="0"/>
- <!-- Front Lidar -->
-  <lidar_gazebo frame="base_laser" topic="frontLidar/scan" simulation="$(arg sim)" sample_size="800" min_angle="-2.35619" max_angle="2.35619" robot_namespace="$(arg robot_namespace)" filename="$(arg frontlidar_meshfile)" />
-  <joint name="laser_mount_joint" type="fixed">
-    <origin xyz="$(arg laser_xyz)" rpy="$(arg laser_rpy)" />
-    <parent link="chassis_link" />
-    <child link="base_laser" />
-  </joint>
-   <!-- Back Lidar -->
-  <lidar_gazebo frame="rear_laser" topic="rearLidar/scan" simulation="$(arg sim)" sample_size="11" min_angle="-0.767944871" max_angle="0.767944871" robot_namespace="$(arg robot_namespace)" filename="$(arg rearlidar_meshfile)"/>
-  <joint name="rear_laser_mount_joint" type="fixed">
-    <origin xyz="$(arg rear_laser_xyz)" rpy="$(arg rear_laser_rpy)" />
-    <parent link="chassis_link" />
-    <child link="rear_laser" />
-  </joint>
-  <!-- Zed Camera -->
-<!-- Camera Center -->
-    <joint name="zed_camera_center_joint" type="fixed">
-        <parent link="chassis_link"/>
-        <child link="zed_camera_center"/>
-        <origin xyz="$(arg zed_xyz)" rpy="0 0 0" />
-    </joint>
-    <link name="zed_camera_center">
-        <visual>
-            <origin xyz="0 0 0" rpy="0 0 0"/>
-            <geometry>
-                <mesh filename="$(arg zed_meshfile)" />
-            </geometry>
-        </visual>
-    </link>
-<!-- Left Camera -->
-    <joint name="zed_left_camera_joint" type="fixed">
-        <parent link="zed_camera_center"/>
-        <child link="zed_left_camera_frame"/>
-        <origin xyz="0 0.06 0" rpy="0 0 0" />
-    </joint>
-    <link name="zed_left_camera_frame" />
-    <joint name="zed_left_camera_optical_joint" type="fixed">
-        <origin xyz="0 0 0" rpy="-${M_PI/2} 0.0 -${M_PI/2}"/>
-        <parent link="zed_left_camera_frame"/>
-        <child link="zed_left_camera_optical_frame"/>
-    </joint>
-    <link name="zed_left_camera_optical_frame"/>
-<!-- Right Camera -->
-    <joint name="zed_right_camera_joint" type="fixed">
-        <parent link="zed_camera_center"/>
-        <child link="zed_right_camera_frame"/>
-        <origin xyz="0 -0.06 0" rpy="0 0 0" />
-    </joint>
-    <link name="zed_right_camera_frame" />
-    <joint name="zed_right_camera_optical_joint" type="fixed">
-        <origin xyz="0 0 0" rpy="-${M_PI/2} 0.0 -${M_PI/2}"/>
-        <parent link="zed_right_camera_frame"/>
-        <child link="zed_right_camera_optical_frame"/>
-    </joint>
-    <link name="zed_right_camera_optical_frame"/>
-<!---->
-<xacro:if value="$(arg sim)">
-    <stereo_camera frame_rgb="zed_camera_center" frame_depth="zed_depth_dummy_frame_sim_only" cameraName="zed"  topic="pointcloud" robot_namespace="$(arg robot_namespace)"/>
-    <link name="zed_depth_dummy_frame_sim_only"></link>
-    <joint name="zed_camera_depth_joint" type="fixed">
-      <origin xyz="0 0 0" rpy="${-pi/2} 0 ${-pi/2}"/>
-      <parent link="zed_camera_center"/>
-      <child link="zed_depth_dummy_frame_sim_only"/>
-    </joint>
-</xacro:if>
-  <!-- realsense Camera -->
-<!-- Links only needed in simulation, created by realsense software otherwise-->
-  <link
-    name="realsense_link">
-      <visual>
-      <origin xyz="0 0 0" rpy="0 0 0"/>
-      <geometry>
-          <mesh filename="$(arg realsense_meshfile)" />
-      </geometry>
-    </visual>
-  </link>
-  <joint name="realsense_joint" type="fixed">
-    <origin xyz="$(arg real_base)" rpy="$(arg real_rpy)"/>
-    <parent link="chassis_link"/>
-    <child link="realsense_link"/>
-  </joint>
-<xacro:if value="$(arg sim)">
-  <stereo_camera frame_rgb="realsense_color_frame" frame_depth="realsense_depth_dummy_frame_sim_only" cameraName="realsense" topic="pointcloud" robot_namespace="$(arg robot_namespace)"/>
-  <link name="realsense_color_frame"> </link>
-  <link name="realsense_depth_frame"></link>
-   <link name="realsense_depth_dummy_frame_sim_only"></link>
-  <link
-    name="realsense_depth_optical_frame">
-  </link>
-  <link
-    name="realsense_color_optical_frame">
-  </link>
-  <joint name="realsense_gb_joint" type="fixed">
-    <origin xyz="$(arg real_rgb_xyz)" rpy="0 0 0"/>
-    <parent link="realsense_link"/>
-    <child link="realsense_color_frame"/>
-  </joint>
-  <joint name="realsense_depth_joint" type="fixed">
-    <origin xyz="$(arg real_depth_xyz)" rpy="0 0 0"/>
-    <parent link="realsense_link"/>
-    <child link="realsense_depth_frame"/>
-  </joint>
-  <joint name="realsense_depth_dummy_joint" type="fixed">
-    <origin xyz="$(arg real_depth_xyz)" rpy="-${M_PI/2} 0.0 -${M_PI/2}"/>
-    <parent link="realsense_link"/>
-    <child link="realsense_depth_dummy_frame_sim_only"/>
-  </joint>
-  <joint name="realsense_optical_color_joint" type="fixed">
-    <origin xyz="0 0 0" rpy="$(arg real_optical_rpy)"/>
-    <parent link="realsense_color_frame"/>
-    <child link="realsense_color_optical_frame"/>
-  </joint>
-  <joint name="realsense_optical_depth_joint" type="fixed">
-    <origin xyz="0 0 0" rpy="$(arg real_depth_rpy)"/>
-    <parent link="realsense_depth_frame"/>
-    <child link="realsense_depth_optical_frame"/>
-  </joint>
-</xacro:if>
-<xacro:if value="$(arg sim)">
-  <!-- Fake UWB -->
-  <gazebo>
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
File: unicorn_description/urdf/wheel.urdf.xacro (robot description, xacro)
@@ -30,6 +30,6 @@
         <friction>
           <ode>
-            <mu>0.4</mu>
-            <mu2>0.4</mu2>
+            <mu>0.8</mu>
+            <mu2>0.8</mu2>
           </ode>
         </friction>
